File: Hardware/Flight/ARM Board/ARM Board.sch (KiCad schematic (older format))
At the start: 24 parts, among them J1 USB_B_Micro, J2 Conn_01x20_Female, J3 SD_WM6698CT-ND, J4 Conn_01x20_Female, U1 STM32L4x6RxT6, U2 MSP430FR2355, Y1 Crystal_GND23

Commit message: Added regulator, CAN bus and power switch
Parts:
- removed J1: USB_B_Micro, ARMlib:USB_Micro-B_Amphenol_10118193-0001LF, symbol Connector:USB_B_Micro
- added C? (x2): 10uF, symbol Device:C
- added C?: 4.7uF, symbol Device:C
- added C?: 100nF, symbol Device:C
- added D? (x2): BAT60JFILM, Diodes_SMD:D_SOD-323_HandSoldering, symbol pspice:DIODE
- added J?: Harwin_M80-5400642, canhw_footprints:connector_Harwin_M80-5000642, symbol Payload_Connectors:Harwin_M80-5400642
- added R?: 120, Resistors_SMD:R_0603, symbol Device:R
- added R?: DNP, Resistors_SMD:R_0603, symbol Device:R
- added SW?: SW_SPST, ARMlib:SPST_GF-123-0054, symbol Switch:SW_SPST
- added U?: MCP2562, symbol canhw:MCP2562
- added VR?: LD39200PU33R, Housings_DFN_QFN:DFN-6-1EP_3x3mm_Pitch0.95mm, symbol Regulators:LD39200PU33R
Connections:
- net labels added: CANRX, CANTX, VBUS, VDD33_IN, VDD5_IN, ~CAN_EN
- net labels removed: VDD5
- wire segments 109 -> 174
Other:
- note added: "TODO\n-Programming IO\n-SD Card Capacitors\n-Connect MSP430\n\n"
- note removed: "TODO\n-Programming IO\n-ADD CANBUS\n-POWER SWITCH & input\n-Battery Choke?\n-Power caps?\n-3.3V Regulator\n-SD Card Capacitors\n"
- moved on the sheet: C1, C2, C?, J?, L?, R1, R?, Y1

Commit message: rearranged libraries
Parts:
- removed U1: STM32L4x6RxT6, STM32L4x6RxT6:STM32L4x6RxT6, symbol ARM-Board-rescue:STM32L4x6RxT6-symbols
- added U?: STM32L4x6RxT6-symbols-ARM-Board-rescue, LQFP64-10x10mm, symbol Payload_Microcontrollers:STM32L4x6RxT6-symbols-ARM-Board-rescue
- J2, J4: symbol ARM-Board-rescue:Conn_01x20_Female-ARMlib -> Payload_Connections:Conn_01x20_Female
- J3, J?: symbol ARM-Board-rescue:SD_WM6698CT-ND-ARMlib -> Payload_Connections:SD_WM6698CT-ND-ARMlib-ARM-Board-rescue
- J?: symbol Payload_Connectors:Harwin_M80-5400642 -> Payload_Connections:Harwin_M80-5400642
- U2: symbol ARM-Board-rescue:MSP430FR2355-MSP430FR2355 -> Payload_Microcontrollers:MSP430FR2355-MSP430FR2355-ARM-Board-rescue
- U?: symbol ARMlib:SRAM_23LC1024T-I_ST -> Payload_Microcontrollers:SRAM_23LC1024T-I_ST-ARMlib
- U?: symbol symbols:STM32L4x6RxT6 -> Payload_Microcontrollers:STM32L4x6RxT6-symbols
- U?: symbol canhw:MCP2562 -> Payload_Canhw:MCP2562-canhw
- VR?: symbol Regulators:LD39200PU33R -> Payload_Regulators:LD39200PU33R
Connections:
- wire segments 174 -> 172
Changed lines of the file:
@@
 EESchema Schematic File Version 4
-LIBS:ARM Board-cache
 EELAYER 26 0
 EELAYER END
@@
 $EndDescr
 $Comp
-L ARM-Board-rescue:STM32L4x6RxT6-symbols U1
-U 2 1 5BE24AAA
-P 9500 3100
-F 0 "U1" H 10450 3650 60  0000 C CNN
-F 1 "STM32L4x6RxT6" H 10450 3550 60  0000 C CNN
-F 2 "STM32L4x6RxT6:STM32L4x6RxT6" H 10350 3450 60  0001 C CNN
-F 3 "" H 9500 3200 60  0000 C CNN
-	2    9500 3100
-	1    0    0    -1
-$EndComp
-$Comp
-L ARM-Board-rescue:SD_WM6698CT-ND-ARMlib J3
+L Payload_Connections:SD_WM6698CT-ND-ARMlib-ARM-Board-rescue J3
 U 1 1 5BE5108C
 P 15550 9150
@@
 	14850 7750 14850 8100
 $Comp
-L ARM-Board-rescue:Conn_01x20_Female-ARMlib J4
+L Payload_Connections:Conn_01x20_Female J4
 U 1 1 5BE939D5
 P 1450 9250
@@
 $EndComp
 $Comp
-L ARM-Board-rescue:Conn_01x20_Female-ARMlib J2
+L Payload_Connections:Conn_01x20_Female J2
 U 1 1 5BE93A8D
 P 1400 5900
@@
 $EndComp
 $Comp
-L ARM-Board-rescue:MSP430FR2355-MSP430FR2355 U2
+L Payload_Microcontrollers:MSP430FR2355-MSP430FR2355-ARM-Board-rescue U2
 U 1 1 5BF776E6
 P 15750 3550
@@
 	8650 3500 9100 3500
 Wire Wire Line
-	9500 3700 9500 3600
-Wire Wire Line
-	9500 3600 9500 3500
-Connection ~ 9500 3600
-Wire Wire Line
 	9500 3500 9300 3500
-Connection ~ 9500 3500
 Connection ~ 9100 3500
 Wire Wire Line
@@
 Connection ~ 11450 3800
 $Comp
-L ARM-Board-rescue:SD_WM6698CT-ND-ARMlib J?
+L Payload_Connections:SD_WM6698CT-ND-ARMlib-ARM-Board-rescue J?
 U 1 1 5BFE231B
 P 17400 9450
@@
 	10900 8300 11000 8300
 Wire Wire Line
-	11000 8300 11000 8950
-Wire Wire Line
 	10900 8950 11000 8950
 Connection ~ 11000 8950
-Wire Wire Line
-	11000 8950 11000 9100
 Text Notes 9000 9100 0    50   ~ 0
 Ground other XTAL pins? Floating in datasheet...\n
@@
 SD Card Logging
 $Comp
-L ARMlib:SRAM_23LC1024T-I_ST U?
+L Payload_Microcontrollers:SRAM_23LC1024T-I_ST-ARMlib U?
 U 1 1 5BFFCC54
 P 15900 6550
@@
 	4400 5200 5250 5200
 $Comp
-L symbols:STM32L4x6RxT6 U?
+L Payload_Microcontrollers:STM32L4x6RxT6-symbols U?
 U 1 1 5C039DAA
 P 7950 5350
@@
 	4700 4900 5250 4900
 $Comp
-L Regulators:LD39200PU33R VR?
+L Payload_Regulators:LD39200PU33R VR?
 U 1 1 5C09F3A5
 P 4100 2250
@@
 	2100 2350 2100 2900
 $Comp
-L Payload_Connectors:Harwin_M80-5400642 J?
+L Payload_Connections:Harwin_M80-5400642 J?
 U 1 1 5C184B36
 P 3650 6800
@@
 $EndComp
 $Comp
-L canhw:MCP2562 U?
+L Payload_Canhw:MCP2562-canhw U?
 U 1 1 5C184EB2
 P 5300 7100
@@
 Wire Wire Line
 	7550 6750 7950 6750
+$Comp
+L Payload_Microcontrollers:STM32L4x6RxT6-symbols-ARM-Board-rescue U?
+U 2 1 5C15893F
+P 9500 3100
+F 0 "U?" H 10400 3487 60  0000 C CNN
+F 1 "STM32L4x6RxT6-symbols-ARM-Board-rescue" H 10400 3381 60  0000 C CNN
+F 2 "LQFP64-10x10mm" H 10350 3450 60  0001 C CNN
+F 3 "" H 9500 3200 60  0000 C CNN
+	2    9500 3100
+	1    0    0    -1
+$EndComp
+Wire Wire Line
+	11000 8900 11000 8950
+Wire Wire Line
+	11000 8950 11000 9100
 $EndSCHEMATC

Commit message: Added JTAG I/O, USB UART connections, modified headers and power circuit, added I2C for MSP430
Parts:
- removed J2: Conn_01x20_Female, ARMlib:IO_Connector, symbol Payload_Connections:Conn_01x20_Female
- removed U2: MSP430FR2355, ARMlib:48-LQFP, symbol Payload_Microcontrollers:MSP430FR2355-MSP430FR2355-ARM-Board-rescue
- added J2: Conn_01x10, Payload_Connectors:JTAG_CONN_20021311-00010T4LF, symbol Connector_Generic:Conn_01x10
- added R15, R16: DNP, Resistors_SMD:R_0603, symbol Device:R
- added R2: 0, Resistors_SMD:R_0603, symbol Device:R
- added R3: 10K, Resistors_SMD:R_0603, symbol Device:R
- added R6, R7: 4.7K, Resistors_SMD:R_0603, symbol Device:R
- C1, C2: footprint (none) -> Capacitors_SMD:C_0603
- C10, C12, C13, C14, C3, C4, C5, C6, C7, C8, C9: renamed from C?; footprint (none) -> Capacitors_SMD:C_0603
- C11: renamed from C?; footprint (none) -> Capacitors_SMD:C_0805
- J3: symbol Payload_Connections:SD_WM6698CT-ND-ARMlib-ARM-Board-rescue -> ARM-Board-rescue:SD_WM6698CT-ND-ARMlib-ARM-Board-rescue-Payload_Connections
- J4: footprint ARMlib:IO_Connector -> Payload_Connectors:IO_Connector; symbol Payload_Connections:Conn_01x20_Female -> ARM-Board-rescue:Conn_01x20_Female-Payload_Connections
- J5: renamed from J?; symbol Payload_Connections:Harwin_M80-5400642 -> ARM-Board-rescue:Harwin_M80-5400642-Payload_Connections
- J6: renamed from J?; symbol Payload_Connections:SD_WM6698CT-ND-ARMlib-ARM-Board-rescue -> ARM-Board-rescue:SD_WM6698CT-ND-ARMlib-ARM-Board-rescue-Payload_Connections
- R1: value R -> DNP
- R8: renamed from R?; value R -> DNP
- U1: renamed from U?; symbol Payload_Microcontrollers:STM32L4x6RxT6-symbols-ARM-Board-rescue -> ARM-Board-rescue:STM32L4x6RxT6-symbols-ARM-Board-rescue-Payload_Microcontrollers
- U2: renamed from U?; symbol Payload_Microcontrollers:STM32L4x6RxT6-symbols -> ARM-Board-rescue:STM32L4x6RxT6-symbols-Payload_Microcontrollers
- U3: renamed from U?; symbol Payload_Microcontrollers:SRAM_23LC1024T-I_ST-ARMlib -> ARM-Board-rescue:SRAM_23LC1024T-I_ST-ARMlib-Payload_Microcontrollers
- U4: renamed from U?; footprint (none) -> Housings_SOIC:SOIC-8_3.9x4.9mm_Pitch1.27mm; symbol Payload_Canhw:MCP2562-canhw -> ARM-Board-rescue:MCP2562-canhw-Payload_Canhw
- VR1: renamed from VR?; symbol Payload_Regulators:LD39200PU33R -> ARM-Board-rescue:LD39200PU33R-Payload_Regulators
- gave numbers to parts that had none: 7
Connections:
- net labels added: JTCK_SWCLK, JTDI, JTDO_SWO, JTMS_SWDIO, JTRST, SCL, SDA, UART_RX, UART_TX, UART_~CTS, UART_~RTS, VDD33_USB, VTREF, ~RST
- wire segments 172 -> 227
Other:
- note removed: "Ground other XTAL pins? Floating in datasheet...\n"
- note removed: "TODO\n-Programming IO\n-SD Card Capacitors\n-Connect MSP430\n\n"
- moved on the sheet: D1, D2, R1, R4, R8

Commit message: Updated libraries and footprints, netlist
Parts:
- J1: footprint (none) -> Payload_Connectors:USB_Micro-B_Amphenol_10118193-0001LF
- J3, J6: footprint (none) -> Payload_Connectors:MICROSD_WM6698CT-ND
- L1: footprint (none) -> Resistors_SMD:R_0603_HandSoldering
- SW1: footprint ARMlib:SPST_GF-123-0054 -> (none)
- U2: footprint LQFP64-10x10mm -> Payload_standard:STM32L4x6RxT6
- Y1: footprint ARMlib:MC-306 32.7680K -> Payload_XTAL:MC-306
Changed lines of the file:
@@
 F 0 "J3" H 12828 8252 60  0000 L CNN
 F 1 "SD_WM6698CT-ND" H 12828 8146 60  0000 L CNN
-F 2 "" V 12300 8050 60  0001 C CNN
+F 2 "Payload_Connectors:MICROSD_WM6698CT-ND" V 12300 8050 60  0001 C CNN
 F 3 "" V 12300 8050 60  0001 C CNN
 	1    12350 8150
@@
 F 0 "Y1" H 10550 8950 50  0000 L CNN
 F 1 "Crystal_GND23" H 10300 8050 50  0000 L CNN
-F 2 "ARMlib:MC-306 32.7680K" H 10550 8600 50  0001 C CNN
+F 2 "Payload_XTAL:MC-306" H 10550 8600 50  0001 C CNN
 F 3 "~" H 10550 8600 50  0001 C CNN
 	1    10550 8600
@@
 F 0 "L1" V 10176 2300 50  0000 C CNN
 F 1 "Ferrite_Bead" V 10267 2300 50  0000 C CNN
-F 2 "" V 10380 2300 50  0001 C CNN
+F 2 "Resistors_SMD:R_0603_HandSoldering" V 10380 2300 50  0001 C CNN
 F 3 "~" H 10450 2300 50  0001 C CNN
 	1    10450 2300
@@
 F 0 "J6" H 14678 8552 60  0000 L CNN
 F 1 "SD_WM6698CT-ND" H 14678 8446 60  0000 L CNN
-F 2 "" V 14150 8350 60  0001 C CNN
+F 2 "Payload_Connectors:MICROSD_WM6698CT-ND" V 14150 8350 60  0001 C CNN
 F 3 "" V 14150 8350 60  0001 C CNN
 	1    14200 8450
@@
 F 0 "J1" H 4155 5567 50  0000 C CNN
 F 1 "USB_OTG" H 4155 5476 50  0000 C CNN
-F 2 "" H 4250 5050 50  0001 C CNN
+F 2 "Payload_Connectors:USB_Micro-B_Amphenol_10118193-0001LF" H 4250 5050 50  0001 C CNN
 F 3 " ~" H 4250 5050 50  0001 C CNN
 	1    4100 5100
@@
 F 0 "U2" H 9550 5837 60  0000 C CNN
 F 1 "STM32L4x6RxT6" H 9550 5731 60  0000 C CNN
-F 2 "LQFP64-10x10mm" H 8800 5700 60  0001 C CNN
+F 2 "Payload_standard:STM32L4x6RxT6" H 8800 5700 60  0001 C CNN
 F 3 "" H 7950 5450 60  0000 C CNN
 	1    7950 5350
@@
 F 0 "SW1" H 2350 3685 50  0000 C CNN
 F 1 "SW_SPST" H 2350 3594 50  0000 C CNN
-F 2 "ARMlib:SPST_GF-123-0054" H 2350 3450 50  0001 C CNN
+F 2 "" H 2350 3450 50  0001 C CNN
 F 3 "" H 2350 3450 50  0001 C CNN
 	1    2350 3450

Commit message: SPI added to header, Layout finished
Parts:
- removed R4: DNP, Resistors_SMD:R_0603, symbol Device:R
- removed SW1: SW_SPST, symbol Switch:SW_SPST
- added J7: 1053131202, Payload_Connectors:MOLEX_1053131202, symbol Molex_Nano:1053131202
- J2: footprint Payload_Connectors:JTAG_CONN_20021311-00010T4LF -> Pin_Headers:Pin_Header_Straight_2x05_Pitch2.54mm
- J4: footprint Payload_Connectors:IO_Connector -> Pin_Headers:Pin_Header_Straight_2x10_Pitch2.54mm
- U2: renamed from U1; value STM32L4x6RxT6-symbols-ARM-Board-rescue -> STM32L4x6RxT6; footprint LQFP64-10x10mm -> Payload_standard:STM32L4x6RxT6
Connections:
- net labels added: D+, D-, ~CS2_2, ~CS3_2
- wire segments 227 -> 230
Changed lines of the file:
@@
 F 0 "J4" H 1444 7975 50  0000 C CNN
 F 1 "Conn_01x20_Female" H 1444 8066 50  0000 C CNN
-F 2 "Payload_Connectors:IO_Connector" H 1500 9200 50  0001 C CNN
+F 2 "Pin_Headers:Pin_Header_Straight_2x10_Pitch2.54mm" H 1500 9200 50  0001 C CNN
 F 3 "~" H 1500 9200 50  0001 C CNN
 	1    1450 9250
@@
 ~HOLD1
 Text GLabel 11850 7600 0    50   Input ~ 0
-MOSI2
+MOSI3
 Text GLabel 11850 7700 0    50   Input ~ 0
-SCK2
-Text GLabel 11850 7800 0    50   Input ~ 0
-~CS2
+SCK3
 Text GLabel 13700 7900 0    50   Input ~ 0
 MOSI3
 Text GLabel 11500 7500 0    50   Input ~ 0
-MISO2
+MISO3
 Wire Wire Line
 	11500 7500 11650 7500
@@
 Text Notes 12700 5300 0    50   ~ 0
 RAM
-Text GLabel 11500 8100 1    50   Input ~ 0
+Text GLabel 11050 7600 1    50   Input ~ 0
 VDD33
 Text GLabel 13300 8250 1    50   Input ~ 0
@@
 Wire Wire Line
 	13300 8450 13700 8450
-Wire Wire Line
-	11500 8100 11500 8150
-Wire Wire Line
-	11500 8150 11850 8150
 $Sheet
 S 5250 4750 650  700
@@
 F5 "~CTS" I R 5900 5300 50
 F6 "USB_5V" I L 5250 4900 50
-F7 "DM" I L 5250 5200 50
-F8 "DP" I L 5250 5100 50
+F7 "D_M" I L 5250 5200 50
+F8 "D_P" I L 5250 5100 50
 $EndSheet
 Wire Wire Line
@@
 Text GLabel 9900 6950 2    50   Input ~ 0
 MISO2
-Text GLabel 9900 6550 2    50   Input ~ 0
+Text GLabel 7950 6350 0    50   Input ~ 0
 SCK2
 Text GLabel 9900 6750 2    50   Input ~ 0
@@
 Text GLabel 7950 8250 0    50   Input ~ 0
 SCK3
-Text GLabel 7950 5850 0    50   Input ~ 0
+Text GLabel 7950 7950 0    50   Input ~ 0
 ~CS3
 Text GLabel 7950 8450 0    50   Input ~ 0
@@
 Wire Wire Line
 	1750 10100 1750 10250
-Text GLabel 7950 6250 0    50   Input ~ 0
+Text GLabel 7950 5850 0    50   Input ~ 0
 ~HOLD1
 Text GLabel 1750 8000 1    50   Input ~ 0
@@
 Wire Wire Line
 	1950 8000 1950 8300
-Text GLabel 4700 4700 1    50   Input ~ 0
-VBUS
 $Comp
 L ARM-Board-rescue:LD39200PU33R-Payload_Regulators VR1
@@
 Connection ~ 3250 2350
 $Comp
-L Switch:SW_SPST SW1
-U 1 1 5C1FDFEF
-P 2350 3450
-F 0 "SW1" H 2350 3685 50  0000 C CNN
-F 1 "SW_SPST" H 2350 3594 50  0000 C CNN
-F 2 "" H 2350 3450 50  0001 C CNN
-F 3 "" H 2350 3450 50  0001 C CNN
-	1    2350 3450
-	1    0    0    -1
-$EndComp
-$Comp
-L Device:R R4
-U 1 1 5C2102C6
-P 7200 6750
-F 0 "R4" H 7270 6796 50  0000 L CNN
-F 1 "DNP" H 7270 6705 50  0000 L CNN
-F 2 "Resistors_SMD:R_0603" V 7130 6750 50  0001 C CNN
-F 3 "~" H 7200 6750 50  0001 C CNN
-	1    7200 6750
-	1    0    0    -1
-$EndComp
-$Comp
-L power:GND #PWR0122
-U 1 1 5C21041D
-P 7200 7000
-F 0 "#PWR0122" H 7200 6750 50  0001 C CNN
-F 1 "GND" H 7205 6827 50  0000 C CNN
-F 2 "" H 7200 7000 50  0001 C CNN
-F 3 "" H 7200 7000 50  0001 C CNN
-	1    7200 7000
-	1    0    0    -1
-$EndComp
-$Comp
-L ARM-Board-rescue:STM32L4x6RxT6-symbols-ARM-Board-rescue-Payload_Microcontrollers U1
+L ARM-Board-rescue:STM32L4x6RxT6-symbols-ARM-Board-rescue-Payload_Microcontrollers U2
 U 2 1 5C15893F
 P 9500 3100
-F 0 "U1" H 10400 3487 60  0000 C CNN
-F 1 "STM32L4x6RxT6-symbols-ARM-Board-rescue" H 10400 3381 60  0000 C CNN
-F 2 "LQFP64-10x10mm" H 10350 3450 60  0001 C CNN
+F 0 "U2" H 10400 3487 60  0000 C CNN
+F 1 "STM32L4x6RxT6" H 10400 3381 60  0000 C CNN
+F 2 "Payload_standard:STM32L4x6RxT6" H 10350 3450 60  0001 C CNN
 F 3 "" H 9500 3200 60  0000 C CNN
 	2    9500 3100
@@
 	2100 3550 2100 3450
 Wire Wire Line
-	2100 3450 2150 3450
-Wire Wire Line
 	1750 3000 2100 3000
 Wire Wire Line
@@
 Text GLabel 2750 3450 2    50   Input ~ 0
 VDD33
-Wire Wire Line
-	2550 3450 2650 3450
 Wire Wire Line
 	10150 5300 10150 5550
@@
 Wire Wire Line
 	10200 5650 9900 5650
-Wire Wire Line
-	7050 6450 7200 6450
-Wire Wire Line
-	7200 6600 7200 6450
-Wire Wire Line
-	7200 6900 7200 7000
 Text GLabel 7750 7150 0    50   Input ~ 0
 SCL
@@
 Wire Wire Line
 	7900 8150 7950 8150
-Text GLabel 2000 5350 2    50   Input ~ 0
+Text GLabel 2000 5150 2    50   Input ~ 0
 JTDI
 Text GLabel 7850 6850 0    50   Input ~ 0
@@
 Wire Wire Line
 	7850 6850 7950 6850
-Wire Wire Line
-	7950 6450 7200 6450
-Connection ~ 7200 6450
 Text GLabel 7850 6750 0    50   Input ~ 0
 JTMS_SWDIO
 Wire Wire Line
 	7850 6750 7950 6750
-Text GLabel 2000 5450 2    50   Input ~ 0
+Text GLabel 1550 5750 2    50   Input ~ 0
 JTMS_SWDIO
-Text GLabel 2000 5550 2    50   Input ~ 0
+Text GLabel 1550 5550 2    50   Input ~ 0
 JTCK_SWCLK
-Wire Wire Line
-	4400 4900 4700 4900
-Wire Wire Line
-	4700 4700 4700 4900
-Connection ~ 4700 4900
-Wire Wire Line
-	4700 4900 5250 4900
-Text GLabel 2000 5250 2    50   Input ~ 0
+Text GLabel 1700 4950 2    50   Input ~ 0
 JTRST
-Text GLabel 2000 5050 2    50   Input ~ 0
-VBUS
-Text GLabel 2000 5150 2    50   Input ~ 0
+Text GLabel 2100 5850 2    50   Input ~ 0
 VTREF
 Text GLabel 2800 3750 2    50   Input ~ 0
@@
 Wire Wire Line
 	2650 3450 2750 3450
-Text GLabel 2000 5650 2    50   Input ~ 0
+Text GLabel 2000 5350 2    50   Input ~ 0
 JTDO_SWO
 $Comp
 L power:GND #PWR0123
 U 1 1 5C452C69
-P 2100 5900
-F 0 "#PWR0123" H 2100 5650 50  0001 C CNN
-F 1 "GND" H 2105 5727 50  0000 C CNN
-F 2 "" H 2100 5900 50  0001 C CNN
-F 3 "" H 2100 5900 50  0001 C CNN
-	1    2100 5900
-	1    0    0    -1
-$EndComp
-Wire Wire Line
-	1550 5050 2000 5050
+P 2600 5750
+F 0 "#PWR0123" H 2600 5500 50  0001 C CNN
+F 1 "GND" H 2605 5577 50  0000 C CNN
+F 2 "" H 2600 5750 50  0001 C CNN
+F 3 "" H 2600 5750 50  0001 C CNN
+	1    2600 5750
+	1    0    0    -1
+$EndComp
 Text GLabel 7250 4700 1    50   Input ~ 0
 ~RST
@@
 	2000 5150 1550 5150
 Wire Wire Line
-	2000 5250 1550 5250
-Wire Wire Line
 	1550 5350 2000 5350
-Wire Wire Line
-	1550 5450 2000 5450
-Wire Wire Line
-	1550 5550 2000 5550
-Wire Wire Line
-	1550 5650 2000 5650
-Text GLabel 2450 5750 2    50   Input ~ 0
+Text GLabel 1750 4850 2    50   Input ~ 0
 ~RST
 Wire Wire Line
-	2450 5750 1550 5750
-Wire Wire Line
 	1550 5850 2100 5850
-Wire Wire Line
-	2100 5850 2100 5900
 Wire Wire Line
 	7750 7250 7950 7250
@@
 F 0 "J2" H 1270 4725 50  0000 C CNN
 F 1 "Conn_01x10" H 1270 4816 50  0000 C CNN
-F 2 "Payload_Connectors:JTAG_CONN_20021311-00010T4LF" H 1350 5450 50  0001 C CNN
+F 2 "Pin_Headers:Pin_Header_Straight_2x05_Pitch2.54mm" H 1350 5450 50  0001 C CNN
 F 3 "~" H 1350 5450 50  0001 C CNN
 	1    1350 5450
 	-1   0    0    1
 $EndComp
+Text GLabel 1750 9500 2    50   Input ~ 0
+MOSI2
+Text GLabel 1750 9400 2    50   Input ~ 0
+SCK2
+Text GLabel 1750 9300 2    50   Input ~ 0
+~CS2
+Text GLabel 1750 9600 2    50   Input ~ 0
+MISO2
+Wire Wire Line
+	1750 9300 1600 9300
+Wire Wire Line
+	1750 9400 1600 9400
+Wire Wire Line
+	1750 9500 1600 9500
+Wire Wire Line
+	1750 9600 1600 9600
+Wire Wire Line
+	11050 7600 11050 8150
+Wire Wire Line
+	11050 8150 11850 8150
+Text GLabel 11850 7800 0    50   Input ~ 0
+~CS3_2
+Text GLabel 7950 8050 0    50   Input ~ 0
+~CS3_2
+Text GLabel 1750 9200 2    50   Input ~ 0
+~CS2_2
+Wire Wire Line
+	1600 9200 1750 9200
+Text GLabel 9900 6650 2    50   Input ~ 0
+~CS2_2
+$Comp
+L Molex_Nano:1053131202 J7
+U 1 1 5C3240C2
+P 2450 3800
+F 0 "J7" V 2348 3930 50  0000 L CNN
+F 1 "1053131202" V 2439 3930 50  0000 L CNN
+F 2 "Payload_Connectors:MOLEX_1053131202" H 2450 3800 50  0001 L BNN
+F 3 "Molex, LLC" H 2450 3800 50  0001 L BNN
+F 4 "None" H 2450 3800 50  0001 L BNN "Field4"
+F 5 "WM14972-ND" H 2450 3800 50  0001 L BNN "Field5"
+F 6 "https://www.digikey.ca/product-detail/en/molex-llc/1053131202/WM14972-ND/6131614?utm_source=snapeda&utm_medium=aggregator&utm_campaign=symbol" H 2450 3800 50  0001 L BNN "Field6"
+F 7 "Nano-Fit Right Angle Header; Through Hole; 2.50mm; Single Row; 2 Circuit; Gold Plated" H 2450 3800 50  0001 L BNN "Field7"
+F 8 "1053131202" H 2450 3800 50  0001 L BNN "Field8"
+	1    2450 3800
+	0    1    1    0
+$EndComp
+Wire Wire Line
+	2350 3450 2350 3600
+Wire Wire Line
+	2100 3450 2350 3450
+Wire Wire Line
+	2450 3600 2450 3450
+Wire Wire Line
+	2450 3450 2650 3450
+Wire Wire Line
+	4400 4900 5250 4900
+Wire Wire Line
+	7050 6450 7950 6450
+Text Label 4850 5100 0    50   ~ 0
+D+
+Text Label 4900 5200 0    50   ~ 0
+D-
+Wire Wire Line
+	2600 5650 2600 5750
+Wire Wire Line
+	1550 5650 2600 5650
+Wire Wire Line
+	2600 5450 2600 5650
+Wire Wire Line
+	1550 5450 2600 5450
+Connection ~ 2600 5650
+Wire Wire Line
+	1550 4950 1600 4950
+Wire Wire Line
+	1750 4850 1600 4850
+Wire Wire Line
+	1600 4850 1600 4950
+Connection ~ 1600 4950
+Wire Wire Line
+	1600 4950 1700 4950
+$Comp
+L power:GND #PWR?
+U 1 1 5C3F5323
+P 4250 2900
+F 0 "#PWR?" H 4250 2650 50  0001 C CNN
+F 1 "GND" H 4255 2727 50  0000 C CNN
+F 2 "" H 4250 2900 50  0001 C CNN
+F 3 "" H 4250 2900 50  0001 C CNN
+	1    4250 2900
+	1    0    0    -1
+$EndComp
 $EndSCHEMATC
