File: Hardware/Flight/ARM Board/ARM Board.sch (KiCad schematic (older format))
At the start: 38 parts, among them J1 USB_OTG, J2 Conn_01x10, J3 SD_WM6698CT-ND, J4 Conn_01x20_Female, J5 Harwin_M80-5400642, J6 SD_WM6698CT-ND, J7 1053131202, U2 STM32L4x6RxT6, U3 SRAM_23LC1024T-I_ST, U4 MCP2562, Y1 Crystal_GND23

Commit message: Started new layout rev 2
Parts:
- removed J3: SD_WM6698CT-ND, Payload_Connectors:MICROSD_WM6698CT-ND, symbol Payload_Connectors:SD_WM6698CT-ND-ARMlib-ARM-Board-rescue
- removed J4: Conn_01x20_Female, Pin_Headers:Pin_Header_Straight_2x10_Pitch2.54mm, symbol Payload_Connectors:Conn_01x20_Female
- removed J5: Harwin_M80-5400642, canhw_footprints:connector_Harwin_M80-5000642, symbol Payload_Connectors:Harwin_M80-5400642
- removed J7: 1053131202, Payload_Connectors:MOLEX_1053131202, symbol ARM-Board-rescue:1053131202-Molex_Nano
- removed U2: STM32L4x6RxT6, Payload_standard:STM32L4x6RxT6, symbol Payload_Microcontrollers:STM32L4x6RxT6-symbols
- removed U3: SRAM_23LC1024T-I_ST, Housings_SSOP:TSSOP-8_4.4x3mm_Pitch0.65mm, symbol Payload_Microcontrollers:SRAM_23LC1024T-I_ST-ARMlib
- removed U4: MCP2562, Housings_SOIC:SOIC-8_3.9x4.9mm_Pitch1.27mm, symbol Payload_Canhw:MCP2562-canhw
- added J3: 1053131202, Payload_Connectors:MOLEX_1053131202, symbol Molex_Nano:1053131202
- added J4: Harwin_M80-5400642, Payload_Connectors:connector_Harwin_M80-5000642, symbol Payload_Connectors:Harwin_M80-5400642
- added J5: SD_WM6698CT-ND-ARMlib-ARM-Board-rescue, Payload_Connectors:MICROSD_WM6698CT-ND, symbol Payload_Connectors:SD_WM6698CT-ND-ARMlib-ARM-Board-rescue
- added J7: Conn_01x20_Female, Pin_Headers:Pin_Header_Straight_2x10_Pitch2.54mm, symbol Payload_Connectors:Conn_01x20_Female
- added U1: STM32L4x6RxT6-symbols, Payload_StandardPackages:STM32L4x6RxT6, symbol Payload_Microcontrollers:STM32L4x6RxT6-symbols
- added U2: SRAM_23LC1024T-I_ST-ARMlib, Housings_SSOP:TSSOP-8_4.4x3mm_Pitch0.65mm, symbol Payload_Microcontrollers:SRAM_23LC1024T-I_ST-ARMlib
- added U3: MCP2562-canhw, Housings_SOIC:SOIC-8_3.9x4.9mm_Pitch1.27mm, symbol Payload_Canhw:MCP2562-canhw
- J6: value SD_WM6698CT-ND -> SD_WM6698CT-ND-ARMlib-ARM-Board-rescue
Connections:
- net labels added: PH3-BOOT0, ~CS1_2, ~HOLD3
- net labels removed: ~CS3_2, ~HOLD1

Commit message: finished layout rev2 on ARM board
Changed lines of the file:
@@
 Text GLabel 9900 6950 2    50   Input ~ 0
 MISO2
-Text GLabel 9900 6550 2    50   Input ~ 0
+Text GLabel 7950 6350 0    50   Input ~ 0
 SCK2
-Text GLabel 9900 6750 2    50   Input ~ 0
+Text GLabel 7950 6250 0    50   Input ~ 0
 ~CS2
 Text GLabel 9900 7050 2    50   Input ~ 0
@@
 Wire Wire Line
 	1600 9200 1750 9200
-Text GLabel 9900 6650 2    50   Input ~ 0
+Text GLabel 9900 6850 2    50   Input ~ 0
 ~CS2_2
 Wire Wire Line
@@
 Wire Wire Line
 	10050 7350 9900 7350
-Text GLabel 7950 6250 0    50   Input ~ 0
+Text GLabel 7950 7550 0    50   Input ~ 0
 ~CS1_2
 Text GLabel 1550 5250 2    50   Input ~ 0

Commit message: updated dongle for LoRa
Parts:
- J3: symbol Molex_Nano:1053131202 -> ARM-Board-rescue:1053131202-Molex_Nano
- J4: symbol Payload_Connectors:Harwin_M80-5400642 -> ARM-Board-rescue:Harwin_M80-5400642-Payload_Connectors
- J5, J6: symbol Payload_Connectors:SD_WM6698CT-ND-ARMlib-ARM-Board-rescue -> ARM-Board-rescue:SD_WM6698CT-ND-ARMlib-ARM-Board-rescue-Payload_Connectors
- J7: symbol Payload_Connectors:Conn_01x20_Female -> ARM-Board-rescue:Conn_01x20_Female-Payload_Connectors
- U1: symbol Payload_Microcontrollers:STM32L4x6RxT6-symbols -> ARM-Board-rescue:STM32L4x6RxT6-symbols-Payload_Microcontrollers
- U2: symbol Payload_Microcontrollers:SRAM_23LC1024T-I_ST-ARMlib -> ARM-Board-rescue:SRAM_23LC1024T-I_ST-ARMlib-Payload_Microcontrollers
- U3: symbol Payload_Canhw:MCP2562-canhw -> ARM-Board-rescue:MCP2562-canhw-Payload_Canhw
- VR1: symbol Payload_Regulators:LD39200PU33R -> ARM-Board-rescue:LD39200PU33R-Payload_Regulators
Changed lines of the file:
@@
 	13450 5400 13450 5700
 $Comp
-L Payload_Regulators:LD39200PU33R VR1
+L ARM-Board-rescue:LD39200PU33R-Payload_Regulators VR1
 U 1 1 5C3883E7
 P 4100 2250
@@
 $EndComp
 $Comp
-L Payload_Microcontrollers:STM32L4x6RxT6-symbols U1
+L ARM-Board-rescue:STM32L4x6RxT6-symbols-Payload_Microcontrollers U1
 U 1 1 5C399EA6
 P 7950 5350
@@
 $EndComp
 $Comp
-L Payload_Canhw:MCP2562-canhw U3
+L ARM-Board-rescue:MCP2562-canhw-Payload_Canhw U3
 U 1 1 5C39AF46
 P 5350 7100
@@
 $EndComp
 $Comp
-L Payload_Connectors:Harwin_M80-5400642 J4
+L ARM-Board-rescue:Harwin_M80-5400642-Payload_Connectors J4
 U 1 1 5C39B5CA
 P 3650 6800
@@
 $EndComp
 $Comp
-L Payload_Connectors:Conn_01x20_Female J7
+L ARM-Board-rescue:Conn_01x20_Female-Payload_Connectors J7
 U 1 1 5C39BC26
 P 1450 9250
@@
 $EndComp
 $Comp
-L Payload_Microcontrollers:STM32L4x6RxT6-symbols U1
+L ARM-Board-rescue:STM32L4x6RxT6-symbols-Payload_Microcontrollers U1
 U 2 1 5C39C6F4
 P 9500 3100
@@
 $EndComp
 $Comp
-L Payload_Connectors:SD_WM6698CT-ND-ARMlib-ARM-Board-rescue J6
+L ARM-Board-rescue:SD_WM6698CT-ND-ARMlib-ARM-Board-rescue-Payload_Connectors J6
 U 1 1 5C39D0BB
 P 14200 8450
@@
 $EndComp
 $Comp
-L Payload_Connectors:SD_WM6698CT-ND-ARMlib-ARM-Board-rescue J5
+L ARM-Board-rescue:SD_WM6698CT-ND-ARMlib-ARM-Board-rescue-Payload_Connectors J5
 U 1 1 5C39D81A
 P 12350 8150
@@
 $EndComp
 $Comp
-L Payload_Microcontrollers:SRAM_23LC1024T-I_ST-ARMlib U2
+L ARM-Board-rescue:SRAM_23LC1024T-I_ST-ARMlib-Payload_Microcontrollers U2
 U 1 1 5C39E125
 P 12700 5550
@@
 	7250 5350 7700 5350
 $Comp
-L Molex_Nano:1053131202 J3
+L ARM-Board-rescue:1053131202-Molex_Nano J3
 U 1 1 5C4A9E40
 P 2450 3800

Commit message: ARM board refactor
Parts:
- removed C1, C2: C_Small, Capacitors_SMD:C_0603, symbol Device:C_Small
- removed C10, C7, C8: 10uF, Capacitors_SMD:C_0603, symbol Device:C
- removed C11: 100uF, Capacitors_SMD:C_0805, symbol Device:C
- removed C12, C13, C14, C4, C6: 100nF, Capacitors_SMD:C_0603, symbol Device:C
- removed C3, C5: 4.7uF, Capacitors_SMD:C_0603, symbol Device:C
- removed C9: 1uF, Capacitors_SMD:C_0603, symbol Device:C
- removed D1, D2: BAT60JFILM, Diodes_SMD:D_SOD-323_HandSoldering, symbol pspice:DIODE
- removed J1: USB_OTG, Payload_Connectors:USB_Micro-B_Amphenol_10118193-0001LF, symbol Connector:USB_OTG
- removed J2: Conn_01x10, Pin_Headers:Pin_Header_Straight_2x05_Pitch2.54mm, symbol Connector_Generic:Conn_01x10
- removed J3: 1053131202, Payload_Connectors:MOLEX_1053131202, symbol ARM-Board-rescue:1053131202-Molex_Nano
- removed L1: Ferrite_Bead, Resistors_SMD:R_0603_HandSoldering, symbol Device:Ferrite_Bead
- removed R15, R16: DNP, Resistors_SMD:R_0603, symbol Device:R
- removed R2: 0, Resistors_SMD:R_0603, symbol Device:R
- removed R3: 10K, Resistors_SMD:R_0603, symbol Device:R
- removed R6, R7: 4.7K, Resistors_SMD:R_0603, symbol Device:R
- removed U1: STM32L4x6RxT6-symbols, Payload_StandardPackages:STM32L4x6RxT6, symbol ARM-Board-rescue:STM32L4x6RxT6-symbols-Payload_Microcontrollers
- removed U2: SRAM_23LC1024T-I_ST-ARMlib, Housings_SSOP:TSSOP-8_4.4x3mm_Pitch0.65mm, symbol ARM-Board-rescue:SRAM_23LC1024T-I_ST-ARMlib-Payload_Microcontrollers
- removed VR1: LD39200PU33R, Housings_DFN_QFN:DFN-6-1EP_3x3mm_Pitch0.95mm, symbol ARM-Board-rescue:LD39200PU33R-Payload_Regulators
- removed Y1: Crystal_GND23, Payload_XTAL:MC-306, symbol Device:Crystal_GND23
- added C?: 0.1uF, symbol Device:C
- added C? (x2): 47pF, symbol Device:C
- added C?: .01uF, symbol Device:C
- added D?: D_TVS, symbol Device:D_TVS
- added J?: USB_A, symbol Connector:USB_A
- added R? (x2): 27, symbol Device:R
- added U?: FT231XS, Package_SO:SSOP-20_3.9x8.7mm_P0.635mm, symbol Interface_USB:FT231XS
- R5: value 120 -> DNP
Connections:
- net labels added: +3V3, +5V, 3V3_BUS, 5_BUS, 5_CANHW, 5_USB
- net labels removed: CANRX, CANTX, D+, D-, JTCK_SWCLK, JTDI, JTDO_SWO, JTMS_SWDIO, JTRST, MISO1, MISO2, MISO3, MOSI1, MOSI2, MOSI3, PH3-BOOT0, SCK1, SCK2, SCK3, SCL, SDA, UART_RX, UART_TX, UART_~CTS, UART_~RTS, VBUS, VDD33, VDD33_IN, VDD33_USB, VDD5_IN, VTREF, ~CAN_EN, ~CS1, ~CS1_2, ~CS2, ~CS2_2, ~CS3, ~HOLD3, ~RST
- wire segments 230 -> 137
Other:
- note added: "CAN LOGIC"
- note added: "CUBESAT BUS CONNECTOR"
- note added: "POWER MANAGEMENT"
- note added: "USB POWER + PROGRAMMING"
- note removed: "RAM"
- note removed: "USB to Basic UART"

Commit message: updated ARM board schematic with updates specified on slack
Parts:
- removed J5, J6: SD_WM6698CT-ND-ARMlib-ARM-Board-rescue, Payload_Connectors:MICROSD_WM6698CT-ND, symbol ARM-Board-rescue:SD_WM6698CT-ND-ARMlib-ARM-Board-rescue-Payload_Connectors
- removed J?: USB_A, symbol Connector:USB_A
- removed R1, R8: DNP, Resistors_SMD:R_0603, symbol Device:R
- added C? (x2): 0.1uF, symbol Device:C
- added C?: 4.7uF, symbol Device:C
- added J? (x2): SD_Card, symbol Connector:SD_Card
- added J?: USB_B_Micro, symbol Connector:USB_B_Micro
- added R?: DNP, Resistors_SMD:R_0603, symbol Device:R
Connections:
- wire segments 137 -> 150
- no-connect marks 0 -> 7
Other:
- note added: "CANHW CURRENT SENSING"
- note added: "ONLY POWERED WHEN USB CONNECTED"

Commit message: Jumpers for ARM board added
Parts:
- added JP? (x18): Jumper, symbol Device:Jumper
- R?: value DNP -> R
Connections:
- wire segments 150 -> 163

Commit message: addressed review comments from Alex
Parts:
- gave numbers to parts that had none: 33

Commit message: ARM board: Added polyfuse Added lines for radio interrupt
Parts:
- added JP21, JP22: Jumper, Jumper:SolderJumper-2_P1.3mm_Open_RoundedPad1.0x1.5mm, symbol Device:Jumper
- C1, C2, C3, C4, C5, C6, C7: footprint (none) -> Capacitors_SMD:C_0603_HandSoldering
- D1: footprint (none) -> Diodes_SMD:D_0603
- J2: renamed from J1; footprint (none) -> Payload_Connectors:10118194-0001LF
- J4: renamed from J2; footprint (none) -> Payload_Connectors:SD_Card_Receptacle
- J5: renamed from J3; footprint (none) -> Payload_Connectors:SD_Card_Receptacle
- JP1, JP10, JP11, JP12, JP13, JP14, JP15, JP16, JP17, JP18, JP2, JP3, JP4, JP5, JP6, JP7, JP8, JP9: footprint (none) -> Jumper:SolderJumper-2_P1.3mm_Open_RoundedPad1.0x1.5mm
- R1: renamed from R5; footprint Resistors_SMD:R_0603 -> Resistors_SMD:R_0603_HandSoldering
- R2: renamed from R1; footprint (none) -> Resistors_SMD:R_0603_HandSoldering
- R3: renamed from R2; footprint (none) -> Resistors_SMD:R_0603_HandSoldering
- R4: renamed from R3; footprint Resistors_SMD:R_0603 -> Resistors_SMD:R_0603_HandSoldering
- renumbered J7 to J1, J4 to J3, U3 to U1, U1 to U2
Connections:
- net labels added: D+, D-, D2+, D2-
- wire segments 163 -> 167
