File: Hardware/Flight/ARM Board/CAN-SENSE.sch (KiCad schematic (older format))
At the start: 4 parts

Commit message: addressed review comments from Alex
Parts:
- gave numbers to parts that had none: 4
Changed lines of the file:
@@
 VIN
 $Comp
-L canhw:INA180 U?
+L canhw:INA180 U5
 U 1 1 5D71919D
 P 7000 3100
-F 0 "U?" H 6950 2628 50  0000 C CNN
+F 0 "U5" H 6950 2628 50  0000 C CNN
 F 1 "INA180" H 6950 2537 50  0000 C CNN
 F 2 "" H 7000 3100 50  0001 C CNN
@@
 $EndComp
 $Comp
-L Device:R R?
+L Device:R R9
 U 1 1 5D719238
 P 6300 2550
-F 0 "R?" V 6093 2550 50  0000 C CNN
+F 0 "R9" V 6093 2550 50  0000 C CNN
 F 1 "62m" V 6184 2550 50  0000 C CNN
 F 2 "" V 6230 2550 50  0001 C CNN
@@
 	6150 3200 6500 3200
 $Comp
-L power:GND #PWR?
+L power:GND #PWR042
 U 1 1 5D719378
 P 6150 3350
-F 0 "#PWR?" H 6150 3100 50  0001 C CNN
+F 0 "#PWR042" H 6150 3100 50  0001 C CNN
 F 1 "GND" H 6155 3177 50  0000 C CNN
 F 2 "" H 6150 3350 50  0001 C CNN
@@
 3v3
 $Comp
-L Device:C C?
+L Device:C C21
 U 1 1 5D71989D
 P 7150 2600
-F 0 "C?" V 6898 2600 50  0000 C CNN
+F 0 "C21" V 6898 2600 50  0000 C CNN
 F 1 "C" V 6989 2600 50  0000 C CNN
 F 2 "" H 7188 2450 50  0001 C CNN
@@
 Connection ~ 6850 2600
 $Comp
-L power:GND #PWR?
+L power:GND #PWR043
 U 1 1 5D7199D4
 P 7400 2700
-F 0 "#PWR?" H 7400 2450 50  0001 C CNN
+F 0 "#PWR043" H 7400 2450 50  0001 C CNN
 F 1 "GND" H 7405 2527 50  0000 C CNN
 F 2 "" H 7400 2700 50  0001 C CNN
@@
 Connection ~ 6450 2550
 $Comp
-L Device:D_TVS D?
+L Device:D_TVS D6
 U 1 1 5D7278BC
 P 5800 2700
-F 0 "D?" V 5754 2779 50  0000 L CNN
+F 0 "D6" V 5754 2779 50  0000 L CNN
 F 1 "D_TVS" V 5845 2779 50  0000 L CNN
 F 2 "" H 5800 2700 50  0001 C CNN
@@
 Connection ~ 5800 2550
 $Comp
-L power:GND #PWR?
+L power:GND #PWR041
 U 1 1 5D727A86
 P 5800 2850
-F 0 "#PWR?" H 5800 2600 50  0001 C CNN
+F 0 "#PWR041" H 5800 2600 50  0001 C CNN
 F 1 "GND" H 5805 2677 50  0000 C CNN
 F 2 "" H 5800 2850 50  0001 C CNN

Commit message: ARM board: Added polyfuse Added lines for radio interrupt
Parts:
- added F1: Polyfuse, Fuses:Fuse_1206_3216Metric_Pad1.42x1.75mm_HandSolder, symbol Device:Polyfuse
- C21: value C -> .1uF; footprint (none) -> Capacitors_SMD:C_0603_HandSoldering
- D6: footprint (none) -> Diodes_SMD:D_0603
- R9: footprint (none) -> Resistors_SMD:R_0603_HandSoldering
- U5: footprint (none) -> TO_SOT_Packages_SMD:SOT-23-5_HandSoldering
Changed lines of the file:
@@
 F 0 "U5" H 6950 2628 50  0000 C CNN
 F 1 "INA180" H 6950 2537 50  0000 C CNN
-F 2 "" H 7000 3100 50  0001 C CNN
+F 2 "TO_SOT_Packages_SMD:SOT-23-5_HandSoldering" H 7000 3100 50  0001 C CNN
 F 3 "http://www.ti.com/lit/ds/symlink/ina180.pdf" H 7000 3100 50  0001 C CNN
 	1    7000 3100
@@
 F 0 "R9" V 6093 2550 50  0000 C CNN
 F 1 "62m" V 6184 2550 50  0000 C CNN
-F 2 "" V 6230 2550 50  0001 C CNN
+F 2 "Resistors_SMD:R_0603_HandSoldering" V 6230 2550 50  0001 C CNN
 F 3 "~" H 6300 2550 50  0001 C CNN
 	1    6300 2550
@@
 	6150 3200 6500 3200
 $Comp
-L power:GND #PWR042
+L power:GND #PWR045
 U 1 1 5D719378
 P 6150 3350
-F 0 "#PWR042" H 6150 3100 50  0001 C CNN
+F 0 "#PWR045" H 6150 3100 50  0001 C CNN
 F 1 "GND" H 6155 3177 50  0000 C CNN
 F 2 "" H 6150 3350 50  0001 C CNN
@@
 P 7150 2600
 F 0 "C21" V 6898 2600 50  0000 C CNN
-F 1 "C" V 6989 2600 50  0000 C CNN
-F 2 "" H 7188 2450 50  0001 C CNN
+F 1 ".1uF" V 6989 2600 50  0000 C CNN
+F 2 "Capacitors_SMD:C_0603_HandSoldering" H 7188 2450 50  0001 C CNN
 F 3 "~" H 7150 2600 50  0001 C CNN
 	1    7150 2600
@@
 Connection ~ 6850 2600
 $Comp
-L power:GND #PWR043
+L power:GND #PWR046
 U 1 1 5D7199D4
 P 7400 2700
-F 0 "#PWR043" H 7400 2450 50  0001 C CNN
+F 0 "#PWR046" H 7400 2450 50  0001 C CNN
 F 1 "GND" H 7405 2527 50  0000 C CNN
 F 2 "" H 7400 2700 50  0001 C CNN
@@
 F 0 "D6" V 5754 2779 50  0000 L CNN
 F 1 "D_TVS" V 5845 2779 50  0000 L CNN
-F 2 "" H 5800 2700 50  0001 C CNN
+F 2 "Diodes_SMD:D_0603" H 5800 2700 50  0001 C CNN
 F 3 "~" H 5800 2700 50  0001 C CNN
 	1    5800 2700
@@
 Wire Wire Line
 	5800 2550 5700 2550
-Connection ~ 5800 2550
 $Comp
-L power:GND #PWR041
+L power:GND #PWR044
 U 1 1 5D727A86
 P 5800 2850
-F 0 "#PWR041" H 5800 2600 50  0001 C CNN
+F 0 "#PWR044" H 5800 2600 50  0001 C CNN
 F 1 "GND" H 5805 2677 50  0000 C CNN
 F 2 "" H 5800 2850 50  0001 C CNN
@@
 	1    0    0    -1
 $EndComp
+$Comp
+L Device:Polyfuse F1
+U 1 1 5C9521C8
+P 6000 2550
+F 0 "F1" V 5775 2550 50  0000 C CNN
+F 1 "Polyfuse" V 5866 2550 50  0000 C CNN
+F 2 "Fuses:Fuse_1206_3216Metric_Pad1.42x1.75mm_HandSolder" H 6050 2350 50  0001 L CNN
+F 3 "~" H 6000 2550 50  0001 C CNN
+	1    6000 2550
+	0    1    1    0
+$EndComp
+Connection ~ 6150 2550
 Wire Wire Line
-	5800 2550 6150 2550
-Connection ~ 6150 2550
+	5850 2550 5800 2550
+Connection ~ 5800 2550
 $EndSCHEMATC
