File: Hardware/Flight/ARM Board/CoreLogic.sch (KiCad schematic (older format))
At the start: 20 parts

Commit message: updated ARM board schematic with updates specified on slack
Parts:
- removed R?: 10K, Resistors_SMD:R_0603, symbol Device:R
- removed R? (x2): DNP, Resistors_SMD:R_0603, symbol Device:R
- removed Y?: Crystal_GND23, Payload_XTAL:MC-306, symbol Device:Crystal_GND23
- added C?: 0.1uF, Capacitors_SMD:C_0603, symbol Device:C
- added C?: 4.7uF, Capacitors_SMD:C_0603, symbol Device:C
- added C?: 1uF, Capacitors_SMD:C_0603, symbol Device:C
- added Y?: Crystal, symbol Device:Crystal
Connections:
- net labels added: CARD_DETECT_1, CARD_DETECT_2, CURR_AMP
- wire segments 81 -> 78

Commit message: Jumpers for ARM board added
Connections:
- net labels added: ~(JTRST|RST)
- wire segments 78 -> 77
Changed lines of the file:
@@
 Wire Wire Line
 	6550 1650 6600 1650
-Text Label 1350 5000 0    50   ~ 0
-JTRST|~RST
+Text Label 1200 5000 0    50   ~ 0
+~(JTRST|RST)
 Text Label 1200 5100 0    50   ~ 0
 PH3-BOOT0
@@
 Text HLabel 6500 2800 1    50   Input ~ 0
 3v3
-Wire Wire Line
-	1200 5000 1350 5000
 Text Label 6250 1650 2    50   ~ 0
-JTRST|~RST
+~(JTRST|RST)
 Text Label 9400 2250 0    50   ~ 0
 JTRST|~RST

Commit message: addressed review comments from Alex
Parts:
- gave numbers to parts that had none: 19

Commit message: ARM board: Added polyfuse Added lines for radio interrupt
Parts:
- C10, C11, C12, C13, C14, C15, C16, C18, C19, C20: footprint Capacitors_SMD:C_0603 -> Capacitors_SMD:C_0603_HandSoldering
- C17: footprint Capacitors_SMD:C_0805 -> Capacitors_SMD:C_0603_HandSoldering
- R6, R7, R8: footprint Resistors_SMD:R_0603 -> Resistors_SMD:R_0603_HandSoldering
- Y1: footprint (none) -> Crystals:Crystal_HC49-U_Vertical
- renumbered J5 to J6, U2 to U3
Connections:
- net labels added: RADIO_INT_1, RADIO_INT_2
Changed lines of the file:
@@
 F 0 "C12" H 1815 2746 50  0000 L CNN
 F 1 "100nF" H 1815 2655 50  0000 L CNN
-F 2 "Capacitors_SMD:C_0603" H 1738 2550 50  0001 C CNN
+F 2 "Capacitors_SMD:C_0603_HandSoldering" H 1738 2550 50  0001 C CNN
 F 3 "~" H 1700 2700 50  0001 C CNN
 	1    1700 2700
@@
 F 0 "C13" H 2265 2746 50  0000 L CNN
 F 1 "100nF" H 2265 2655 50  0000 L CNN
-F 2 "Capacitors_SMD:C_0603" H 2188 2550 50  0001 C CNN
+F 2 "Capacitors_SMD:C_0603_HandSoldering" H 2188 2550 50  0001 C CNN
 F 3 "~" H 2150 2700 50  0001 C CNN
 	1    2150 2700
@@
 F 0 "C11" H 1365 2746 50  0000 L CNN
 F 1 "100nF" H 1365 2655 50  0000 L CNN
-F 2 "Capacitors_SMD:C_0603" H 1288 2550 50  0001 C CNN
+F 2 "Capacitors_SMD:C_0603_HandSoldering" H 1288 2550 50  0001 C CNN
 F 3 "~" H 1250 2700 50  0001 C CNN
 	1    1250 2700
@@
 F 0 "C15" H 5315 2296 50  0000 L CNN
 F 1 "1uF" H 5315 2205 50  0000 L CNN
-F 2 "Capacitors_SMD:C_0603" H 5238 2100 50  0001 C CNN
+F 2 "Capacitors_SMD:C_0603_HandSoldering" H 5238 2100 50  0001 C CNN
 F 3 "~" H 5200 2250 50  0001 C CNN
 	1    5200 2250
@@
 F 0 "C16" H 5665 2296 50  0000 L CNN
 F 1 "10uF" H 5665 2205 50  0000 L CNN
-F 2 "Capacitors_SMD:C_0603" H 5588 2100 50  0001 C CNN
+F 2 "Capacitors_SMD:C_0603_HandSoldering" H 5588 2100 50  0001 C CNN
 F 3 "~" H 5550 2250 50  0001 C CNN
 	1    5550 2250
@@
 P 1250 2850
 AR Path="/5D19DB50" Ref="#PWR?"  Part="1"
-AR Path="/5D19D8A9/5D19DB50" Ref="#PWR029"  Part="1"
-F 0 "#PWR029" H 1250 2600 50  0001 C CNN
+AR Path="/5D19D8A9/5D19DB50" Ref="#PWR032"  Part="1"
+F 0 "#PWR032" H 1250 2600 50  0001 C CNN
 F 1 "GND" H 1255 2677 50  0000 C CNN
 F 2 "" H 1250 2850 50  0001 C CNN
@@
 P 1700 2850
 AR Path="/5D19DB56" Ref="#PWR?"  Part="1"
-AR Path="/5D19D8A9/5D19DB56" Ref="#PWR030"  Part="1"
-F 0 "#PWR030" H 1700 2600 50  0001 C CNN
+AR Path="/5D19D8A9/5D19DB56" Ref="#PWR033"  Part="1"
+F 0 "#PWR033" H 1700 2600 50  0001 C CNN
 F 1 "GND" H 1705 2677 50  0000 C CNN
 F 2 "" H 1700 2850 50  0001 C CNN
@@
 P 2150 2850
 AR Path="/5D19DB5C" Ref="#PWR?"  Part="1"
-AR Path="/5D19D8A9/5D19DB5C" Ref="#PWR032"  Part="1"
-F 0 "#PWR032" H 2150 2600 50  0001 C CNN
+AR Path="/5D19D8A9/5D19DB5C" Ref="#PWR035"  Part="1"
+F 0 "#PWR035" H 2150 2600 50  0001 C CNN
 F 1 "GND" H 2155 2677 50  0000 C CNN
 F 2 "" H 2150 2850 50  0001 C CNN
@@
 P 5200 2400
 AR Path="/5D19DB62" Ref="#PWR?"  Part="1"
-AR Path="/5D19D8A9/5D19DB62" Ref="#PWR036"  Part="1"
-F 0 "#PWR036" H 5200 2150 50  0001 C CNN
+AR Path="/5D19D8A9/5D19DB62" Ref="#PWR039"  Part="1"
+F 0 "#PWR039" H 5200 2150 50  0001 C CNN
 F 1 "GND" H 5205 2227 50  0000 C CNN
 F 2 "" H 5200 2400 50  0001 C CNN
@@
 P 5550 2400
 AR Path="/5D19DB68" Ref="#PWR?"  Part="1"
-AR Path="/5D19D8A9/5D19DB68" Ref="#PWR037"  Part="1"
-F 0 "#PWR037" H 5550 2150 50  0001 C CNN
+AR Path="/5D19D8A9/5D19DB68" Ref="#PWR040"  Part="1"
+F 0 "#PWR040" H 5550 2150 50  0001 C CNN
 F 1 "GND" H 5555 2227 50  0000 C CNN
 F 2 "" H 5550 2400 50  0001 C CNN
@@
 F 0 "C17" H 6065 2296 50  0000 L CNN
 F 1 "100uF" H 6065 2205 50  0000 L CNN
-F 2 "Capacitors_SMD:C_0805" H 5988 2100 50  0001 C CNN
+F 2 "Capacitors_SMD:C_0603_HandSoldering" H 5988 2100 50  0001 C CNN
 F 3 "~" H 5950 2250 50  0001 C CNN
 	1    5950 2250
@@
 P 5950 2400
 AR Path="/5D19DB83" Ref="#PWR?"  Part="1"
-AR Path="/5D19D8A9/5D19DB83" Ref="#PWR038"  Part="1"
-F 0 "#PWR038" H 5950 2150 50  0001 C CNN
+AR Path="/5D19D8A9/5D19DB83" Ref="#PWR041"  Part="1"
+F 0 "#PWR041" H 5950 2150 50  0001 C CNN
 F 1 "GND" H 5955 2227 50  0000 C CNN
 F 2 "" H 5950 2400 50  0001 C CNN
@@
 P 4650 2950
 AR Path="/5D19DB89" Ref="#PWR?"  Part="1"
-AR Path="/5D19D8A9/5D19DB89" Ref="#PWR034"  Part="1"
-F 0 "#PWR034" H 4650 2700 50  0001 C CNN
+AR Path="/5D19D8A9/5D19DB89" Ref="#PWR037"  Part="1"
+F 0 "#PWR037" H 4650 2700 50  0001 C CNN
 F 1 "GND" H 4655 2777 50  0000 C CNN
 F 2 "" H 4650 2950 50  0001 C CNN
@@
 F 0 "R7" V 6200 1600 50  0000 L CNN
 F 1 "0" V 6300 1600 50  0000 L CNN
-F 2 "Resistors_SMD:R_0603" V 6330 1650 50  0001 C CNN
+F 2 "Resistors_SMD:R_0603_HandSoldering" V 6330 1650 50  0001 C CNN
 F 3 "~" H 6400 1650 50  0001 C CNN
 	1    6400 1650
@@
 P 7450 1650
 AR Path="/5D19DC14" Ref="U?"  Part="1"
-AR Path="/5D19D8A9/5D19DC14" Ref="U2"  Part="1"
-F 0 "U2" H 8425 2137 60  0000 C CNN
+AR Path="/5D19D8A9/5D19DC14" Ref="U3"  Part="1"
+F 0 "U3" H 8425 2137 60  0000 C CNN
 F 1 "STM32L4x6RxT6-symbols" H 8425 2031 60  0000 C CNN
 F 2 "Payload_StandardPackages:STM32L4x6RxT6" H 8300 2000 60  0001 C CNN
@@
 P 2700 2150
 AR Path="/5D19DC1B" Ref="U?"  Part="2"
-AR Path="/5D19D8A9/5D19DC1B" Ref="U2"  Part="2"
-F 0 "U2" H 3600 2537 60  0000 C CNN
+AR Path="/5D19D8A9/5D19DC1B" Ref="U3"  Part="2"
+F 0 "U3" H 3600 2537 60  0000 C CNN
 F 1 "STM32L4x6RxT6-symbols" H 3600 2431 60  0000 C CNN
 F 2 "Payload_StandardPackages:STM32L4x6RxT6" H 3550 2500 60  0001 C CNN
@@
 P 3800 5950
 AR Path="/5D1A8E63" Ref="#PWR?"  Part="1"
-AR Path="/5D19D8A9/5D1A8E63" Ref="#PWR033"  Part="1"
-F 0 "#PWR033" H 3800 5700 50  0001 C CNN
+AR Path="/5D19D8A9/5D1A8E63" Ref="#PWR036"  Part="1"
+F 0 "#PWR036" H 3800 5700 50  0001 C CNN
 F 1 "GND" H 3805 5777 50  0000 C CNN
 F 2 "" H 3800 5950 50  0001 C CNN
@@
 P 1750 6000
 AR Path="/5D1BC4B3" Ref="#PWR?"  Part="1"
-AR Path="/5D19D8A9/5D1BC4B3" Ref="#PWR031"  Part="1"
-F 0 "#PWR031" H 1750 5750 50  0001 C CNN
+AR Path="/5D19D8A9/5D1BC4B3" Ref="#PWR034"  Part="1"
+F 0 "#PWR034" H 1750 5750 50  0001 C CNN
 F 1 "GND" H 1755 5827 50  0000 C CNN
 F 2 "" H 1750 6000 50  0001 C CNN
@@
 P 1000 5500
 AR Path="/5D1BC4BD" Ref="J?"  Part="1"
-AR Path="/5D19D8A9/5D1BC4BD" Ref="J5"  Part="1"
-F 0 "J5" H 920 4775 50  0000 C CNN
+AR Path="/5D19D8A9/5D1BC4BD" Ref="J6"  Part="1"
+F 0 "J6" H 920 4775 50  0000 C CNN
 F 1 "Conn_01x10" H 920 4866 50  0000 C CNN
 F 2 "Pin_Headers:Pin_Header_Straight_2x05_Pitch2.54mm" H 1000 5500 50  0001 C CNN
@@
 F 0 "C20" H 10442 5646 50  0000 L CNN
 F 1 "C_Small" H 10442 5555 50  0000 L CNN
-F 2 "Capacitors_SMD:C_0603" H 10350 5600 50  0001 C CNN
+F 2 "Capacitors_SMD:C_0603_HandSoldering" H 10350 5600 50  0001 C CNN
 F 3 "~" H 10350 5600 50  0001 C CNN
 	1    10350 5600
@@
 F 0 "C19" H 9450 5600 50  0000 L CNN
 F 1 "C_Small" H 9250 5500 50  0000 L CNN
-F 2 "Capacitors_SMD:C_0603" H 9650 5550 50  0001 C CNN
+F 2 "Capacitors_SMD:C_0603_HandSoldering" H 9650 5550 50  0001 C CNN
 F 3 "~" H 9650 5550 50  0001 C CNN
 	1    9650 5550
@@
 P 10000 5900
 AR Path="/5D1F8EC7" Ref="#PWR?"  Part="1"
-AR Path="/5D19D8A9/5D1F8EC7" Ref="#PWR040"  Part="1"
-F 0 "#PWR040" H 10000 5650 50  0001 C CNN
+AR Path="/5D19D8A9/5D1F8EC7" Ref="#PWR043"  Part="1"
+F 0 "#PWR043" H 10000 5650 50  0001 C CNN
 F 1 "GND" H 10005 5727 50  0000 C CNN
 F 2 "" H 10000 5900 50  0001 C CNN
@@
 F 0 "R8" H 6720 3246 50  0000 L CNN
 F 1 "4.7K" H 6720 3155 50  0000 L CNN
-F 2 "Resistors_SMD:R_0603" V 6580 3200 50  0001 C CNN
+F 2 "Resistors_SMD:R_0603_HandSoldering" V 6580 3200 50  0001 C CNN
 F 3 "~" H 6650 3200 50  0001 C CNN
 	1    6650 3200
@@
 F 0 "R6" H 6420 3246 50  0000 L CNN
 F 1 "4.7K" H 6420 3155 50  0000 L CNN
-F 2 "Resistors_SMD:R_0603" V 6280 3200 50  0001 C CNN
+F 2 "Resistors_SMD:R_0603_HandSoldering" V 6280 3200 50  0001 C CNN
 F 3 "~" H 6350 3200 50  0001 C CNN
 	1    6350 3200
@@
 F 0 "Y1" H 10000 5568 50  0000 C CNN
 F 1 "Crystal" H 10000 5477 50  0000 C CNN
-F 2 "" H 10000 5300 50  0001 C CNN
+F 2 "Crystals:Crystal_HC49-U_Vertical" H 10000 5300 50  0001 C CNN
 F 3 "~" H 10000 5300 50  0001 C CNN
 	1    10000 5300
@@
 F 0 "C18" H 6715 1846 50  0000 L CNN
 F 1 "0.1uF" H 6715 1755 50  0000 L CNN
-F 2 "Capacitors_SMD:C_0603" H 6638 1650 50  0001 C CNN
+F 2 "Capacitors_SMD:C_0603_HandSoldering" H 6638 1650 50  0001 C CNN
 F 3 "~" H 6600 1800 50  0001 C CNN
 	1    6600 1800
@@
 P 6600 1950
 AR Path="/5D56B111" Ref="#PWR?"  Part="1"
-AR Path="/5D19D8A9/5D56B111" Ref="#PWR039"  Part="1"
-F 0 "#PWR039" H 6600 1700 50  0001 C CNN
+AR Path="/5D19D8A9/5D56B111" Ref="#PWR042"  Part="1"
+F 0 "#PWR042" H 6600 1700 50  0001 C CNN
 F 1 "GND" H 6605 1777 50  0000 C CNN
 F 2 "" H 6600 1950 50  0001 C CNN
@@
 F 0 "C10" H 915 2746 50  0000 L CNN
 F 1 "4.7uF" H 915 2655 50  0000 L CNN
-F 2 "Capacitors_SMD:C_0603" H 838 2550 50  0001 C CNN
+F 2 "Capacitors_SMD:C_0603_HandSoldering" H 838 2550 50  0001 C CNN
 F 3 "~" H 800 2700 50  0001 C CNN
 	1    800  2700
@@
 P 800 2850
 AR Path="/5D57213C" Ref="#PWR?"  Part="1"
-AR Path="/5D19D8A9/5D57213C" Ref="#PWR028"  Part="1"
-F 0 "#PWR028" H 800 2600 50  0001 C CNN
+AR Path="/5D19D8A9/5D57213C" Ref="#PWR031"  Part="1"
+F 0 "#PWR031" H 800 2600 50  0001 C CNN
 F 1 "GND" H 805 2677 50  0000 C CNN
 F 2 "" H 800 2850 50  0001 C CNN
@@
 F 0 "C14" H 4965 2296 50  0000 L CNN
 F 1 "1uF" H 4965 2205 50  0000 L CNN
-F 2 "Capacitors_SMD:C_0603" H 4888 2100 50  0001 C CNN
+F 2 "Capacitors_SMD:C_0603_HandSoldering" H 4888 2100 50  0001 C CNN
 F 3 "~" H 4850 2250 50  0001 C CNN
 	1    4850 2250
@@
 P 4850 2400
 AR Path="/5D5794A0" Ref="#PWR?"  Part="1"
-AR Path="/5D19D8A9/5D5794A0" Ref="#PWR035"  Part="1"
-F 0 "#PWR035" H 4850 2150 50  0001 C CNN
+AR Path="/5D19D8A9/5D5794A0" Ref="#PWR038"  Part="1"
+F 0 "#PWR038" H 4850 2150 50  0001 C CNN
 F 1 "GND" H 4855 2227 50  0000 C CNN
 F 2 "" H 4850 2400 50  0001 C CNN
@@
 Text HLabel 7450 3650 0    50   Input ~ 0
 CURR_AMP
+Text HLabel 7450 3750 0    50   Input ~ 0
+RADIO_INT_1
+Text HLabel 7450 3950 0    50   Input ~ 0
+RADIO_INT_2
 $EndSCHEMATC

Commit message: ARM review comments
Parts:
- added D7, D8, D9: LED, LEDs:LED_0603_HandSoldering, symbol Device:LED
- added R10, R11, R12: 70, Resistors_SMD:R_0603_HandSoldering, symbol Device:R
Connections:
- net labels added: +3V3
- net labels removed: 3v3, JTRST|~RST
- wire segments 77 -> 87
Other:
- note added: "2v drop, 20mA max per pin"
Changed lines of the file:
@@
 	1    0    0    -1
 $EndComp
-Text HLabel 750  2550 0    50   Input ~ 0
-3v3
 Wire Wire Line
 	2150 2550 2500 2550
@@
 L power:GND #PWR?
 U 1 1 5D1BC4B3
-P 1750 6000
+P 1750 6200
 AR Path="/5D1BC4B3" Ref="#PWR?"  Part="1"
 AR Path="/5D19D8A9/5D1BC4B3" Ref="#PWR034"  Part="1"
-F 0 "#PWR034" H 1750 5750 50  0001 C CNN
-F 1 "GND" H 1755 5827 50  0000 C CNN
-F 2 "" H 1750 6000 50  0001 C CNN
-F 3 "" H 1750 6000 50  0001 C CNN
-	1    1750 6000
+F 0 "#PWR034" H 1750 5950 50  0001 C CNN
+F 1 "GND" H 1755 6027 50  0000 C CNN
+F 2 "" H 1750 6200 50  0001 C CNN
+F 3 "" H 1750 6200 50  0001 C CNN
+	1    1750 6200
 	1    0    0    -1
 $EndComp
@@
 	1200 5500 1750 5500
 Connection ~ 1750 5700
-Text Notes 850  6400 0    50   ~ 0
+Text Notes 850  6500 0    50   ~ 0
 STM PROGRAMMING HEADER
 Wire Wire Line
@@
 Text Label 7350 3050 2    50   ~ 0
 JTMS_SWDIO
-Text HLabel 1200 5900 2    50   Input ~ 0
-3v3
-Wire Wire Line
-	1750 5700 1750 6000
-Text HLabel 1200 5300 2    50   Input ~ 0
-3v3
+Wire Wire Line
+	1750 5700 1750 6200
 Text Label 3850 5550 2    50   ~ 0
 ~CS3
@@
 	6650 3550 6200 3550
 Connection ~ 6650 3550
-Text HLabel 6500 2800 1    50   Input ~ 0
-3v3
 Text Label 6250 1650 2    50   ~ 0
 ~(JTRST|RST)
 Text Label 9400 2250 0    50   ~ 0
-JTRST|~RST
+~(JTRST|RST)
 $Comp
 L Device:Crystal Y1
@@
 	1    0    0    -1
 $EndComp
-Wire Wire Line
-	750  2550 800  2550
 $Comp
 L power:GND #PWR?
@@
 Text HLabel 9400 1950 2    50   Input ~ 0
 CARD_DETECT_2
-Text HLabel 5050 5400 1    50   Input ~ 0
-3v3
 Wire Wire Line
 	5050 5400 5050 5550
@@
 Text HLabel 7450 3950 0    50   Input ~ 0
 RADIO_INT_2
+$Comp
+L Device:LED D7
+U 1 1 5C9DEAAB
+P 10200 2050
+F 0 "D7" V 10238 1933 50  0000 R CNN
+F 1 "LED" V 10147 1933 50  0000 R CNN
+F 2 "LEDs:LED_0603_HandSoldering" H 10200 2050 50  0001 C CNN
+F 3 "~" H 10200 2050 50  0001 C CNN
+	1    10200 2050
+	0    -1   -1   0
+$EndComp
+$Comp
+L Device:LED D8
+U 1 1 5C9DEB45
+P 10550 2050
+F 0 "D8" V 10588 1933 50  0000 R CNN
+F 1 "LED" V 10497 1933 50  0000 R CNN
+F 2 "LEDs:LED_0603_HandSoldering" H 10550 2050 50  0001 C CNN
+F 3 "~" H 10550 2050 50  0001 C CNN
+	1    10550 2050
+	0    -1   -1   0
+$EndComp
+$Comp
+L Device:LED D9
+U 1 1 5C9DEB8B
+P 10900 2050
+F 0 "D9" V 10938 1933 50  0000 R CNN
+F 1 "LED" V 10847 1933 50  0000 R CNN
+F 2 "LEDs:LED_0603_HandSoldering" H 10900 2050 50  0001 C CNN
+F 3 "~" H 10900 2050 50  0001 C CNN
+	1    10900 2050
+	0    -1   -1   0
+$EndComp
+$Comp
+L Device:R R10
+U 1 1 5C9DEBE6
+P 10200 2350
+F 0 "R10" H 10270 2396 50  0000 L CNN
+F 1 "70" H 10270 2305 50  0000 L CNN
+F 2 "Resistors_SMD:R_0603_HandSoldering" V 10130 2350 50  0001 C CNN
+F 3 "~" H 10200 2350 50  0001 C CNN
+	1    10200 2350
+	1    0    0    -1
+$EndComp
+$Comp
+L Device:R R11
+U 1 1 5C9DF0E8
+P 10550 2350
+F 0 "R11" H 10620 2396 50  0000 L CNN
+F 1 "70" H 10620 2305 50  0000 L CNN
+F 2 "Resistors_SMD:R_0603_HandSoldering" V 10480 2350 50  0001 C CNN
+F 3 "~" H 10550 2350 50  0001 C CNN
+	1    10550 2350
+	1    0    0    -1
+$EndComp
+$Comp
+L Device:R R12
+U 1 1 5C9DF136
+P 10900 2350
+F 0 "R12" H 10970 2396 50  0000 L CNN
+F 1 "70" H 10970 2305 50  0000 L CNN
+F 2 "Resistors_SMD:R_0603_HandSoldering" V 10830 2350 50  0001 C CNN
+F 3 "~" H 10900 2350 50  0001 C CNN
+	1    10900 2350
+	1    0    0    -1
+$EndComp
+Wire Wire Line
+	10200 2500 10200 2550
+Wire Wire Line
+	10200 2550 9400 2550
+Wire Wire Line
+	9400 2650 10550 2650
+Wire Wire Line
+	10550 2650 10550 2500
+Wire Wire Line
+	10900 2500 10900 2750
+Wire Wire Line
+	10900 2750 9400 2750
+$Comp
+L power:+3V3 #PWR0101
+U 1 1 5C9E455B
+P 10200 1900
+F 0 "#PWR0101" H 10200 1750 50  0001 C CNN
+F 1 "+3V3" H 10215 2073 50  0000 C CNN
+F 2 "" H 10200 1900 50  0001 C CNN
+F 3 "" H 10200 1900 50  0001 C CNN
+	1    10200 1900
+	1    0    0    -1
+$EndComp
+$Comp
+L power:+3V3 #PWR0102
+U 1 1 5C9E4623
+P 10550 1900
+F 0 "#PWR0102" H 10550 1750 50  0001 C CNN
+F 1 "+3V3" H 10565 2073 50  0000 C CNN
+F 2 "" H 10550 1900 50  0001 C CNN
+F 3 "" H 10550 1900 50  0001 C CNN
+	1    10550 1900
+	1    0    0    -1
+$EndComp
+$Comp
+L power:+3V3 #PWR0103
+U 1 1 5C9E4662
+P 10900 1900
+F 0 "#PWR0103" H 10900 1750 50  0001 C CNN
+F 1 "+3V3" H 10915 2073 50  0000 C CNN
+F 2 "" H 10900 1900 50  0001 C CNN
+F 3 "" H 10900 1900 50  0001 C CNN
+	1    10900 1900
+	1    0    0    -1
+$EndComp
+$Comp
+L power:+3V3 #PWR0104
+U 1 1 5C9E46A1
+P 6500 2800
+F 0 "#PWR0104" H 6500 2650 50  0001 C CNN
+F 1 "+3V3" H 6515 2973 50  0000 C CNN
+F 2 "" H 6500 2800 50  0001 C CNN
+F 3 "" H 6500 2800 50  0001 C CNN
+	1    6500 2800
+	1    0    0    -1
+$EndComp
+$Comp
+L power:+3V3 #PWR0105
+U 1 1 5C9E4A53
+P 800 2350
+F 0 "#PWR0105" H 800 2200 50  0001 C CNN
+F 1 "+3V3" H 815 2523 50  0000 C CNN
+F 2 "" H 800 2350 50  0001 C CNN
+F 3 "" H 800 2350 50  0001 C CNN
+	1    800  2350
+	1    0    0    -1
+$EndComp
+Wire Wire Line
+	800  2350 800  2550
+$Comp
+L power:+3V3 #PWR0106
+U 1 1 5C9E85B4
+P 1750 4850
+F 0 "#PWR0106" H 1750 4700 50  0001 C CNN
+F 1 "+3V3" H 1765 5023 50  0000 C CNN
+F 2 "" H 1750 4850 50  0001 C CNN
+F 3 "" H 1750 4850 50  0001 C CNN
+	1    1750 4850
+	1    0    0    -1
+$EndComp
+Wire Wire Line
+	1200 5300 1750 5300
+Wire Wire Line
+	1750 5300 1750 4850
+$Comp
+L power:+3V3 #PWR0107
+U 1 1 5C9F18CC
+P 1950 5650
+F 0 "#PWR0107" H 1950 5500 50  0001 C CNN
+F 1 "+3V3" H 1965 5823 50  0000 C CNN
+F 2 "" H 1950 5650 50  0001 C CNN
+F 3 "" H 1950 5650 50  0001 C CNN
+	1    1950 5650
+	1    0    0    -1
+$EndComp
+Wire Wire Line
+	1950 5650 1950 5900
+Wire Wire Line
+	1950 5900 1200 5900
+$Comp
+L power:+3V3 #PWR0108
+U 1 1 5C9F3DB0
+P 5050 5400
+F 0 "#PWR0108" H 5050 5250 50  0001 C CNN
+F 1 "+3V3" H 5065 5573 50  0000 C CNN
+F 2 "" H 5050 5400 50  0001 C CNN
+F 3 "" H 5050 5400 50  0001 C CNN
+	1    5050 5400
+	1    0    0    -1
+$EndComp
+Text Notes 10100 1550 0    50   ~ 0
+2v drop, 20mA max per pin
 $EndSCHEMATC

Commit message: connected GPIO to ARM board
Parts:
- U3: symbol ARM-Board-rescue:STM32L4x6RxT6-symbols-Payload_Microcontrollers -> Payload_Microcontrollers:STM32L4x6RxT6-symbols
- U4: symbol ARM-Board-rescue:SRAM_23LC1024T-I_ST-ARMlib-Payload_Microcontrollers -> Payload_Microcontrollers:SRAM_23LC1024T-I_ST-ARMlib
Connections:
- net labels added: RES0, RES1, RES2, RES3, RES4, RES5
Changed lines of the file:
@@
 Connection ~ 2500 2650
 $Comp
-L ARM-Board-rescue:STM32L4x6RxT6-symbols-Payload_Microcontrollers U?
+L Payload_Microcontrollers:STM32L4x6RxT6-symbols U?
 U 1 1 5D19DC14
 P 7450 1650
@@
 F 3 "" H 7450 1750 60  0000 C CNN
 	1    7450 1650
-	1    0    0    -1
-$EndComp
-$Comp
-L ARM-Board-rescue:STM32L4x6RxT6-symbols-Payload_Microcontrollers U?
-U 2 1 5D19DC1B
-P 2700 2150
-AR Path="/5D19DC1B" Ref="U?"  Part="2"
-AR Path="/5D19D8A9/5D19DC1B" Ref="U3"  Part="2"
-F 0 "U3" H 3600 2537 60  0000 C CNN
-F 1 "STM32L4x6RxT6-symbols" H 3600 2431 60  0000 C CNN
-F 2 "Payload_StandardPackages:STM32L4x6RxT6" H 3550 2500 60  0001 C CNN
-F 3 "" H 2700 2250 60  0000 C CNN
-	2    2700 2150
 	1    0    0    -1
 $EndComp
@@
 RAM
 $Comp
-L ARM-Board-rescue:SRAM_23LC1024T-I_ST-ARMlib-Payload_Microcontrollers U?
+L Payload_Microcontrollers:SRAM_23LC1024T-I_ST-ARMlib U?
 U 1 1 5D1A8E77
 P 4200 5400
@@
 Text Notes 10100 1550 0    50   ~ 0
 2v drop, 20mA max per pin
+Text HLabel 7450 4050 0    50   Input ~ 0
+RES0
+Text HLabel 7450 4150 0    50   Input ~ 0
+RES1
+Text HLabel 7450 4250 0    50   Input ~ 0
+RES2
+Text HLabel 7450 4350 0    50   Input ~ 0
+RES3
+Text HLabel 7450 4850 0    50   Input ~ 0
+RES4
+Text HLabel 7450 5050 0    50   Input ~ 0
+RES5
+$Comp
+L Payload_Microcontrollers:STM32L4x6RxT6-symbols U?
+U 2 1 5D19DC1B
+P 2700 2150
+AR Path="/5D19DC1B" Ref="U?"  Part="2"
+AR Path="/5D19D8A9/5D19DC1B" Ref="U3"  Part="2"
+F 0 "U3" H 3600 2537 60  0000 C CNN
+F 1 "STM32L4x6RxT6-symbols" H 3600 2431 60  0000 C CNN
+F 2 "Payload_StandardPackages:STM32L4x6RxT6" H 3550 2500 60  0001 C CNN
+F 3 "" H 2700 2250 60  0000 C CNN
+	2    2700 2150
+	1    0    0    -1
+$EndComp
 $EndSCHEMATC

Commit message: updated battery, experiment board. Added temp sensor to ARM board
Connections:
- net labels added: TEMP
Changed lines of the file:
@@
 $Descr A4 11693 8268
 encoding utf-8
-Sheet 3 4
+Sheet 4 4
 Title ""
 Date ""
@@
 	1    0    0    -1
 $EndComp
+Text HLabel 9400 2050 2    50   Input ~ 0
+TEMP
 $EndSCHEMATC

Commit message: addressed Alex's ARM review comments
Parts:
- removed R7: 0, Resistors_SMD:R_0603_HandSoldering, symbol Device:R
- added JP31: Jumper, Jumper:SolderJumper-2_P1.3mm_Open_RoundedPad1.0x1.5mm, symbol Device:Jumper
- C17: value 100uF -> 100nF
Connections:
- net labels added: ~FAULT1, ~FAULT2
- net labels removed: RES4, RES5
Changed lines of the file:
@@
 AR Path="/5D19D8A9/5D19DB79" Ref="C17"  Part="1"
 F 0 "C17" H 6065 2296 50  0000 L CNN
-F 1 "100uF" H 6065 2205 50  0000 L CNN
+F 1 "100nF" H 6065 2205 50  0000 L CNN
 F 2 "Capacitors_SMD:C_0603_HandSoldering" H 5988 2100 50  0001 C CNN
 F 3 "~" H 5950 2250 50  0001 C CNN
@@
 Wire Wire Line
 	7350 3050 7450 3050
-$Comp
-L Device:R R?
-U 1 1 5D19DBE5
-P 6400 1650
-AR Path="/5D19DBE5" Ref="R?"  Part="1"
-AR Path="/5D19D8A9/5D19DBE5" Ref="R7"  Part="1"
-F 0 "R7" V 6200 1600 50  0000 L CNN
-F 1 "0" V 6300 1600 50  0000 L CNN
-F 2 "Resistors_SMD:R_0603_HandSoldering" V 6330 1650 50  0001 C CNN
-F 3 "~" H 6400 1650 50  0001 C CNN
-	1    6400 1650
-	0    1    1    0
-$EndComp
 Wire Wire Line
 	2700 2650 2500 2650
@@
 	6650 3550 6200 3550
 Connection ~ 6650 3550
-Text Label 6250 1650 2    50   ~ 0
+Text Label 5950 1650 2    50   ~ 0
 ~(JTRST|RST)
 Text Label 9400 2250 0    50   ~ 0
@@
 RES3
 Text HLabel 7450 4850 0    50   Input ~ 0
-RES4
+~FAULT1
 Text HLabel 7450 5050 0    50   Input ~ 0
-RES5
+~FAULT2
 $Comp
 L Payload_Microcontrollers:STM32L4x6RxT6-symbols U?
@@
 Text HLabel 9400 2050 2    50   Input ~ 0
 TEMP
+$Comp
+L Device:Jumper JP31
+U 1 1 5CD1B376
+P 6250 1650
+F 0 "JP31" H 6250 1914 50  0000 C CNN
+F 1 "Jumper" H 6250 1823 50  0000 C CNN
+F 2 "Jumper:SolderJumper-2_P1.3mm_Open_RoundedPad1.0x1.5mm" H 6250 1650 50  0001 C CNN
+F 3 "~" H 6250 1650 50  0001 C CNN
+	1    6250 1650
+	1    0    0    -1
+$EndComp
 $EndSCHEMATC
