File: Hardware/Flight/ARM Board/CoreLogic.sch (KiCad schematic (older format))
At the start: 25 parts, among them J6 Conn_01x10, U3 STM32L4x6RxT6-symbols, U4 SRAM_23LC1024T-I_ST-ARMlib, Y1 Crystal

Commit message: addressing aarons comments for radio board
Connections:
- net labels added: 3v3_BACKUP
Changed lines of the file:
@@
-	1    0    0    -1
-$EndComp
-$Comp
-L power:+3V3 #PWR0105
-U 1 1 5C9E4A53
-P 800 2350
-F 0 "#PWR0105" H 800 2200 50  0001 C CNN
-F 1 "+3V3" H 815 2523 50  0000 C CNN
-F 2 "" H 800 2350 50  0001 C CNN
-F 3 "" H 800 2350 50  0001 C CNN
-	1    800  2350
 	1    0    0    -1
 $EndComp
@@
 Text HLabel 7450 4250 0    50   Input ~ 0
 RES2
-Text HLabel 7450 4350 0    50   Input ~ 0
-RES3
 Text HLabel 7450 4850 0    50   Input ~ 0
 ~FAULT1
@@
 	1    0    0    -1
 $EndComp
+Text Label 800  2350 1    50   ~ 0
+3v3_BACKUP
+Text HLabel 7450 4350 0    50   Input ~ 0
+RES3
 $EndSCHEMATC
