File: Hardware/GSE/Dongle/Dongle.sch (KiCad schematic (older format))
At the start: 16 parts, among them U1 XBee_SMT

Commit message: power supply for stm32
Other:
- note added: "USB TO UART"
- note added: "XBEE SOCKET"
Changed lines of the file:
@@
 Text Notes 700  1750 0    50   ~ 0
 TO TABLET
+Text Notes 3600 4950 0    50   ~ 0
+USB TO UART
+Text Notes 7100 5350 0    50   ~ 0
+XBEE SOCKET
 $EndSCHEMATC

Commit message: Minor changes to cap values
Parts:
- C?: value 37pF -> 47pF
- C?: value 0.1uF -> 0.01uF
- U?: symbol Regulators:AP2114H-3.3TRG1 -> Dongle-rescue:AP2114H-3.3TRG1-Regulators
Changed lines of the file:
@@
 EESchema Schematic File Version 4
+LIBS:Dongle-cache
 EELAYER 26 0
 EELAYER END
@@
 $EndComp
 $Comp
-L Regulators:AP2114H-3.3TRG1 U?
+L Dongle-rescue:AP2114H-3.3TRG1-Regulators U?
 U 1 1 5BF8B9B1
 P 5950 2100
@@
 P 1800 3650
 F 0 "C?" H 2000 3700 50  0000 L CNN
-F 1 "37pF" H 1950 3600 50  0000 L CNN
+F 1 "47pF" H 1950 3600 50  0000 L CNN
 F 2 "" H 1838 3500 50  0001 C CNN
 F 3 "~" H 1800 3650 50  0001 C CNN
@@
 P 2050 2350
 F 0 "C?" H 1750 2400 50  0000 L CNN
-F 1 "0.1uF" H 1700 2300 50  0000 L CNN
+F 1 "0.01uF" H 1700 2300 50  0000 L CNN
 F 2 "" H 2088 2200 50  0001 C CNN
 F 3 "~" H 2050 2350 50  0001 C CNN

Commit message: dongle netlist
Parts:
- C1, C2, C3, C4, C5, C6, C7, C8: renamed from C?; footprint (none) -> Capacitors_SMD:C_0805_HandSoldering
- J1, J3: renamed from J?; footprint (none) -> Connectors:USB_A
- J2: renamed from J?; footprint (none) -> Connectors:SMA_SMD_Jack_Straight
- R1, R2: renamed from R?; footprint (none) -> Resistors_SMD:R_0805_HandSoldering
- U3: renamed from U?; footprint (none) -> TO_SOT_Packages_SMD:SOT-223
- gave numbers to parts that had none: 1

Commit message: GSE dongle layout
Parts:
- removed J3: USB_A, Connectors:USB_A, symbol Connector:USB_A
- added J3: Conn_01x02_Male, Payload2019_Connectors:Molex_KK_1718570002, symbol Connector:Conn_01x02_Male
- J2: footprint Connectors:SMA_SMD_Jack_Straight -> Connectors_Molex:Molex_SMA_Jack_Edge_Mount
Connections:
- wire segments 46 -> 44
Changed lines of the file:
@@
 F 0 "J2" H 9449 3626 50  0000 L CNN
 F 1 "Conn_Coaxial" H 9449 3535 50  0000 L CNN
-F 2 "Connectors:SMA_SMD_Jack_Straight" H 9350 3650 50  0001 C CNN
+F 2 "Connectors_Molex:Molex_SMA_Jack_Edge_Mount" H 9350 3650 50  0001 C CNN
 F 3 " ~" H 9350 3650 50  0001 C CNN
 	1    9350 3650
@@
 $EndComp
 $Comp
-L Connector:USB_A J3
-U 1 1 5BF8CA16
-P 10250 2550
-F 0 "J3" H 10020 2541 50  0000 R CNN
-F 1 "USB_A" H 10020 2450 50  0000 R CNN
-F 2 "Connectors:USB_A" H 10400 2500 50  0001 C CNN
-F 3 " ~" H 10400 2500 50  0001 C CNN
-	1    10250 2550
-	-1   0    0    -1
-$EndComp
-$Comp
 L Interface_USB:FT231XS U2
 U 1 1 5BF8DADB
@@
 	5500 2050 5050 2050
 Connection ~ 5050 2050
-Text GLabel 9950 2350 0    50   Input ~ 0
+Text GLabel 10150 2450 0    50   Input ~ 0
 5V
 $Comp
@@
 L power:GND #PWR0119
 U 1 1 5BF9DE3A
-P 10250 3050
-F 0 "#PWR0119" H 10250 2800 50  0001 C CNN
-F 1 "GND" H 10255 2877 50  0000 C CNN
-F 2 "" H 10250 3050 50  0001 C CNN
-F 3 "" H 10250 3050 50  0001 C CNN
-	1    10250 3050
-	1    0    0    -1
+P 10050 2650
+F 0 "#PWR0119" H 10050 2400 50  0001 C CNN
+F 1 "GND" H 10055 2477 50  0000 C CNN
+F 2 "" H 10050 2650 50  0001 C CNN
+F 3 "" H 10050 2650 50  0001 C CNN
+	1    10050 2650
+	-1   0    0    -1
 $EndComp
 Text Notes 1000 1050 0    50   ~ 0
@@
 Text Notes 9050 3450 0    50   ~ 0
 TO ANTENNA
-Wire Wire Line
-	10250 3050 10250 3000
-Wire Wire Line
-	10250 3000 10350 3000
-Wire Wire Line
-	10350 3000 10350 2950
-Connection ~ 10250 3000
-Wire Wire Line
-	10250 3000 10250 2950
 Text Notes 9850 2100 0    50   ~ 0
 TO EXTERNAL BATTERY
@@
 Text Notes 7100 5350 0    50   ~ 0
 XBEE SOCKET
+$Comp
+L Connector:Conn_01x02_Male J3
+U 1 1 5C0427DA
+P 10350 2450
+F 0 "J3" H 10456 2628 50  0000 C CNN
+F 1 "Conn_01x02_Male" H 10456 2537 50  0000 C CNN
+F 2 "Payload2019_Connectors:Molex_KK_1718570002" H 10350 2450 50  0001 C CNN
+F 3 "~" H 10350 2450 50  0001 C CNN
+	1    10350 2450
+	-1   0    0    -1
+$EndComp
+Wire Wire Line
+	10050 2650 10050 2550
+Wire Wire Line
+	10050 2550 10150 2550
 $EndSCHEMATC

Commit message: new connectors for GSE board
Parts:
- added U4: TPD3E001DRLR, TO_SOT_Packages_SMD:SOT-553, symbol Power_Protection:TPD3E001DRLR
- J1: footprint Connectors:USB_A -> Payload2019_Connectors:629104151021
- J2: footprint Connectors_Molex:Molex_SMA_Jack_Edge_Mount -> Payload2019_Connectors:CONSMA002
Connections:
- wire segments 44 -> 56
Changed lines of the file:
@@
 F 0 "J2" H 9449 3626 50  0000 L CNN
 F 1 "Conn_Coaxial" H 9449 3535 50  0000 L CNN
-F 2 "Connectors_Molex:Molex_SMA_Jack_Edge_Mount" H 9350 3650 50  0001 C CNN
+F 2 "Payload2019_Connectors:CONSMA002" H 9350 3650 50  0001 C CNN
 F 3 " ~" H 9350 3650 50  0001 C CNN
 	1    9350 3650
@@
 F 0 "J1" H 905 2817 50  0000 C CNN
 F 1 "USB_A" H 905 2726 50  0000 C CNN
-F 2 "Connectors:USB_A" H 1000 2300 50  0001 C CNN
+F 2 "Payload2019_Connectors:629104151021" H 1000 2300 50  0001 C CNN
 F 3 " ~" H 1000 2300 50  0001 C CNN
 	1    850  2350
@@
 	3150 3300 2350 3300
 Wire Wire Line
-	1550 3300 1550 2350
-Wire Wire Line
-	1650 2450 1650 3200
+	1550 3300 1550 2950
+Wire Wire Line
+	1650 2450 1650 2850
 Wire Wire Line
 	1650 3200 1800 3200
@@
 	5500 2050 5050 2050
 Connection ~ 5050 2050
-Text GLabel 10150 2450 0    50   Input ~ 0
+Text GLabel 9500 2450 0    50   Input ~ 0
 5V
 $Comp
@@
 	2050 2150 2050 2200
 Wire Wire Line
-	1150 2150 2050 2150
+	1150 2150 1250 2150
 Connection ~ 2050 2150
 $Comp
@@
 Wire Wire Line
 	10050 2550 10150 2550
+$Comp
+L Power_Protection:TPD3E001DRLR U4
+U 1 1 5C05F3B1
+P 1850 1600
+F 0 "U4" H 1850 1967 50  0000 C CNN
+F 1 "TPD3E001DRLR" H 1850 1876 50  0000 C CNN
+F 2 "TO_SOT_Packages_SMD:SOT-553" H 1150 1300 50  0001 C CNN
+F 3 "http://www.ti.com/lit/ds/symlink/tpd3e001.pdf" H 1650 1850 50  0001 C CNN
+	1    1850 1600
+	1    0    0    -1
+$EndComp
+Wire Wire Line
+	9500 2450 10150 2450
+Wire Wire Line
+	1450 1600 1250 1600
+Wire Wire Line
+	1250 1600 1250 2150
+Connection ~ 1250 2150
+Wire Wire Line
+	1250 2150 2050 2150
+Wire Wire Line
+	2250 1500 2850 1500
+Wire Wire Line
+	2850 1500 2850 2950
+Wire Wire Line
+	2850 2950 1550 2950
+Connection ~ 1550 2950
+Wire Wire Line
+	1550 2950 1550 2350
+Wire Wire Line
+	2250 1600 2700 1600
+Wire Wire Line
+	2700 1600 2700 2850
+Wire Wire Line
+	2700 2850 1650 2850
+Connection ~ 1650 2850
+Wire Wire Line
+	1650 2850 1650 3200
+$Comp
+L power:GND #PWR0120
+U 1 1 5C062C64
+P 1850 1900
+F 0 "#PWR0120" H 1850 1650 50  0001 C CNN
+F 1 "GND" H 1855 1727 50  0000 C CNN
+F 2 "" H 1850 1900 50  0001 C CNN
+F 3 "" H 1850 1900 50  0001 C CNN
+	1    1850 1900
+	1    0    0    -1
+$EndComp
 $EndSCHEMATC

Commit message: updated dongle for LoRa
Parts:
- removed C7: 100pF, Capacitors_SMD:C_0805_HandSoldering, symbol Device:C
- removed J3: Conn_01x02_Male, Payload2019_Connectors:Molex_KK_1718570002, symbol Connector:Conn_01x02_Male
- removed U1: XBee_SMT, RF_Module:Digi_XBee_SMT, symbol RF_ZigBee:XBee_SMT
- added C?: 0.1uF, symbol Device:C
- added C? (x2): C, symbol Device:C
- added J?: Conn_01x05_Female, symbol Connector:Conn_01x05_Female
- added J?: USB_B_Micro, symbol Connector:USB_B_Micro
- added R? (x3): 10k, symbol Device:R
- added U?: PIC18F26K83, symbol canhw:PIC18F26K83
- added U?: RFM95W-915S2, symbol RF_AM_FM:RFM95W-915S2
- added Y?: Crystal, symbol Device:Crystal
- C8: value 1uF -> 10uF
Connections:
- net labels added: +3.3V, +5V, CS, ICSPCLK, ICSPDAT, MISO, MOSI, OSC1, OSC2, RESET, SCK, USBDM, USBDP, ~MCLR
- net labels removed: 5V, DTR
- wire segments 56 -> 94
Other:
- note added: "LoRa RADIO"
- note added: "PIC CIRCUIT"
- note added: "TO PIC PROGRAMMER"
- note added: "VOLTAGE REGULATOR"
- note removed: "3.3v"
- note removed: "XBEE SOCKET"

Commit message: new dongle with LoRa for review
Parts:
- removed J?: USB_B_Micro, symbol Connector:USB_B_Micro
- removed U4: TPD3E001DRLR, TO_SOT_Packages_SMD:SOT-553, symbol Power_Protection:TPD3E001DRLR
- added D1: D_TVS, Diodes_SMD:D_0603, symbol Device:D_TVS
- C1, C2, C3, C4, C5, C6, C8: footprint Capacitors_SMD:C_0805_HandSoldering -> Capacitors_SMD:C_0603_HandSoldering
- C10, C7, C9: renamed from C?; footprint (none) -> Capacitors_SMD:C_0603_HandSoldering
- J1: footprint Payload2019_Connectors:629104151021 -> Payload_Connectors:629104151021
- J2: footprint Payload2019_Connectors:CONSMA002 -> Payload_Connectors:CONSMA002
- J4: renamed from J?; footprint (none) -> Payload_Connectors:PinHeader_5x2.54_SMD_90deg_952-3198-1-ND
- R1, R2: footprint Resistors_SMD:R_0805_HandSoldering -> Resistors_SMD:R_0603_HandSoldering
- R3, R4, R5: renamed from R?; footprint (none) -> Resistors_SMD:R_0603_HandSoldering
- U1: renamed from U?; footprint (none) -> Housings_SOIC:SOIC-28W_7.5x18.7mm_Pitch1.27mm
- U5: renamed from U?; footprint (none) -> RF_Modules:Hopref_RFM9XW_SMD
- Y1: renamed from Y?; footprint (none) -> Crystals:Crystal_HC49-U_Vertical
Connections:
- net labels added: D1+, D1-, DIO0, DIO1, DIO2, DIO3, DIO4, DIO5, USBD+, USBD-
- net labels removed: USBDM, USBDP
- wire segments 94 -> 83
Other:
- note removed: "TO EXTERNAL BATTERY"

Commit message: updated dongle based on review
Parts:
- U1: value PIC18F26K83 -> PICLF26K83; symbol canhw:PIC18F26K83 -> canhw:PICLF26K83
Changed lines of the file:
@@
 Design heavily based on https://cdn.sparkfun.com/datasheets/Wireless/Zigbee/XBee-Explorer-Dongle-v23.pdf
-Wire Wire Line
-	1650 2450 1150 2450
-Wire Wire Line
-	1550 2350 1150 2350
 Wire Wire Line
 	850  2900 850  2850
@@
 USB TO UART
 $Comp
-L canhw:PIC18F26K83 U1
+L canhw:PICLF26K83 U1
 U 1 1 5C4F4F80
 P 5550 4300
 F 0 "U1" H 5525 5215 50  0000 C CNN
-F 1 "PIC18F26K83" H 5525 5124 50  0000 C CNN
+F 1 "PICLF26K83" H 5525 5124 50  0000 C CNN
 F 2 "Housings_SOIC:SOIC-28W_7.5x18.7mm_Pitch1.27mm" H 6000 4300 50  0001 C CNN
-F 3 "http://ww1.microchip.com/downloads/en/DeviceDoc/40001943A.pdf" H 6000 4300 50  0001 C CNN
+F 3 "" H 6000 4300 50  0001 C CNN
 	1    5550 4300
-	1    0    0    -1
-$EndComp
-$Comp
-L power:+5V #PWR0103
-U 1 1 5C4F533C
-P 6450 3500
-F 0 "#PWR0103" H 6450 3350 50  0001 C CNN
-F 1 "+5V" H 6465 3673 50  0000 C CNN
-F 2 "" H 6450 3500 50  0001 C CNN
-F 3 "" H 6450 3500 50  0001 C CNN
-	1    6450 3500
 	1    0    0    -1
 $EndComp
@@
 Wire Wire Line
 	4600 3650 4800 3650
-$Comp
-L power:+5V #PWR0106
-U 1 1 5C4F8A5B
-P 4600 3200
-F 0 "#PWR0106" H 4600 3050 50  0001 C CNN
-F 1 "+5V" H 4615 3373 50  0000 C CNN
-F 2 "" H 4600 3200 50  0001 C CNN
-F 3 "" H 4600 3200 50  0001 C CNN
-	1    4600 3200
-	1    0    0    -1
-$EndComp
 $Comp
 L Connector:Conn_01x05_Female J4
@@
 Text Notes 1100 5900 0    50   ~ 0
 TO PIC PROGRAMMER
+Text Label 8100 4100 2    50   ~ 0
+USBD+
 Text Label 8100 4000 2    50   ~ 0
-USBD+
-Text Label 8100 4100 2    50   ~ 0
 USBD-
 Text Label 2900 3200 0    50   ~ 0
@@
 	1150 2150 2400 2150
 Wire Wire Line
-	1650 2450 1650 3200
-Wire Wire Line
-	1550 2350 1550 3300
+	1650 2350 1650 3200
+Wire Wire Line
+	1550 2450 1550 3300
 $Comp
 L Device:D_TVS D1
@@
 Wire Wire Line
 	2400 2150 2850 2150
+Wire Wire Line
+	1650 2350 1150 2350
+Wire Wire Line
+	1150 2450 1550 2450
+$Comp
+L power:+3.3V #PWR?
+U 1 1 5C7F9CD3
+P 4600 3200
+F 0 "#PWR?" H 4600 3050 50  0001 C CNN
+F 1 "+3.3V" H 4615 3373 50  0000 C CNN
+F 2 "" H 4600 3200 50  0001 C CNN
+F 3 "" H 4600 3200 50  0001 C CNN
+	1    4600 3200
+	1    0    0    -1
+$EndComp
+$Comp
+L power:+3.3V #PWR?
+U 1 1 5C7F9D60
+P 6450 3500
+F 0 "#PWR?" H 6450 3350 50  0001 C CNN
+F 1 "+3.3V" H 6465 3673 50  0000 C CNN
+F 2 "" H 6450 3500 50  0001 C CNN
+F 3 "" H 6450 3500 50  0001 C CNN
+	1    6450 3500
+	1    0    0    -1
+$EndComp
 $EndSCHEMATC
