File: Hardware/Flight/Radio Board/Radio Board.sch (KiCad schematic (older format))
At the start: 3 parts

Commit message: radio board int resets and antenna
Parts:
- added J? (x2): Conn_Coaxial, symbol Connector:Conn_Coaxial
- added R? (x4): 10k, symbol Device:R
Connections:
- net labels added: RST1, RST2
- wire segments 4 -> 18
Other:
- note removed: "TODO\nRESET PINS\nANTENNAS"
- moved on the sheet: U?

Commit message: Radio board layout
Parts:
- added C1, C2: 10uF, Capacitors_SMD:C_0805_HandSoldering, symbol Device:C
- J1: renamed from J?; footprint (none) -> Pin_Headers:Pin_Header_Straight_2x10_Pitch2.54mm
- J2, J3: renamed from J?; footprint (none) -> Downloaded Connectors:U.FL_Hirose_U.FL-R-SMT-1_Vertical
- R1, R2, R3, R4: renamed from R?; footprint (none) -> Resistors_SMD:R_0805_HandSoldering
- U1, U2: renamed from U?; footprint (none) -> RF_Modules:Hopref_RFM9XW_THT
Connections:
- wire segments 18 -> 26

Commit message: radio board for review
Parts:
- C1, C2: footprint Capacitors_SMD:C_0805_HandSoldering -> Capacitors_SMD:C_0603_HandSoldering
- J1: symbol Payload_Connections:Conn_01x20_Female -> Payload_Connectors:Conn_01x20_Female
- R1, R2, R3, R4: footprint Resistors_SMD:R_0805_HandSoldering -> Resistors_SMD:R_0603_HandSoldering
Connections:
- net labels removed: RST1, RST2
- wire segments 26 -> 24
Changed lines of the file:
@@
 $EndComp
 $Comp
-L Payload_Connections:Conn_01x20_Female J1
+L Payload_Connectors:Conn_01x20_Female J1
 U 1 1 5C146FED
 P 2950 4300
@@
 Text GLabel 3100 4250 2    50   Input ~ 0
 CS2
-Text GLabel 3100 4150 2    50   Input ~ 0
+Text GLabel 3100 4750 2    50   Input ~ 0
 INT1
-Text GLabel 3100 4050 2    50   Input ~ 0
+Text GLabel 3100 4850 2    50   Input ~ 0
 INT2
 $Comp
@@
 	1    0    0    -1
 $EndComp
-Text GLabel 3100 3950 2    50   Input ~ 0
-RST1
-Text GLabel 3100 3850 2    50   Input ~ 0
-RST2
 $Comp
 L Device:R R2
@@
 F 0 "R2" H 4820 4696 50  0000 L CNN
 F 1 "10k" H 4820 4605 50  0000 L CNN
-F 2 "Resistors_SMD:R_0805_HandSoldering" V 4680 4650 50  0001 C CNN
+F 2 "Resistors_SMD:R_0603_HandSoldering" V 4680 4650 50  0001 C CNN
 F 3 "~" H 4750 4650 50  0001 C CNN
 	1    4750 4650
@@
 	1    0    0    -1
 $EndComp
-Text GLabel 4650 5350 0    50   Input ~ 0
-RST2
-Wire Wire Line
-	4650 5350 4750 5350
-Connection ~ 4750 5350
 Wire Wire Line
 	4750 5350 5600 5350
@@
 F 0 "R4" H 5270 4696 50  0000 L CNN
 F 1 "10k" H 5270 4605 50  0000 L CNN
-F 2 "Resistors_SMD:R_0805_HandSoldering" V 5130 4650 50  0001 C CNN
+F 2 "Resistors_SMD:R_0603_HandSoldering" V 5130 4650 50  0001 C CNN
 F 3 "~" H 5200 4650 50  0001 C CNN
 	1    5200 4650
@@
 F 0 "R1" H 4820 2896 50  0000 L CNN
 F 1 "10k" H 4820 2805 50  0000 L CNN
-F 2 "Resistors_SMD:R_0805_HandSoldering" V 4680 2850 50  0001 C CNN
+F 2 "Resistors_SMD:R_0603_HandSoldering" V 4680 2850 50  0001 C CNN
 F 3 "~" H 4750 2850 50  0001 C CNN
 	1    4750 2850
@@
 	1    0    0    -1
 $EndComp
-Text GLabel 4650 3550 0    50   Input ~ 0
-RST1
-Wire Wire Line
-	4650 3550 4750 3550
-Connection ~ 4750 3550
 Wire Wire Line
 	4750 3550 5600 3550
@@
 F 0 "R3" H 5270 2896 50  0000 L CNN
 F 1 "10k" H 5270 2805 50  0000 L CNN
-F 2 "Resistors_SMD:R_0805_HandSoldering" V 5130 2850 50  0001 C CNN
+F 2 "Resistors_SMD:R_0603_HandSoldering" V 5130 2850 50  0001 C CNN
 F 3 "~" H 5200 2850 50  0001 C CNN
 	1    5200 2850
@@
 F 0 "C1" H 6665 2496 50  0000 L CNN
 F 1 "10uF" H 6665 2405 50  0000 L CNN
-F 2 "Capacitors_SMD:C_0805_HandSoldering" H 6588 2300 50  0001 C CNN
+F 2 "Capacitors_SMD:C_0603_HandSoldering" H 6588 2300 50  0001 C CNN
 F 3 "~" H 6550 2450 50  0001 C CNN
 	1    6550 2450
@@
 F 0 "C2" H 8015 4746 50  0000 L CNN
 F 1 "10uF" H 8015 4655 50  0000 L CNN
-F 2 "Capacitors_SMD:C_0805_HandSoldering" H 7938 4550 50  0001 C CNN
+F 2 "Capacitors_SMD:C_0603_HandSoldering" H 7938 4550 50  0001 C CNN
 F 3 "~" H 7900 4700 50  0001 C CNN
 	1    7900 4700

Commit message: Radio Review
Added Debug LEDs
Rerouted traces to keep away from edge
Made RF traces shorter
Switched RFM95W to SMD version
Parts:
- added D1, D2, D3, D4: LED, LEDs:LED_0603_HandSoldering, symbol Device:LED
- added JP1, JP2, JP3, JP4: Jumper, Jumper:SolderJumper-2_P1.3mm_Open_RoundedPad1.0x1.5mm, symbol Device:Jumper
- added R5, R6, R7, R8: 70, Resistors_SMD:R_0603_HandSoldering, symbol Device:R
- U1, U2: footprint RF_Modules:Hopref_RFM9XW_THT -> RF_Modules:Hopref_RFM9XW_SMD
Connections:
- wire segments 24 -> 40
Other:
- moved on the sheet: U1, U2

Commit message: updated battery, experiment board. Added temp sensor to ARM board
Parts:
- removed J1: Conn_01x20_Female, Pin_Headers:Pin_Header_Straight_2x10_Pitch2.54mm, symbol Payload_Connectors:Conn_01x20_Female
- added J1: Bus_Connector, Payload_Connectors:Pin_Header_Straight_2x10_Pitch2.54mm, symbol Payload_Connectors:Bus_Connector
Changed lines of the file:
@@
-$EndComp
-$Comp
-L Payload_Connectors:Conn_01x20_Female J1
-U 1 1 5C146FED
-P 1700 4000
-F 0 "J1" H 1877 3941 50  0000 L CNN
-F 1 "Conn_01x20_Female" H 1877 3850 50  0000 L CNN
-F 2 "Pin_Headers:Pin_Header_Straight_2x10_Pitch2.54mm" H 1750 3950 50  0001 C CNN
-F 3 "" H 1750 3950 50  0001 C CNN
-	1    1700 4000
-	-1   0    0    1
 $EndComp
 $Comp
@@
 Wire Wire Line
 	6200 4700 6900 4700
+$Comp
+L Payload_Connectors:Bus_Connector J1
+U 1 1 5CC7A6A1
+P 1650 3950
+F 0 "J1" H 1461 5175 50  0000 C CNN
+F 1 "Bus_Connector" H 1461 5084 50  0000 C CNN
+F 2 "Payload_Connectors:Pin_Header_Straight_2x10_Pitch2.54mm" H 1750 4700 50  0001 C CNN
+F 3 "" H 1750 4700 50  0001 C CNN
+	1    1650 3950
+	1    0    0    -1
+$EndComp
 $EndSCHEMATC

Commit message: addressing aarons comments for radio board
Parts:
- removed JP1, JP2, JP3, JP4: Jumper, Jumper:SolderJumper-2_P1.3mm_Open_RoundedPad1.0x1.5mm, symbol Device:Jumper
- R3, R4: value 10k -> DNP
Connections:
- net labels added: ~CS1, ~CS2
- net labels removed: CS1, CS2
- wire segments 40 -> 42
Changed lines of the file:
@@
 Wire Wire Line
 	2100 3050 2100 2750
-Text GLabel 1850 4350 2    50   Input ~ 0
-MISO
-Text GLabel 1850 4250 2    50   Input ~ 0
-MOSI
-Text GLabel 1850 4150 2    50   Input ~ 0
-SCK
-Text GLabel 1850 4050 2    50   Input ~ 0
-CS1
-Text GLabel 1850 3950 2    50   Input ~ 0
-CS2
-Text GLabel 1850 4450 2    50   Input ~ 0
-INT1
-Text GLabel 1850 4550 2    50   Input ~ 0
-INT2
 $Comp
 L power:GND #PWR0103
@@
 	1    0    0    -1
 $EndComp
-Text GLabel 6650 2600 2    50   Input ~ 0
-INT1
-Text GLabel 5200 1900 0    50   Input ~ 0
-SCK
 $Comp
 L power:+3V3 #PWR0106
@@
 	1    0    0    -1
 $EndComp
-Text GLabel 5200 4500 0    50   Input ~ 0
-MISO
-Text GLabel 5200 4400 0    50   Input ~ 0
-MOSI
-Text GLabel 5200 4300 0    50   Input ~ 0
-SCK
 $Comp
 L power:+3V3 #PWR0110
@@
 P 4800 4100
 F 0 "R4" H 4870 4146 50  0000 L CNN
-F 1 "10k" H 4870 4055 50  0000 L CNN
+F 1 "DNP" H 4870 4055 50  0000 L CNN
 F 2 "Resistors_SMD:R_0603_HandSoldering" V 4730 4100 50  0001 C CNN
 F 3 "~" H 4800 4100 50  0001 C CNN
@@
 Wire Wire Line
 	4350 4250 4350 4800
-Text GLabel 4700 4600 0    50   Input ~ 0
-CS2
 Wire Wire Line
 	4700 4600 4800 4600
 Connection ~ 4800 4600
-Text GLabel 5200 2100 0    50   Input ~ 0
-MISO
-Text GLabel 5200 2000 0    50   Input ~ 0
-MOSI
 $Comp
 L Device:R R1
@@
 P 4800 1700
 F 0 "R3" H 4870 1746 50  0000 L CNN
-F 1 "10k" H 4870 1655 50  0000 L CNN
+F 1 "DNP" H 4870 1655 50  0000 L CNN
 F 2 "Resistors_SMD:R_0603_HandSoldering" V 4730 1700 50  0001 C CNN
 F 3 "~" H 4800 1700 50  0001 C CNN
@@
 Wire Wire Line
 	4350 1850 4350 2400
-Text GLabel 4700 2200 0    50   Input ~ 0
-CS1
 Wire Wire Line
 	4700 2200 4800 2200
@@
 	1    0    0    -1
 $EndComp
-$Comp
-L Device:Jumper JP1
-U 1 1 5CA0A75B
-P 6800 2950
-F 0 "JP1" H 6800 3100 50  0000 C CNN
-F 1 "Jumper" H 6800 2850 50  0000 C CNN
-F 2 "Jumper:SolderJumper-2_P1.3mm_Open_RoundedPad1.0x1.5mm" H 6800 2950 50  0001 C CNN
-F 3 "~" H 6800 2950 50  0001 C CNN
-	1    6800 2950
-	1    0    0    -1
-$EndComp
 Wire Wire Line
 	7400 2950 7450 2950
@@
 Wire Wire Line
 	6500 2600 6650 2600
-$Comp
-L Device:Jumper JP3
-U 1 1 5CA0CD47
-P 7200 2300
-F 0 "JP3" H 7200 2450 50  0000 C CNN
-F 1 "Jumper" H 7200 2200 50  0000 C CNN
-F 2 "Jumper:SolderJumper-2_P1.3mm_Open_RoundedPad1.0x1.5mm" H 7200 2300 50  0001 C CNN
-F 3 "~" H 7200 2300 50  0001 C CNN
-	1    7200 2300
-	1    0    0    -1
-$EndComp
 Wire Wire Line
 	7800 2300 7850 2300
@@
 	1    0    0    -1
 $EndComp
-Wire Wire Line
-	6200 2300 6900 2300
-Text GLabel 6650 5000 2    50   Input ~ 0
-INT2
 $Comp
 L Device:LED D4
@@
 	1    0    0    -1
 $EndComp
-$Comp
-L Device:Jumper JP2
-U 1 1 5CA0E67D
-P 6800 5350
-F 0 "JP2" H 6800 5500 50  0000 C CNN
-F 1 "Jumper" H 6800 5250 50  0000 C CNN
-F 2 "Jumper:SolderJumper-2_P1.3mm_Open_RoundedPad1.0x1.5mm" H 6800 5350 50  0001 C CNN
-F 3 "~" H 6800 5350 50  0001 C CNN
-	1    6800 5350
-	1    0    0    -1
-$EndComp
 Wire Wire Line
 	7400 5350 7450 5350
@@
 Wire Wire Line
 	6500 5000 6650 5000
-$Comp
-L Device:Jumper JP4
-U 1 1 5CA0E687
-P 7200 4700
-F 0 "JP4" H 7200 4850 50  0000 C CNN
-F 1 "Jumper" H 7200 4600 50  0000 C CNN
-F 2 "Jumper:SolderJumper-2_P1.3mm_Open_RoundedPad1.0x1.5mm" H 7200 4700 50  0001 C CNN
-F 3 "~" H 7200 4700 50  0001 C CNN
-	1    7200 4700
-	1    0    0    -1
-$EndComp
 Wire Wire Line
 	7800 4700 7850 4700
@@
 	1    0    0    -1
 $EndComp
-Wire Wire Line
-	6200 4700 6900 4700
 $Comp
 L Payload_Connectors:Bus_Connector J1
@@
 	1    0    0    -1
 $EndComp
+Wire Wire Line
+	6200 4700 7500 4700
+Wire Wire Line
+	6500 5350 7100 5350
+Text Label 5200 1900 2    50   ~ 0
+SCK
+Text Label 5200 2000 2    50   ~ 0
+MOSI
+Text Label 5200 2100 2    50   ~ 0
+MISO
+Text Label 4700 2200 2    50   ~ 0
+~CS1
+Wire Wire Line
+	6200 2300 7500 2300
+Wire Wire Line
+	6500 2950 7100 2950
+Text Label 6650 2600 0    50   ~ 0
+INT1
+Text Label 5200 4300 2    50   ~ 0
+SCK
+Text Label 5200 4400 2    50   ~ 0
+MOSI
+Text Label 5200 4500 2    50   ~ 0
+MISO
+Text Label 4700 4600 2    50   ~ 0
+~CS2
+Text Label 6650 5000 0    50   ~ 0
+INT2
+Text Label 1850 3950 0    50   ~ 0
+~CS2
+Text Label 1850 4050 0    50   ~ 0
+~CS1
+Text Label 1850 4150 0    50   ~ 0
+SCK
+Text Label 1850 4250 0    50   ~ 0
+MOSI
+Text Label 1850 4350 0    50   ~ 0
+MISO
+Text Label 1850 4450 0    50   ~ 0
+INT1
+Text Label 1850 4550 0    50   ~ 0
+INT2
 $EndSCHEMATC
