File: Hardware/Flight/Battery Board/Battery Board/Battery Board.sch (KiCad schematic (older format))
At the start: 7 parts

Commit message: added battery board + ADCs for experiment board
Parts:
- removed J?: Conn_01x20_Female, symbol Payload_Connectors:Conn_01x20_Female
- added C1, C2: 1nF, symbol Device:C
- added C3, C4, C?: 0.1uF, symbol Device:C
- added C5: 22uF, symbol Device:C
- added C6, C7: 10uF, symbol Device:C
- added D1: D_Schottky_x2_KCom_KAA, symbol Device:D_Schottky_x2_KCom_KAA
- added J5: Conn_01x20, symbol Connector_Generic:Conn_01x20
- added J6: Conn_01x02, symbol Connector_Generic:Conn_01x02
- added U1, U2: ACS711KEXLT-31AB-T, symbol Payload_Sensors:ACS711KEXLT-31AB-T
- added U?: TLA2022IRUGT, symbol Payload_ADC:TLA2022IRUGT
- gave numbers to parts that had none: 6
Connections:
- net labels added: +24V, CURR_1, CURR_2, SCL, SDA
- wire segments 30 -> 81
- no-connect marks 0 -> 11
Other:
- note removed: "-24V source"
- moved on the sheet: U3

Commit message: updated battery, experiment board. Added temp sensor to ARM board
Parts:
- removed J5: Conn_01x20, symbol Connector_Generic:Conn_01x20
- added J?: Bus_Connector, symbol Payload_Connectors:Bus_Connector
- added R? (x2): 10k, symbol Device:R
Connections:
- net labels added: ~Fault1, ~Fault2
- wire segments 81 -> 89
Changed lines of the file:
@@
 L Device:D_Schottky_x2_KCom_KAA D1
 U 1 1 5C9F2FC4
-P 3900 2850
-F 0 "D1" V 3946 2928 50  0000 L CNN
-F 1 "D_Schottky_x2_KCom_KAA" V 3750 1800 50  0000 L CNN
-F 2 "" H 3900 2850 50  0001 C CNN
-F 3 "~" H 3900 2850 50  0001 C CNN
-	1    3900 2850
+P 4050 2850
+F 0 "D1" V 4096 2928 50  0000 L CNN
+F 1 "D_Schottky_x2_KCom_KAA" V 3900 1800 50  0000 L CNN
+F 2 "" H 4050 2850 50  0001 C CNN
+F 3 "~" H 4050 2850 50  0001 C CNN
+	1    4050 2850
 	0    -1   -1   0
 $EndComp
@@
 	2250 3350 2400 3350
 Wire Wire Line
-	2250 2450 3900 2450
-Wire Wire Line
-	3900 2450 3900 2550
+	2250 2450 4050 2450
+Wire Wire Line
+	4050 2450 4050 2550
 Wire Wire Line
 	2250 1750 2250 2450
 Wire Wire Line
-	3900 3150 3900 4650
-Wire Wire Line
-	3900 4650 2250 4650
+	4050 3150 4050 4650
+Wire Wire Line
+	4050 4650 2250 4650
 Wire Wire Line
 	2250 4650 2250 3650
@@
 	4300 2650 4300 2850
 Wire Wire Line
-	4300 2850 4100 2850
+	4300 2850 4250 2850
 $Comp
 L power:+24V #PWR012
@@
 $EndComp
 $Comp
-L Connector_Generic:Conn_01x20 J5
-U 1 1 5CA1B4EE
-P 8600 1900
-F 0 "J5" H 8680 1892 50  0000 L CNN
-F 1 "Conn_01x20" H 8680 1801 50  0000 L CNN
-F 2 "" H 8600 1900 50  0001 C CNN
-F 3 "~" H 8600 1900 50  0001 C CNN
-	1    8600 1900
-	1    0    0    -1
-$EndComp
-$Comp
 L Connector_Generic:Conn_01x02 J6
 U 1 1 5CA1B590
@@
 Text Label 8400 2700 2    50   ~ 0
 SCL
+$Comp
+L Payload_Connectors:Bus_Connector J?
+U 1 1 5CA3FA86
+P 8600 2000
+F 0 "J?" H 7981 2101 50  0000 R CNN
+F 1 "Bus_Connector" H 7981 2010 50  0000 R CNN
+F 2 "" H 8700 2750 50  0001 C CNN
+F 3 "" H 8700 2750 50  0001 C CNN
+	1    8600 2000
+	-1   0    0    -1
+$EndComp
+Wire Wire Line
+	2950 2300 2950 2200
+Text Label 3700 4200 0    50   ~ 0
+~Fault2
+Wire Wire Line
+	2950 4200 2950 4100
+Text Label 8400 1800 2    50   ~ 0
+~Fault1
+Text Label 8400 1900 2    50   ~ 0
+~Fault2
+$Comp
+L Device:R R?
+U 1 1 5CA46901
+P 3650 3900
+F 0 "R?" H 3720 3946 50  0000 L CNN
+F 1 "10k" H 3720 3855 50  0000 L CNN
+F 2 "" V 3580 3900 50  0001 C CNN
+F 3 "~" H 3650 3900 50  0001 C CNN
+	1    3650 3900
+	1    0    0    -1
+$EndComp
+Wire Wire Line
+	3650 4050 3650 4200
+Wire Wire Line
+	3650 4200 3700 4200
+Wire Wire Line
+	2950 4200 3650 4200
+Connection ~ 3650 4200
+$Comp
+L power:+3V3 #PWR?
+U 1 1 5CA4A84A
+P 3650 3750
+F 0 "#PWR?" H 3650 3600 50  0001 C CNN
+F 1 "+3V3" H 3665 3923 50  0000 C CNN
+F 2 "" H 3650 3750 50  0001 C CNN
+F 3 "" H 3650 3750 50  0001 C CNN
+	1    3650 3750
+	-1   0    0    -1
+$EndComp
+Text Label 3700 2300 0    50   ~ 0
+~Fault1
+$Comp
+L Device:R R?
+U 1 1 5CA4A8F0
+P 3650 2000
+F 0 "R?" H 3720 2046 50  0000 L CNN
+F 1 "10k" H 3720 1955 50  0000 L CNN
+F 2 "" V 3580 2000 50  0001 C CNN
+F 3 "~" H 3650 2000 50  0001 C CNN
+	1    3650 2000
+	1    0    0    -1
+$EndComp
+Wire Wire Line
+	3650 2150 3650 2300
+Wire Wire Line
+	3650 2300 3700 2300
+Connection ~ 3650 2300
+$Comp
+L power:+3V3 #PWR?
+U 1 1 5CA4A8FA
+P 3650 1850
+F 0 "#PWR?" H 3650 1700 50  0001 C CNN
+F 1 "+3V3" H 3665 2023 50  0000 C CNN
+F 2 "" H 3650 1850 50  0001 C CNN
+F 3 "" H 3650 1850 50  0001 C CNN
+	1    3650 1850
+	-1   0    0    -1
+$EndComp
+Wire Wire Line
+	2950 2300 3650 2300
 $EndSCHEMATC

Commit message: addressed Alex's ARM review comments
Parts:
- added D? (x3): LED, symbol Device:LED
- added J?: Conn_01x02, symbol Connector_Generic:Conn_01x02
- added Q?: Q_PMOS_DGS, symbol Device:Q_PMOS_DGS
- added R?: 1.2k, symbol Device:R
- added R?: 150, symbol Device:R
- added R?: 70, symbol Device:R
- added R?: 10k, symbol Device:R
Connections:
- net labels added: SWITCH
- wire segments 89 -> 93
Other:
- note added: "POWER SWITCH"
Changed lines of the file:
@@
 P 4050 2850
 F 0 "D1" V 4096 2928 50  0000 L CNN
-F 1 "D_Schottky_x2_KCom_KAA" V 3900 1800 50  0000 L CNN
+F 1 "D_Schottky_x2_KCom_KAA" V 4500 2300 50  0000 L CNN
 F 2 "" H 4050 2850 50  0001 C CNN
 F 3 "~" H 4050 2850 50  0001 C CNN
@@
 	2250 1450 2400 1450
 Wire Wire Line
-	1500 1450 2250 1450
-Connection ~ 2250 1450
-Wire Wire Line
 	2250 1450 2250 1550
 Wire Wire Line
@@
 	2300 2850 2300 2900
 Wire Wire Line
-	1600 3350 2250 3350
-Wire Wire Line
 	2250 3350 2250 3450
 Wire Wire Line
@@
 L power:+24V #PWR011
 U 1 1 5CA1651D
-P 4300 2650
-F 0 "#PWR011" H 4300 2500 50  0001 C CNN
-F 1 "+24V" H 4315 2823 50  0000 C CNN
-F 2 "" H 4300 2650 50  0001 C CNN
-F 3 "" H 4300 2650 50  0001 C CNN
-	1    4300 2650
-	1    0    0    -1
-$EndComp
-Wire Wire Line
-	4300 2650 4300 2850
-Wire Wire Line
-	4300 2850 4250 2850
+P 4750 2650
+F 0 "#PWR011" H 4750 2500 50  0001 C CNN
+F 1 "+24V" H 4765 2823 50  0000 C CNN
+F 2 "" H 4750 2650 50  0001 C CNN
+F 3 "" H 4750 2650 50  0001 C CNN
+	1    4750 2650
+	1    0    0    -1
+$EndComp
 $Comp
 L power:+24V #PWR012
@@
 Wire Wire Line
 	2950 2300 3650 2300
+$Comp
+L Device:LED D?
+U 1 1 5CCF7F1F
+P 6100 5250
+F 0 "D?" V 6138 5133 50  0000 R CNN
+F 1 "LED" V 6047 5133 50  0000 R CNN
+F 2 "" H 6100 5250 50  0001 C CNN
+F 3 "~" H 6100 5250 50  0001 C CNN
+	1    6100 5250
+	0    -1   -1   0
+$EndComp
+$Comp
+L Device:LED D?
+U 1 1 5CCF842B
+P 5400 5250
+F 0 "D?" V 5438 5133 50  0000 R CNN
+F 1 "LED" V 5347 5133 50  0000 R CNN
+F 2 "" H 5400 5250 50  0001 C CNN
+F 3 "~" H 5400 5250 50  0001 C CNN
+	1    5400 5250
+	0    -1   -1   0
+$EndComp
+$Comp
+L Device:LED D?
+U 1 1 5CCF84A5
+P 5750 5250
+F 0 "D?" V 5788 5133 50  0000 R CNN
+F 1 "LED" V 5697 5133 50  0000 R CNN
+F 2 "" H 5750 5250 50  0001 C CNN
+F 3 "~" H 5750 5250 50  0001 C CNN
+	1    5750 5250
+	0    -1   -1   0
+$EndComp
+$Comp
+L power:+24V #PWR?
+U 1 1 5CCF8A94
+P 5400 5100
+F 0 "#PWR?" H 5400 4950 50  0001 C CNN
+F 1 "+24V" H 5415 5273 50  0000 C CNN
+F 2 "" H 5400 5100 50  0001 C CNN
+F 3 "" H 5400 5100 50  0001 C CNN
+	1    5400 5100
+	1    0    0    -1
+$EndComp
+$Comp
+L power:+5V #PWR?
+U 1 1 5CCF8B35
+P 5750 5100
+F 0 "#PWR?" H 5750 4950 50  0001 C CNN
+F 1 "+5V" H 5765 5273 50  0000 C CNN
+F 2 "" H 5750 5100 50  0001 C CNN
+F 3 "" H 5750 5100 50  0001 C CNN
+	1    5750 5100
+	1    0    0    -1
+$EndComp
+$Comp
+L power:+3V3 #PWR?
+U 1 1 5CCF8CA8
+P 6100 5100
+F 0 "#PWR?" H 6100 4950 50  0001 C CNN
+F 1 "+3V3" H 6115 5273 50  0000 C CNN
+F 2 "" H 6100 5100 50  0001 C CNN
+F 3 "" H 6100 5100 50  0001 C CNN
+	1    6100 5100
+	1    0    0    -1
+$EndComp
+$Comp
+L Device:R R?
+U 1 1 5CCF8E98
+P 5400 5550
+F 0 "R?" H 5470 5596 50  0000 L CNN
+F 1 "1.2k" H 5470 5505 50  0000 L CNN
+F 2 "" V 5330 5550 50  0001 C CNN
+F 3 "~" H 5400 5550 50  0001 C CNN
+	1    5400 5550
+	1    0    0    -1
+$EndComp
+$Comp
+L Device:R R?
+U 1 1 5CCF909C
+P 5750 5550
+F 0 "R?" H 5820 5596 50  0000 L CNN
+F 1 "150" H 5820 5505 50  0000 L CNN
+F 2 "" V 5680 5550 50  0001 C CNN
+F 3 "~" H 5750 5550 50  0001 C CNN
+	1    5750 5550
+	1    0    0    -1
+$EndComp
+$Comp
+L Device:R R?
+U 1 1 5CCF90F0
+P 6100 5550
+F 0 "R?" H 6170 5596 50  0000 L CNN
+F 1 "70" H 6170 5505 50  0000 L CNN
+F 2 "" V 6030 5550 50  0001 C CNN
+F 3 "~" H 6100 5550 50  0001 C CNN
+	1    6100 5550
+	1    0    0    -1
+$EndComp
+$Comp
+L power:GND #PWR?
+U 1 1 5CCF97C9
+P 5400 5700
+F 0 "#PWR?" H 5400 5450 50  0001 C CNN
+F 1 "GND" H 5405 5527 50  0000 C CNN
+F 2 "" H 5400 5700 50  0001 C CNN
+F 3 "" H 5400 5700 50  0001 C CNN
+	1    5400 5700
+	1    0    0    -1
+$EndComp
+$Comp
+L power:GND #PWR?
+U 1 1 5CCF9844
+P 5750 5700
+F 0 "#PWR?" H 5750 5450 50  0001 C CNN
+F 1 "GND" H 5755 5527 50  0000 C CNN
+F 2 "" H 5750 5700 50  0001 C CNN
+F 3 "" H 5750 5700 50  0001 C CNN
+	1    5750 5700
+	1    0    0    -1
+$EndComp
+$Comp
+L power:GND #PWR?
+U 1 1 5CCF9887
+P 6100 5700
+F 0 "#PWR?" H 6100 5450 50  0001 C CNN
+F 1 "GND" H 6105 5527 50  0000 C CNN
+F 2 "" H 6100 5700 50  0001 C CNN
+F 3 "" H 6100 5700 50  0001 C CNN
+	1    6100 5700
+	1    0    0    -1
+$EndComp
+$Comp
+L Device:Q_PMOS_DGS Q?
+U 1 1 5CD1F1BC
+P 4450 2950
+F 0 "Q?" V 4793 2950 50  0000 C CNN
+F 1 "Q_PMOS_DGS" V 4702 2950 50  0000 C CNN
+F 2 "" H 4650 3050 50  0001 C CNN
+F 3 "~" H 4450 2950 50  0001 C CNN
+	1    4450 2950
+	0    -1   -1   0
+$EndComp
+Wire Wire Line
+	1500 1450 2250 1450
+Connection ~ 2250 1450
+Wire Wire Line
+	1600 3350 2250 3350
+Wire Wire Line
+	4650 2850 4750 2850
+Wire Wire Line
+	4750 2850 4750 2650
+Text Label 4450 3150 3    50   ~ 0
+SWITCH
+$Comp
+L Connector_Generic:Conn_01x02 J?
+U 1 1 5CD3456E
+P 1350 5150
+F 0 "J?" H 1270 5367 50  0000 C CNN
+F 1 "Conn_01x02" H 1270 5276 50  0000 C CNN
+F 2 "" H 1350 5150 50  0001 C CNN
+F 3 "~" H 1350 5150 50  0001 C CNN
+	1    1350 5150
+	-1   0    0    -1
+$EndComp
+$Comp
+L power:+24V #PWR?
+U 1 1 5CD345DC
+P 1750 5000
+F 0 "#PWR?" H 1750 4850 50  0001 C CNN
+F 1 "+24V" H 1765 5173 50  0000 C CNN
+F 2 "" H 1750 5000 50  0001 C CNN
+F 3 "" H 1750 5000 50  0001 C CNN
+	1    1750 5000
+	1    0    0    -1
+$EndComp
+Wire Wire Line
+	1750 5000 1750 5150
+Wire Wire Line
+	1750 5150 1550 5150
+Text Label 1750 5250 0    50   ~ 0
+SWITCH
+Wire Wire Line
+	1750 5250 1650 5250
+$Comp
+L Device:R R?
+U 1 1 5CD38F7A
+P 1650 5400
+F 0 "R?" H 1720 5446 50  0000 L CNN
+F 1 "10k" H 1720 5355 50  0000 L CNN
+F 2 "" V 1580 5400 50  0001 C CNN
+F 3 "~" H 1650 5400 50  0001 C CNN
+	1    1650 5400
+	1    0    0    -1
+$EndComp
+Connection ~ 1650 5250
+Wire Wire Line
+	1650 5250 1550 5250
+$Comp
+L power:GND #PWR?
+U 1 1 5CD39002
+P 1650 5550
+F 0 "#PWR?" H 1650 5300 50  0001 C CNN
+F 1 "GND" H 1655 5377 50  0000 C CNN
+F 2 "" H 1650 5550 50  0001 C CNN
+F 3 "" H 1650 5550 50  0001 C CNN
+	1    1650 5550
+	1    0    0    -1
+$EndComp
+Text Notes 1300 5950 0    50   ~ 0
+POWER SWITCH
 $EndSCHEMATC

Commit message: addressing aarons comments for radio board
Parts:
- removed Q?: Q_PMOS_DGS, symbol Device:Q_PMOS_DGS
- added Q? (x2): Q_PMOS_DGS, symbol Device:Q_PMOS_DGS
- C1, C2, C3, C4, C5, C6, C7: footprint (none) -> Capacitors_SMD:C_0603_HandSoldering
- C8: renamed from C?; footprint (none) -> Capacitors_SMD:C_0603_HandSoldering
- gave numbers to parts that had none: 12
Connections:
- wire segments 93 -> 96
Other:
- moved on the sheet: U3

Commit message: fixed battery board comments
Parts:
- removed C8: 0.1uF, Capacitors_SMD:C_0603_HandSoldering, symbol Device:C
- removed Q?: Q_PMOS_DGS, symbol Device:Q_PMOS_DGS
- removed U5: TLA2022IRUGT, symbol Payload_ADC:TLA2022IRUGT
- added F1, F2: Fuse, symbol Device:Fuse
- added U5: MAX11645EUA, symbol Payload_ADC:MAX11645EUA
- gave numbers to parts that had none: 1
Connections:
- wire segments 96 -> 95
- no-connect marks 11 -> 10
Other:
- note added: "+24V source 1"
- note added: "+24V source 2"
- note added: "EXPERIMENT POWER"
- note removed: "+24V source"
Changed lines of the file:
@@
 	1400 5250 1400 5400
 Text Notes 800  1150 0    50   ~ 0
-+24V source
++24V source 1
 $Comp
 L Regulator_Switching:TSR_1-2433 U3
@@
 Wire Wire Line
 	6500 2700 6700 2700
-$Comp
-L Payload_ADC:TLA2022IRUGT U5
-U 1 1 5CA2B004
-P 6200 5400
-F 0 "U5" H 6225 5825 50  0000 C CNN
-F 1 "TLA2022IRUGT" H 6225 5734 50  0000 C CNN
-F 2 "" H 6200 5300 50  0001 C CNN
-F 3 "" H 6200 5300 50  0001 C CNN
-	1    6200 5400
-	1    0    0    -1
-$EndComp
-$Comp
-L Device:C C8
-U 1 1 5CA2B394
-P 7000 5650
-F 0 "C8" H 7115 5696 50  0000 L CNN
-F 1 "0.1uF" H 7115 5605 50  0000 L CNN
-F 2 "Capacitors_SMD:C_0603_HandSoldering" H 7038 5500 50  0001 C CNN
-F 3 "~" H 7000 5650 50  0001 C CNN
-	1    7000 5650
-	1    0    0    -1
-$EndComp
-Wire Wire Line
-	6750 5400 7000 5400
-Wire Wire Line
-	7000 5400 7000 5500
-$Comp
-L power:GND #PWR0101
-U 1 1 5CA2C8D2
-P 7000 5800
-F 0 "#PWR0101" H 7000 5550 50  0001 C CNN
-F 1 "GND" H 7005 5627 50  0000 C CNN
-F 2 "" H 7000 5800 50  0001 C CNN
-F 3 "" H 7000 5800 50  0001 C CNN
-	1    7000 5800
-	1    0    0    -1
-$EndComp
-NoConn ~ 6750 5600
-NoConn ~ 6750 5500
-NoConn ~ 5700 5300
-$Comp
-L power:+3V3 #PWR0102
-U 1 1 5CA3079D
-P 7000 5100
-F 0 "#PWR0102" H 7000 4950 50  0001 C CNN
-F 1 "+3V3" H 7015 5273 50  0000 C CNN
-F 2 "" H 7000 5100 50  0001 C CNN
-F 3 "" H 7000 5100 50  0001 C CNN
-	1    7000 5100
-	1    0    0    -1
-$EndComp
-Wire Wire Line
-	7000 5100 7000 5400
-Connection ~ 7000 5400
-Text Label 6750 5200 0    50   ~ 0
-SCL
-Text Label 6750 5300 0    50   ~ 0
-SDA
-$Comp
-L power:GND #PWR0103
-U 1 1 5CA3218A
-P 5400 5750
-F 0 "#PWR0103" H 5400 5500 50  0001 C CNN
-F 1 "GND" H 5405 5577 50  0000 C CNN
-F 2 "" H 5400 5750 50  0001 C CNN
-F 3 "" H 5400 5750 50  0001 C CNN
-	1    5400 5750
-	1    0    0    -1
-$EndComp
-Wire Wire Line
-	5400 5750 5400 5400
-Wire Wire Line
-	5400 5400 5700 5400
-Wire Wire Line
-	5700 5200 5400 5200
-Wire Wire Line
-	5400 5200 5400 5400
-Connection ~ 5400 5400
-Text Label 5700 5500 2    50   ~ 0
+Text Label 6000 4900 2    50   ~ 0
 CURR_1
-Text Label 5700 5600 2    50   ~ 0
+Text Label 6000 5000 2    50   ~ 0
 CURR_2
 Text Label 2600 4050 2    50   ~ 0
@@
 Text Notes 900  7450 0    50   ~ 0
 POWER SWITCH
-$Comp
-L Device:Q_PMOS_DGS Q?
-U 1 1 5CD4BCBF
-P 1700 1550
-F 0 "Q?" V 2043 1550 50  0000 C CNN
-F 1 "Q_PMOS_DGS" V 1952 1550 50  0000 C CNN
-F 2 "" H 1900 1650 50  0001 C CNN
-F 3 "~" H 1700 1550 50  0001 C CNN
-	1    1700 1550
+Wire Wire Line
+	2250 1750 2250 2950
+Wire Wire Line
+	4050 2950 4050 3900
+Wire Wire Line
+	1250 4700 1700 4700
+Wire Wire Line
+	1100 1450 1600 1450
+$Comp
+L Device:Q_PMOS_DGS Q2
+U 1 1 5CD7D860
+P 5350 2800
+F 0 "Q2" V 5693 2800 50  0000 C CNN
+F 1 "Q_PMOS_DGS" V 5602 2800 50  0000 C CNN
+F 2 "" H 5550 2900 50  0001 C CNN
+F 3 "~" H 5350 2800 50  0001 C CNN
+	1    5350 2800
 	0    -1   -1   0
 $EndComp
 Wire Wire Line
-	2250 1750 2250 2950
-Wire Wire Line
-	4050 2950 4050 3900
-Wire Wire Line
-	1250 4700 1600 4700
-Wire Wire Line
-	1100 1450 1500 1450
-Wire Wire Line
-	1900 1450 2250 1450
-Text Label 1700 1750 3    50   ~ 0
-SWITCH
-$Comp
-L Device:Q_PMOS_DGS Q?
-U 1 1 5CD7D860
-P 1800 4800
-F 0 "Q?" V 2143 4800 50  0000 C CNN
-F 1 "Q_PMOS_DGS" V 2052 4800 50  0000 C CNN
-F 2 "" H 2000 4900 50  0001 C CNN
-F 3 "~" H 1800 4800 50  0001 C CNN
-	1    1800 4800
-	0    -1   -1   0
-$EndComp
-Text Label 1800 5000 3    50   ~ 0
-SWITCH
-Wire Wire Line
-	2000 4700 2250 4700
-Wire Wire Line
 	2250 2950 4050 2950
 $Comp
-L power:+24V #PWR?
+L power:+24V #PWR011
 U 1 1 5CDAC21E
 P 1300 6550
-F 0 "#PWR?" H 1300 6400 50  0001 C CNN
+F 0 "#PWR011" H 1300 6400 50  0001 C CNN
 F 1 "+24V" H 1315 6723 50  0000 C CNN
 F 2 "" H 1300 6550 50  0001 C CNN
@@
 	1300 6550 1300 6650
 $Comp
-L power:+24V #PWR?
+L power:+24V #PWR012
 U 1 1 5CDB4642
 P 4950 2450
-F 0 "#PWR?" H 4950 2300 50  0001 C CNN
+F 0 "#PWR012" H 4950 2300 50  0001 C CNN
 F 1 "+24V" H 4965 2623 50  0000 C CNN
 F 2 "" H 4950 2450 50  0001 C CNN
@@
 	7500 2700 7950 2700
 $Comp
-L power:+3V3 #PWR?
+L power:+3V3 #PWR026
 U 1 1 5CA6E329
 P 7950 2600
-F 0 "#PWR?" H 7950 2450 50  0001 C CNN
+F 0 "#PWR026" H 7950 2450 50  0001 C CNN
 F 1 "+3V3" H 7965 2773 50  0000 C CNN
 F 2 "" H 7950 2600 50  0001 C CNN
@@
 Wire Wire Line
 	7950 2600 7950 2700
-Connection ~ 4950 3600
-Wire Wire Line
-	4950 3600 6500 3600
-Wire Wire Line
-	4950 2700 4950 3600
 Wire Wire Line
 	4250 4200 4950 4200
-Wire Wire Line
-	4950 4200 4950 3600
 Wire Wire Line
 	4950 2450 4950 2700
 Connection ~ 4950 2700
 Wire Wire Line
-	4950 2700 6500 2700
+	4950 2700 5150 2700
+$Comp
+L Payload_ADC:MAX11645EUA U5
+U 1 1 5CA817A4
+P 6450 5050
+F 0 "U5" H 6425 5425 50  0000 C CNN
+F 1 "MAX11645EUA" H 6425 5334 50  0000 C CNN
+F 2 "" H 6450 4900 50  0001 C CNN
+F 3 "" H 6450 4900 50  0001 C CNN
+	1    6450 5050
+	1    0    0    -1
+$EndComp
+NoConn ~ 6000 5200
+NoConn ~ 6000 5100
+$Comp
+L power:+3V3 #PWR017
+U 1 1 5CA89C30
+P 7100 4800
+F 0 "#PWR017" H 7100 4650 50  0001 C CNN
+F 1 "+3V3" H 7115 4973 50  0000 C CNN
+F 2 "" H 7100 4800 50  0001 C CNN
+F 3 "" H 7100 4800 50  0001 C CNN
+	1    7100 4800
+	1    0    0    -1
+$EndComp
+Wire Wire Line
+	7100 4800 7100 4900
+Wire Wire Line
+	7100 4900 6850 4900
+$Comp
+L power:GND #PWR025
+U 1 1 5CA8C5C6
+P 7100 5250
+F 0 "#PWR025" H 7100 5000 50  0001 C CNN
+F 1 "GND" H 7105 5077 50  0000 C CNN
+F 2 "" H 7100 5250 50  0001 C CNN
+F 3 "" H 7100 5250 50  0001 C CNN
+	1    7100 5250
+	1    0    0    -1
+$EndComp
+Wire Wire Line
+	6850 5000 7100 5000
+Wire Wire Line
+	7100 5000 7100 5250
+Text Label 6850 5200 0    50   ~ 0
+SCL
+Text Label 6850 5100 0    50   ~ 0
+SDA
+Text Notes 900  4400 0    50   ~ 0
++24V source 2
+Text Notes 9850 4050 0    50   ~ 0
+EXPERIMENT POWER
+$Comp
+L Device:Fuse F1
+U 1 1 5CA9F3FE
+P 1750 1450
+F 0 "F1" V 1553 1450 50  0000 C CNN
+F 1 "Fuse" V 1644 1450 50  0000 C CNN
+F 2 "" V 1680 1450 50  0001 C CNN
+F 3 "~" H 1750 1450 50  0001 C CNN
+	1    1750 1450
+	0    1    1    0
+$EndComp
+$Comp
+L Device:Fuse F2
+U 1 1 5CAA649E
+P 1850 4700
+F 0 "F2" V 1653 4700 50  0000 C CNN
+F 1 "Fuse" V 1744 4700 50  0000 C CNN
+F 2 "" V 1780 4700 50  0001 C CNN
+F 3 "~" H 1850 4700 50  0001 C CNN
+	1    1850 4700
+	0    1    1    0
+$EndComp
+Wire Wire Line
+	5550 2700 5800 2700
+Wire Wire Line
+	5800 2700 5800 3600
+Connection ~ 5800 2700
+Wire Wire Line
+	5800 2700 6500 2700
+Wire Wire Line
+	5800 3600 6500 3600
+Wire Wire Line
+	4950 2700 4950 4200
+Text Label 5350 3000 3    50   ~ 0
+SWITCH
+Wire Wire Line
+	1900 1450 2250 1450
+Wire Wire Line
+	2000 4700 2250 4700
 $EndSCHEMATC
