File: Hardware/Flight/Battery Board/Battery Board/Battery Board.sch (KiCad schematic (older format))
At the start: 34 parts, among them J1 Conn_01x02, J2 Conn_01x02, J3 Conn_01x02, J4 Conn_01x02, J5 Conn_01x02, J6 Conn_01x02, J7 Bus_Connector, Q2 Q_PMOS_DGS, U1 ACS711KEXLT-31AB-T, U2 ACS711KEXLT-31AB-T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

Commit message: fixed changes in experiment board
Parts:
- gave numbers to parts that had none: 2
Changed lines of the file:
@@
 	2000 4700 2250 4700
 $Comp
-L Device:C C?
+L Device:C C8
 U 1 1 5CF7D729
 P 7400 5100
-F 0 "C?" H 7515 5146 50  0000 L CNN
+F 0 "C8" H 7515 5146 50  0000 L CNN
 F 1 "4.7uF" H 7515 5055 50  0000 L CNN
 F 2 "" H 7438 4950 50  0001 C CNN
@@
 $EndComp
 $Comp
-L Device:C C?
+L Device:C C9
 U 1 1 5CF7D7A7
 P 7850 5100
-F 0 "C?" H 7965 5146 50  0000 L CNN
+F 0 "C9" H 7965 5146 50  0000 L CNN
 F 1 "0.1uF" H 7965 5055 50  0000 L CNN
 F 2 "" H 7888 4950 50  0001 C CNN
@@
 Connection ~ 7400 4900
 $Comp
-L power:GND #PWR?
+L power:GND #PWR027
 U 1 1 5CF8E1FA
 P 7400 5250
-F 0 "#PWR?" H 7400 5000 50  0001 C CNN
+F 0 "#PWR027" H 7400 5000 50  0001 C CNN
 F 1 "GND" H 7405 5077 50  0000 C CNN
 F 2 "" H 7400 5250 50  0001 C CNN
@@
 $EndComp
 $Comp
-L power:GND #PWR?
+L power:GND #PWR028
 U 1 1 5CF8E249
 P 7850 5250
-F 0 "#PWR?" H 7850 5000 50  0001 C CNN
+F 0 "#PWR028" H 7850 5000 50  0001 C CNN
 F 1 "GND" H 7855 5077 50  0000 C CNN
 F 2 "" H 7850 5250 50  0001 C CNN
