File: Hardware/Flight/Experiment Board/Experiment Board.sch (KiCad schematic (older format))
At the start: 30 parts, among them J1 Conn_01x05_Female, J2 Conn_01x05, J4 Conn_01x02, U1 PIC18F26K83, Y1 Crystal

Commit message: finished schematic for experiment board
Parts:
- removed C5, C? (x3): 1000uF, symbol Device:C
- removed J2: Conn_01x05, symbol Connector_Generic:Conn_01x05
- removed J4, J?: Conn_01x02, symbol Connector_Generic:Conn_01x02
- removed JP? (x12): Jumper, symbol Device:Jumper
- removed L3, L4, L? (x2): 10uH, symbol pspice:INDUCTOR
- added C4: 100nF, symbol Device:C
- added J2, J6, J7: Conn_01x02, symbol Connector_Generic:Conn_01x02
- added J3: Conn_01x20, symbol Connector_Generic:Conn_01x20
- added J4, J5: Conn_01x03, symbol Connector_Generic:Conn_01x03
- added U4: LSM6DS3, Package_LGA:LGA-14_3x2.5mm_P0.5mm_LayoutBorder3x4y, symbol Sensor_Motion:LSM6DS3
Connections:
- net labels added: +3V3, ADC1, ADC2, CURR_1, CURR_2, CURR_3, CURR_4, FAULT3, FAULT4, FAULT5, FAULT6
- wire segments 112 -> 76
- no-connect marks 0 -> 2
Other:
- note added: "BUS INPUT"
- note added: "FLOW SENSORS"
- note added: "PIC PROGRAMMER"
- note removed: "H BRIDGE"
- note removed: "SOLENOID 1"
- note removed: "SOLENOID 2"

Commit message: added battery board + ADCs for experiment board
Parts:
- added C? (x2): 0.1uF, symbol Device:C
- added U?: ADS1015IDGS, Package_SO:TSSOP-10_3x3mm_P0.5mm, symbol Analog_ADC:ADS1015IDGS
- added U?: TLA2022IRUGT, symbol Payload_ADC:TLA2022IRUGT
Connections:
- net labels removed: CURR_1, CURR_2, CURR_3, CURR_4
- wire segments 76 -> 97
- no-connect marks 2 -> 5
Other:
- note added: "5V on flow sensors required\nadd level shifting\ncheck adc datasheet to confirm support"
Changed lines of the file:
@@
 Text Label 1350 3400 0    50   ~ 0
 ADC2
-Text Label 1350 3500 0    50   ~ 0
-CURR_1
-Text Label 1350 3600 0    50   ~ 0
-CURR_2
-Text Label 1350 3700 0    50   ~ 0
-CURR_3
-Text Label 1350 3800 0    50   ~ 0
-CURR_4
-Text Label 7450 2900 0    50   ~ 0
-CURR_1
-Text Label 7450 3300 0    50   ~ 0
-CURR_2
-Text Label 7400 4400 0    50   ~ 0
-CURR_3
-Text Label 7400 4800 0    50   ~ 0
-CURR_4
 Text Label 1350 4800 0    50   ~ 0
 SCL
@@
 Text Label 7400 4900 0    50   ~ 0
 FAULT6
+$Comp
+L Analog_ADC:ADS1015IDGS U?
+U 1 1 5C9FA6D0
+P 9350 3800
+F 0 "U?" H 9050 4500 50  0000 C CNN
+F 1 "ADS1015IDGS" H 9050 4350 50  0000 C CNN
+F 2 "Package_SO:TSSOP-10_3x3mm_P0.5mm" H 9350 3300 50  0001 C CNN
+F 3 "http://www.ti.com/lit/ds/symlink/ads1015.pdf" H 9300 2900 50  0001 C CNN
+	1    9350 3800
+	1    0    0    -1
+$EndComp
+$Comp
+L power:+3V3 #PWR?
+U 1 1 5C9FA956
+P 9350 3100
+F 0 "#PWR?" H 9350 2950 50  0001 C CNN
+F 1 "+3V3" H 9365 3273 50  0000 C CNN
+F 2 "" H 9350 3100 50  0001 C CNN
+F 3 "" H 9350 3100 50  0001 C CNN
+	1    9350 3100
+	1    0    0    -1
+$EndComp
+Wire Wire Line
+	9350 3100 9350 3200
+$Comp
+L power:+3V3 #PWR?
+U 1 1 5C9FC444
+P 10150 3750
+F 0 "#PWR?" H 10150 3600 50  0001 C CNN
+F 1 "+3V3" H 10165 3923 50  0000 C CNN
+F 2 "" H 10150 3750 50  0001 C CNN
+F 3 "" H 10150 3750 50  0001 C CNN
+	1    10150 3750
+	1    0    0    -1
+$EndComp
+Wire Wire Line
+	10150 3750 10150 4000
+Wire Wire Line
+	10150 4000 9750 4000
+Text Label 9750 3800 0    50   ~ 0
+SCL
+Text Label 9750 3900 0    50   ~ 0
+SDA
+$Comp
+L Device:C C?
+U 1 1 5C9FE1D0
+P 9600 3200
+F 0 "C?" V 9348 3200 50  0000 C CNN
+F 1 "0.1uF" V 9439 3200 50  0000 C CNN
+F 2 "" H 9638 3050 50  0001 C CNN
+F 3 "~" H 9600 3200 50  0001 C CNN
+	1    9600 3200
+	0    1    1    0
+$EndComp
+Wire Wire Line
+	9450 3200 9350 3200
+Connection ~ 9350 3200
+Wire Wire Line
+	9350 3200 9350 3300
+$Comp
+L power:GND #PWR?
+U 1 1 5C9FFAB0
+P 9800 3250
+F 0 "#PWR?" H 9800 3000 50  0001 C CNN
+F 1 "GND" H 9805 3077 50  0000 C CNN
+F 2 "" H 9800 3250 50  0001 C CNN
+F 3 "" H 9800 3250 50  0001 C CNN
+	1    9800 3250
+	1    0    0    -1
+$EndComp
+Wire Wire Line
+	9750 3200 9800 3200
+Wire Wire Line
+	9800 3200 9800 3250
+Wire Wire Line
+	7400 4400 8650 4400
+Wire Wire Line
+	8650 4400 8650 3900
+Wire Wire Line
+	8650 3900 8950 3900
+Wire Wire Line
+	7400 4800 8750 4800
+Wire Wire Line
+	8750 4800 8750 4000
+Wire Wire Line
+	8750 4000 8950 4000
+Wire Wire Line
+	7450 2900 8750 2900
+Wire Wire Line
+	8950 3700 8750 3700
+Wire Wire Line
+	8750 3700 8750 2900
+Wire Wire Line
+	8950 3800 8650 3800
+Wire Wire Line
+	8650 3800 8650 3300
+Wire Wire Line
+	8650 3300 7450 3300
+$Comp
+L power:GND #PWR?
+U 1 1 5CA0F165
+P 9350 4200
+F 0 "#PWR?" H 9350 3950 50  0001 C CNN
+F 1 "GND" H 9355 4027 50  0000 C CNN
+F 2 "" H 9350 4200 50  0001 C CNN
+F 3 "" H 9350 4200 50  0001 C CNN
+	1    9350 4200
+	1    0    0    -1
+$EndComp
+$Comp
+L Payload_ADC:TLA2022IRUGT U?
+U 1 1 5CA119B1
+P 5550 5600
+F 0 "U?" H 5575 6025 50  0000 C CNN
+F 1 "TLA2022IRUGT" H 5575 5934 50  0000 C CNN
+F 2 "" H 5550 5500 50  0001 C CNN
+F 3 "" H 5550 5500 50  0001 C CNN
+	1    5550 5600
+	1    0    0    -1
+$EndComp
+NoConn ~ 6100 5700
+NoConn ~ 6100 5800
+NoConn ~ 5050 5500
+Wire Wire Line
+	6350 5400 6350 5600
+$Comp
+L Device:C C?
+U 1 1 5CA1C4CB
+P 6350 5750
+F 0 "C?" H 6465 5796 50  0000 L CNN
+F 1 "0.1uF" H 6465 5705 50  0000 L CNN
+F 2 "" H 6388 5600 50  0001 C CNN
+F 3 "~" H 6350 5750 50  0001 C CNN
+	1    6350 5750
+	1    0    0    -1
+$EndComp
+Connection ~ 6350 5600
+$Comp
+L power:GND #PWR?
+U 1 1 5CA1C5C1
+P 6350 5900
+F 0 "#PWR?" H 6350 5650 50  0001 C CNN
+F 1 "GND" H 6355 5727 50  0000 C CNN
+F 2 "" H 6350 5900 50  0001 C CNN
+F 3 "" H 6350 5900 50  0001 C CNN
+	1    6350 5900
+	1    0    0    -1
+$EndComp
+Wire Wire Line
+	6100 5600 6350 5600
+Text Label 6100 5400 0    50   ~ 0
+SCL
+Text Label 6100 5500 0    50   ~ 0
+SDA
+$Comp
+L power:+5V #PWR?
+U 1 1 5CA25E04
+P 6350 5400
+F 0 "#PWR?" H 6350 5250 50  0001 C CNN
+F 1 "+5V" H 6365 5573 50  0000 C CNN
+F 2 "" H 6350 5400 50  0001 C CNN
+F 3 "" H 6350 5400 50  0001 C CNN
+	1    6350 5400
+	1    0    0    -1
+$EndComp
+Text Notes 6700 5750 0    50   ~ 0
+5V on flow sensors required\nadd level shifting\ncheck adc datasheet to confirm support
 $EndSCHEMATC

Commit message: connected GPIO to ARM board
Connections:
- net labels added: SCL_5
- net labels removed: ADC1, ADC2, OSC1, OSC2
- wire segments 97 -> 128
Other:
- note added: "SOLENOID 1"
- note added: "SOLENOID 2"
- note removed: "5V on flow sensors required\nadd level shifting\ncheck adc datasheet to confirm support"

Commit message: updated battery, experiment board. Added temp sensor to ARM board
Parts:
- removed J3: Conn_01x20, symbol Connector_Generic:Conn_01x20
- removed U1: PIC18F26K83, symbol canhw:PIC18F26K83
- added J?: Bus_Connector, symbol Payload_Connectors:Bus_Connector
- added U?: PICLF26K83, symbol canhw:PICLF26K83
- C3: value C -> 0.1uF
Connections:
- net labels added: ~FAULT3, ~FAULT4, ~FAULT5, ~FAULT6
- net labels removed: FAULT3, FAULT4, FAULT5, FAULT6
Changed lines of the file:
@@
 $EndDescr
-$Comp
-L canhw:PIC18F26K83 U1
-U 1 1 5C95C4B4
-P 4500 4100
-F 0 "U1" H 4475 5015 50  0000 C CNN
-F 1 "PIC18F26K83" H 4475 4924 50  0000 C CNN
-F 2 "" H 4950 4100 50  0001 C CNN
-F 3 "http://ww1.microchip.com/downloads/en/DeviceDoc/40001943A.pdf" H 4950 4100 50  0001 C CNN
-	1    4500 4100
-	1    0    0    -1
-$EndComp
 $Comp
 L Device:R R1
@@
 Connection ~ 3450 3450
 $Comp
-L power:+5V #PWR06
-U 1 1 5C95C5C8
-P 3450 3150
-F 0 "#PWR06" H 3450 3000 50  0001 C CNN
-F 1 "+5V" H 3465 3323 50  0000 C CNN
-F 2 "" H 3450 3150 50  0001 C CNN
-F 3 "" H 3450 3150 50  0001 C CNN
-	1    3450 3150
-	1    0    0    -1
-$EndComp
-$Comp
 L Device:C C3
 U 1 1 5C95C615
 P 5200 2850
 F 0 "C3" V 4948 2850 50  0000 C CNN
-F 1 "C" V 5039 2850 50  0000 C CNN
+F 1 "0.1uF" V 5039 2850 50  0000 C CNN
 F 2 "" H 5238 2700 50  0001 C CNN
 F 3 "~" H 5200 2850 50  0001 C CNN
@@
 Wire Wire Line
 	4950 2850 5050 2850
-$Comp
-L power:+5V #PWR08
-U 1 1 5C95C6D1
-P 5350 2800
-F 0 "#PWR08" H 5350 2650 50  0001 C CNN
-F 1 "+5V" H 5365 2973 50  0000 C CNN
-F 2 "" H 5350 2800 50  0001 C CNN
-F 3 "" H 5350 2800 50  0001 C CNN
-	1    5350 2800
-	1    0    0    -1
-$EndComp
 Wire Wire Line
 	5350 2800 5350 2850
@@
 F9 "I2L" I L 6350 3450 50
 F10 "FAULT1" I L 6350 3200 50
-F11 "FAULT2" I R 7000 2900 50
-F12 "FAULT3" I R 7000 3500 50
+F11 "~FAULT2" I R 7000 2900 50
+F12 "~FAULT3" I R 7000 3500 50
 $EndSheet
 $Comp
@@
 F9 "I2L" I L 6300 4950 50
 F10 "FAULT1" I L 6300 4700 50
-F11 "FAULT2" I R 6950 4400 50
-F12 "FAULT3" I R 6950 5000 50
+F11 "~FAULT2" I R 6950 4400 50
+F12 "~FAULT3" I R 6950 5000 50
 $EndSheet
 $Comp
@@
 Wire Wire Line
 	5950 3950 5950 4450
-$Comp
-L Connector_Generic:Conn_01x20 J3
-U 1 1 5CCD12DD
-P 1150 4100
-F 0 "J3" H 1070 2875 50  0000 C CNN
-F 1 "Conn_01x20" H 1070 2966 50  0000 C CNN
-F 2 "" H 1150 4100 50  0001 C CNN
-F 3 "~" H 1150 4100 50  0001 C CNN
-	1    1150 4100
-	-1   0    0    1
-$EndComp
 $Comp
 L Connector_Generic:Conn_01x02 J2
@@
 	4550 950  4550 1100
 Text Label 3750 3750 2    50   ~ 0
-FAULT3
+~FAULT3
 Text Label 3750 3850 2    50   ~ 0
-FAULT4
+~FAULT4
 Text Label 3750 3950 2    50   ~ 0
-FAULT5
+~FAULT5
 Text Label 3750 4050 2    50   ~ 0
-FAULT6
+~FAULT6
 Text Label 7000 2900 0    50   ~ 0
-FAULT3
+~FAULT3
 Text Label 7000 3500 0    50   ~ 0
-FAULT4
+~FAULT4
 Text Label 6950 4400 0    50   ~ 0
-FAULT5
+~FAULT5
 Text Label 6950 5000 0    50   ~ 0
-FAULT6
+~FAULT6
 $Comp
 L Analog_ADC:ADS1015IDGS U?
@@
 	3350 4250 3350 4850
 Wire Wire Line
-	3750 4150 2850 4150
-Wire Wire Line
 	2850 4150 2850 4850
+$Comp
+L Payload_Connectors:Bus_Connector J?
+U 1 1 5CC8A777
+P 1150 4100
+F 0 "J?" H 961 5325 50  0000 C CNN
+F 1 "Bus_Connector" H 961 5234 50  0000 C CNN
+F 2 "" H 1250 4850 50  0001 C CNN
+F 3 "" H 1250 4850 50  0001 C CNN
+	1    1150 4100
+	1    0    0    -1
+$EndComp
+$Comp
+L canhw:PICLF26K83 U?
+U 1 1 5CC984D5
+P 4500 4100
+F 0 "U?" H 4475 5015 50  0000 C CNN
+F 1 "PICLF26K83" H 4475 4924 50  0000 C CNN
+F 2 "" H 4950 4100 50  0001 C CNN
+F 3 "http://ww1.microchip.com/downloads/en/DeviceDoc/40001943A.pdf" H 4950 4100 50  0001 C CNN
+	1    4500 4100
+	1    0    0    -1
+$EndComp
+$Comp
+L power:+3V3 #PWR?
+U 1 1 5CC98691
+P 3450 3150
+F 0 "#PWR?" H 3450 3000 50  0001 C CNN
+F 1 "+3V3" H 3465 3323 50  0000 C CNN
+F 2 "" H 3450 3150 50  0001 C CNN
+F 3 "" H 3450 3150 50  0001 C CNN
+	1    3450 3150
+	1    0    0    -1
+$EndComp
+$Comp
+L power:+3V3 #PWR?
+U 1 1 5CC986C2
+P 5350 2800
+F 0 "#PWR?" H 5350 2650 50  0001 C CNN
+F 1 "+3V3" H 5365 2973 50  0000 C CNN
+F 2 "" H 5350 2800 50  0001 C CNN
+F 3 "" H 5350 2800 50  0001 C CNN
+	1    5350 2800
+	1    0    0    -1
+$EndComp
+Wire Wire Line
+	2850 4150 3750 4150
 $EndSCHEMATC

Commit message: addressed Alex's ARM review comments
Parts:
- added D? (x3): LED, symbol Device:LED
- added R? (x3): 70, symbol Device:R
Connections:
- net labels added: LED_1, LED_2, LED_3
- wire segments 128 -> 134
Changed lines of the file:
@@
 Wire Wire Line
 	2850 4150 3750 4150
+$Comp
+L Device:LED D?
+U 1 1 5CA7305B
+P 6400 5800
+F 0 "D?" V 6438 5683 50  0000 R CNN
+F 1 "LED" V 6347 5683 50  0000 R CNN
+F 2 "" H 6400 5800 50  0001 C CNN
+F 3 "~" H 6400 5800 50  0001 C CNN
+	1    6400 5800
+	0    -1   -1   0
+$EndComp
+$Comp
+L Device:R R?
+U 1 1 5CA73153
+P 6400 6100
+F 0 "R?" H 6470 6146 50  0000 L CNN
+F 1 "70" H 6470 6055 50  0000 L CNN
+F 2 "" V 6330 6100 50  0001 C CNN
+F 3 "~" H 6400 6100 50  0001 C CNN
+	1    6400 6100
+	1    0    0    -1
+$EndComp
+$Comp
+L power:+3V3 #PWR?
+U 1 1 5CA734E3
+P 6400 5650
+F 0 "#PWR?" H 6400 5500 50  0001 C CNN
+F 1 "+3V3" H 6415 5823 50  0000 C CNN
+F 2 "" H 6400 5650 50  0001 C CNN
+F 3 "" H 6400 5650 50  0001 C CNN
+	1    6400 5650
+	1    0    0    -1
+$EndComp
+Text Label 6350 6350 2    50   ~ 0
+LED_1
+Wire Wire Line
+	6350 6350 6400 6350
+Wire Wire Line
+	6400 6350 6400 6250
+$Comp
+L Device:LED D?
+U 1 1 5CA7C5B4
+P 6800 5800
+F 0 "D?" V 6838 5683 50  0000 R CNN
+F 1 "LED" V 6747 5683 50  0000 R CNN
+F 2 "" H 6800 5800 50  0001 C CNN
+F 3 "~" H 6800 5800 50  0001 C CNN
+	1    6800 5800
+	0    -1   -1   0
+$EndComp
+$Comp
+L Device:R R?
+U 1 1 5CA7C5BA
+P 6800 6100
+F 0 "R?" H 6870 6146 50  0000 L CNN
+F 1 "70" H 6870 6055 50  0000 L CNN
+F 2 "" V 6730 6100 50  0001 C CNN
+F 3 "~" H 6800 6100 50  0001 C CNN
+	1    6800 6100
+	1    0    0    -1
+$EndComp
+$Comp
+L power:+3V3 #PWR?
+U 1 1 5CA7C5C0
+P 6800 5650
+F 0 "#PWR?" H 6800 5500 50  0001 C CNN
+F 1 "+3V3" H 6815 5823 50  0000 C CNN
+F 2 "" H 6800 5650 50  0001 C CNN
+F 3 "" H 6800 5650 50  0001 C CNN
+	1    6800 5650
+	1    0    0    -1
+$EndComp
+Text Label 6750 6350 2    50   ~ 0
+LED_2
+Wire Wire Line
+	6750 6350 6800 6350
+Wire Wire Line
+	6800 6350 6800 6250
+$Comp
+L Device:LED D?
+U 1 1 5CA80FE8
+P 7200 5800
+F 0 "D?" V 7238 5683 50  0000 R CNN
+F 1 "LED" V 7147 5683 50  0000 R CNN
+F 2 "" H 7200 5800 50  0001 C CNN
+F 3 "~" H 7200 5800 50  0001 C CNN
+	1    7200 5800
+	0    -1   -1   0
+$EndComp
+$Comp
+L Device:R R?
+U 1 1 5CA80FEE
+P 7200 6100
+F 0 "R?" H 7270 6146 50  0000 L CNN
+F 1 "70" H 7270 6055 50  0000 L CNN
+F 2 "" V 7130 6100 50  0001 C CNN
+F 3 "~" H 7200 6100 50  0001 C CNN
+	1    7200 6100
+	1    0    0    -1
+$EndComp
+$Comp
+L power:+3V3 #PWR?
+U 1 1 5CA80FF4
+P 7200 5650
+F 0 "#PWR?" H 7200 5500 50  0001 C CNN
+F 1 "+3V3" H 7215 5823 50  0000 C CNN
+F 2 "" H 7200 5650 50  0001 C CNN
+F 3 "" H 7200 5650 50  0001 C CNN
+	1    7200 5650
+	1    0    0    -1
+$EndComp
+Text Label 7150 6350 2    50   ~ 0
+LED_3
+Wire Wire Line
+	7150 6350 7200 6350
+Wire Wire Line
+	7200 6350 7200 6250
+Text Label 5200 4350 0    50   ~ 0
+LED_1
+Text Label 5200 4450 0    50   ~ 0
+LED_2
+Text Label 5200 4550 0    50   ~ 0
+LED_3
 $EndSCHEMATC

Commit message: fixed battery board comments
Parts:
- removed C?: 0.1uF, symbol Device:C
- removed U?: ADS1015IDGS, Package_SO:TSSOP-10_3x3mm_P0.5mm, symbol Analog_ADC:ADS1015IDGS
- added C15, C17: 0.1uF, symbol Device:C
- added C16: 1nF, symbol Device:C
- added R3: 1k, symbol Device:R
- added U7: ACS711KEXLT-31AB-T, symbol Payload_Sensors:ACS711KEXLT-31AB-T
- added U8: TLA2022IRUGT, symbol Payload_ADC:TLA2022IRUGT
- gave numbers to parts that had none: 10
Connections:
- net labels added: +24_IN
- net labels removed: ~FAULT4, ~FAULT5, ~FAULT6
- wire segments 134 -> 143
- no-connect marks 5 -> 13

Commit message: swapped ADC package on experiment board
Parts:
- removed C17: 0.1uF, symbol Device:C
- removed U1, U8: TLA2022IRUGT, symbol Payload_ADC:TLA2022IRUGT
- added C?: 0.1uF, symbol Device:C
- added U?: MAX11644EUA, symbol Payload_ADC:MAX11644EUA
- added U?: MCP3221A5T, symbol Payload_ADC:MCP3221A5T
- C9: value 0.1uF -> 4.7uF
Connections:
- net labels removed: SCL_5
- no-connect marks 13 -> 8
Changed lines of the file:
@@
 Text Label 1400 1150 0    50   ~ 0
 ~MCLR
-$Comp
-L power:+5V #PWR03
-U 1 1 5C95E0EF
-P 1750 1100
-F 0 "#PWR03" H 1750 950 50  0001 C CNN
-F 1 "+5V" H 1765 1273 50  0000 C CNN
-F 2 "" H 1750 1100 50  0001 C CNN
-F 3 "" H 1750 1100 50  0001 C CNN
-	1    1750 1100
-	1    0    0    -1
-$EndComp
 Wire Wire Line
 	1750 1100 1750 1250
@@
 ~FAULT3
 $Comp
-L Payload_ADC:TLA2022IRUGT U1
-U 1 1 5CA119B1
-P 3250 6350
-F 0 "U1" H 3275 6775 50  0000 C CNN
-F 1 "TLA2022IRUGT" H 3275 6684 50  0000 C CNN
-F 2 "" H 3250 6250 50  0001 C CNN
-F 3 "" H 3250 6250 50  0001 C CNN
-	1    3250 6350
-	1    0    0    -1
-$EndComp
-NoConn ~ 3800 6450
-NoConn ~ 3800 6550
-NoConn ~ 2750 6250
-Wire Wire Line
-	4100 5800 4100 6350
-$Comp
 L Device:C C9
 U 1 1 5CA1C4CB
-P 4100 6500
-F 0 "C9" H 4215 6546 50  0000 L CNN
-F 1 "0.1uF" H 4215 6455 50  0000 L CNN
-F 2 "" H 4138 6350 50  0001 C CNN
-F 3 "~" H 4100 6500 50  0001 C CNN
-	1    4100 6500
-	1    0    0    -1
-$EndComp
-Connection ~ 4100 6350
+P 3850 6350
+F 0 "C9" H 3965 6396 50  0000 L CNN
+F 1 "4.7uF" H 3965 6305 50  0000 L CNN
+F 2 "" H 3888 6200 50  0001 C CNN
+F 3 "~" H 3850 6350 50  0001 C CNN
+	1    3850 6350
+	1    0    0    -1
+$EndComp
 $Comp
 L power:GND #PWR027
 U 1 1 5CA1C5C1
-P 4100 6700
-F 0 "#PWR027" H 4100 6450 50  0001 C CNN
-F 1 "GND" H 4105 6527 50  0000 C CNN
-F 2 "" H 4100 6700 50  0001 C CNN
-F 3 "" H 4100 6700 50  0001 C CNN
-	1    4100 6700
-	1    0    0    -1
-$EndComp
-Wire Wire Line
-	3800 6350 4100 6350
+P 3650 6850
+F 0 "#PWR027" H 3650 6600 50  0001 C CNN
+F 1 "GND" H 3655 6677 50  0000 C CNN
+F 2 "" H 3650 6850 50  0001 C CNN
+F 3 "" H 3650 6850 50  0001 C CNN
+	1    3650 6850
+	1    0    0    -1
+$EndComp
 $Comp
 L power:+5V #PWR026
 U 1 1 5CA25E04
-P 4100 5800
-F 0 "#PWR026" H 4100 5650 50  0001 C CNN
-F 1 "+5V" H 4115 5973 50  0000 C CNN
-F 2 "" H 4100 5800 50  0001 C CNN
-F 3 "" H 4100 5800 50  0001 C CNN
-	1    4100 5800
-	1    0    0    -1
-$EndComp
-$Comp
-L power:GND #PWR018
-U 1 1 5CA2E14D
-P 2600 6700
-F 0 "#PWR018" H 2600 6450 50  0001 C CNN
-F 1 "GND" H 2605 6527 50  0000 C CNN
-F 2 "" H 2600 6700 50  0001 C CNN
-F 3 "" H 2600 6700 50  0001 C CNN
-	1    2600 6700
-	1    0    0    -1
-$EndComp
-Wire Wire Line
-	2600 6700 2600 6350
-Wire Wire Line
-	2600 6350 2750 6350
-Text Label 2750 6150 2    50   ~ 0
-SCL_5
+P 3700 6150
+F 0 "#PWR026" H 3700 6000 50  0001 C CNN
+F 1 "+5V" H 3715 6323 50  0000 C CNN
+F 2 "" H 3700 6150 50  0001 C CNN
+F 3 "" H 3700 6150 50  0001 C CNN
+	1    3700 6150
+	1    0    0    -1
+$EndComp
 $Sheet
-S 4850 5900 850  200
+S 4650 6400 850  200
 U 5CA3E00F
 F0 "LogicShifter" 50
 F1 "LogicShifter.sch" 50
-F2 "3v3_DATA" I R 5700 6000 50
-F3 "5_DATA" I L 4850 6000 50
+F2 "3v3_DATA" I R 5500 6500 50
+F3 "5_DATA" I L 4650 6500 50
 $EndSheet
-Text Label 5700 6400 0    50   ~ 0
+Text Label 5500 6500 0    50   ~ 0
 SDA
-Text Label 5700 6000 0    50   ~ 0
+Text Label 5500 6900 0    50   ~ 0
 SCL
 $Sheet
-S 4850 6300 850  200
+S 4650 6800 850  200
 U 5CA45F2C
 F0 "sheet5CA45F2C" 50
 F1 "LogicShifter.sch" 50
-F2 "3v3_DATA" I R 5700 6400 50
-F3 "5_DATA" I L 4850 6400 50
+F2 "3v3_DATA" I R 5500 6900 50
+F3 "5_DATA" I L 4650 6900 50
 $EndSheet
 Wire Wire Line
-	3800 6150 4700 6150
-Wire Wire Line
-	4700 6150 4700 6000
-Wire Wire Line
-	4700 6000 4850 6000
-Wire Wire Line
-	3800 6250 4700 6250
-Wire Wire Line
-	4700 6250 4700 6400
-Wire Wire Line
-	4700 6400 4850 6400
+	3600 6650 4500 6650
+Wire Wire Line
+	4500 6650 4500 6500
+Wire Wire Line
+	4500 6500 4650 6500
+Wire Wire Line
+	3600 6750 4500 6750
+Wire Wire Line
+	4500 6750 4500 6900
+Wire Wire Line
+	4500 6900 4650 6900
 Wire Wire Line
 	1400 5650 1400 5850
@@
 Wire Wire Line
 	2050 6550 2050 7050
-Wire Wire Line
-	4100 6700 4100 6650
 Connection ~ 5350 2850
 Wire Wire Line
@@
 Text Label 1500 2400 0    50   ~ 0
 +24_IN
-$Comp
-L Payload_ADC:TLA2022IRUGT U8
-U 1 1 5CE8F1E1
-P 9900 1350
-F 0 "U8" H 9925 1775 50  0000 C CNN
-F 1 "TLA2022IRUGT" H 9925 1684 50  0000 C CNN
-F 2 "" H 9900 1250 50  0001 C CNN
-F 3 "" H 9900 1250 50  0001 C CNN
-	1    9900 1350
-	1    0    0    -1
-$EndComp
 Wire Wire Line
 	8100 1100 8100 1000
@@
 Wire Wire Line
 	7800 800  9050 800
-NoConn ~ 9400 1450
 $Comp
 L power:GND #PWR048
@@
 $EndComp
 Wire Wire Line
-	9250 1700 9250 1350
+	9250 1700 9250 1450
 Wire Wire Line
 	9250 1350 9400 1350
-NoConn ~ 10450 1450
-NoConn ~ 10450 1550
-NoConn ~ 9400 1250
-Wire Wire Line
-	9250 1150 9400 1150
-Text Label 10450 1150 0    50   ~ 0
+Text Label 10300 1350 0    50   ~ 0
 SCL
-Text Label 10450 1250 0    50   ~ 0
+Text Label 10300 1550 0    50   ~ 0
 SDA
-$Comp
-L power:+3V3 #PWR?
-U 1 1 5CEC15DF
-P 10750 1100
-AR Path="/5CCC856A/5CEC15DF" Ref="#PWR?"  Part="1"
-AR Path="/5CC8A1AA/5CEC15DF" Ref="#PWR?"  Part="1"
-AR Path="/5CEC15DF" Ref="#PWR049"  Part="1"
-F 0 "#PWR049" H 10750 950 50  0001 C CNN
-F 1 "+3V3" H 10765 1273 50  0000 C CNN
-F 2 "" H 10750 1100 50  0001 C CNN
-F 3 "" H 10750 1100 50  0001 C CNN
-	1    10750 1100
-	1    0    0    -1
-$EndComp
-Wire Wire Line
-	10750 1100 10750 1350
-Wire Wire Line
-	10750 1350 10450 1350
-$Comp
-L Device:C C17
-U 1 1 5CEC83D1
-P 10750 1500
-F 0 "C17" H 10865 1546 50  0000 L CNN
-F 1 "0.1uF" H 10865 1455 50  0000 L CNN
-F 2 "" H 10788 1350 50  0001 C CNN
-F 3 "~" H 10750 1500 50  0001 C CNN
-	1    10750 1500
-	1    0    0    -1
-$EndComp
-$Comp
-L power:GND #PWR050
-U 1 1 5CEC83D7
-P 10750 1700
-F 0 "#PWR050" H 10750 1450 50  0001 C CNN
-F 1 "GND" H 10755 1527 50  0000 C CNN
-F 2 "" H 10750 1700 50  0001 C CNN
-F 3 "" H 10750 1700 50  0001 C CNN
-	1    10750 1700
-	1    0    0    -1
-$EndComp
-Wire Wire Line
-	10750 1700 10750 1650
-Connection ~ 10750 1350
 $Comp
 L power:+3V3 #PWR?
@@
 $EndComp
 Wire Wire Line
-	9250 1050 9250 1150
+	9250 1050 9250 1350
 Wire Wire Line
 	6950 4750 7600 4750
@@
 Wire Wire Line
 	7500 3250 7500 3600
+$Comp
+L Payload_ADC:MAX11644EUA U?
+U 1 1 5CAC927A
+P 3200 6600
+F 0 "U?" H 3175 6975 50  0000 C CNN
+F 1 "MAX11644EUA" H 3175 6884 50  0000 C CNN
+F 2 "" H 3200 6450 50  0001 C CNN
+F 3 "" H 3200 6450 50  0001 C CNN
+	1    3200 6600
+	1    0    0    -1
+$EndComp
+Wire Wire Line
+	3700 6150 3700 6450
+Wire Wire Line
+	3700 6450 3600 6450
+$Comp
+L Device:C C?
+U 1 1 5CAD40E9
+P 4300 6350
+F 0 "C?" H 4415 6396 50  0000 L CNN
+F 1 "0.1uF" H 4415 6305 50  0000 L CNN
+F 2 "" H 4338 6200 50  0001 C CNN
+F 3 "~" H 4300 6350 50  0001 C CNN
+	1    4300 6350
+	1    0    0    -1
+$EndComp
+Wire Wire Line
+	3650 6850 3650 6550
+Wire Wire Line
+	3650 6550 3600 6550
+$Comp
+L power:GND #PWR?
+U 1 1 5CAD9054
+P 3850 6500
+F 0 "#PWR?" H 3850 6250 50  0001 C CNN
+F 1 "GND" H 3750 6400 50  0000 C CNN
+F 2 "" H 3850 6500 50  0001 C CNN
+F 3 "" H 3850 6500 50  0001 C CNN
+	1    3850 6500
+	1    0    0    -1
+$EndComp
+$Comp
+L power:GND #PWR?
+U 1 1 5CAD909B
+P 4300 6500
+F 0 "#PWR?" H 4300 6250 50  0001 C CNN
+F 1 "GND" H 4200 6400 50  0000 C CNN
+F 2 "" H 4300 6500 50  0001 C CNN
+F 3 "" H 4300 6500 50  0001 C CNN
+	1    4300 6500
+	1    0    0    -1
+$EndComp
+Wire Wire Line
+	3700 6150 3850 6150
+Wire Wire Line
+	3850 6150 3850 6200
+Connection ~ 3700 6150
+Wire Wire Line
+	3850 6150 4300 6150
+Wire Wire Line
+	4300 6150 4300 6200
+Connection ~ 3850 6150
+NoConn ~ 2750 6650
+NoConn ~ 2750 6750
+$Comp
+L Payload_ADC:MCP3221A5T U?
+U 1 1 5CAF3CEC
+P 9850 1450
+F 0 "U?" H 9850 1775 50  0000 C CNN
+F 1 "MCP3221A5T" H 9850 1684 50  0000 C CNN
+F 2 "" H 9850 1450 50  0001 C CNN
+F 3 "" H 9850 1450 50  0001 C CNN
+	1    9850 1450
+	1    0    0    -1
+$EndComp
+Wire Wire Line
+	9400 1450 9250 1450
+$Comp
+L power:+3V3 #PWR?
+U 1 1 5CB1E389
+P 1750 1100
+F 0 "#PWR?" H 1750 950 50  0001 C CNN
+F 1 "+3V3" H 1765 1273 50  0000 C CNN
+F 2 "" H 1750 1100 50  0001 C CNN
+F 3 "" H 1750 1100 50  0001 C CNN
+	1    1750 1100
+	1    0    0    -1
+$EndComp
 $EndSCHEMATC
