File: Hardware/Flight/Experiment Board/Experiment Board.sch (KiCad schematic (older format))
At the start: 29 parts, among them J1 Conn_01x05_Female, J2 Conn_01x02, J3 Bus_Connector, J4 Conn_01x03, J5 Conn_01x03, J6 Conn_01x02, J7 Conn_01x02, U4 LSM6DS3, U5 PICLF26K83, U7 ACS711KEXLT-31AB-T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

Commit message: fixed changes in experiment board
Parts:
- removed C16: 1nF, symbol Device:C
- added C10: 0.1uF, Capacitors_SMD:C_0603_HandSoldering, symbol Device:C
- added C6: 100nF, Capacitors_SMD:C_0603_HandSoldering, symbol Device:C
- added C9: 10uF, Capacitors_SMD:C_0603_HandSoldering, symbol Device:C
- C1, C2: footprint (none) -> Capacitors_SMD:C_0603_HandSoldering
- C3: renamed from C4; footprint (none) -> Capacitors_SMD:C_0603_HandSoldering
- C4: renamed from C9; footprint (none) -> Capacitors_SMD:C_0603_HandSoldering
- C5: renamed from C?; footprint (none) -> Capacitors_SMD:C_0603_HandSoldering
- C7: renamed from C3; footprint (none) -> Capacitors_SMD:C_0603_HandSoldering
- C8: renamed from C15; footprint (none) -> Capacitors_SMD:C_0603_HandSoldering
- D1: renamed from D2; footprint (none) -> LEDs:LED_0603_HandSoldering
- D2: renamed from D3; footprint (none) -> LEDs:LED_0603_HandSoldering
- D3: renamed from D4; footprint (none) -> LEDs:LED_0603_HandSoldering
- J1: renamed from J2; footprint (none) -> Payload_Connectors:SolderWirePad_2x_1-5mmDrill
- J2: renamed from J3; footprint (none) -> Payload_Connectors:Pin_Header_Straight_2x10_Pitch2.54mm
- J3: renamed from J4; footprint (none) -> Connectors_Molex:Molex_KK-6410-03_03x2.54mm_Straight
- J4: renamed from J5; footprint (none) -> Connectors_Molex:Molex_KK-6410-03_03x2.54mm_Straight
- J5: renamed from J1; footprint (none) -> Payload_Connectors:PinHeader_5x2.54_SMD_90deg_952-3198-1-ND
- J6: renamed from J7; footprint (none) -> Payload_Connectors:SolderWirePad_2x_1-5mmDrill
- J7: renamed from J6; footprint (none) -> Payload_Connectors:SolderWirePad_2x_1-5mmDrill
- R1, R2, R3, R4, R5: footprint (none) -> Resistors_SMD:R_0603_HandSoldering
- U1: renamed from U?; footprint (none) -> Housings_SSOP:TSSOP-8_4.4x3mm_Pitch0.65mm
- U2: renamed from U5; footprint (none) -> Housings_SOIC:SOIC-28W_7.5x18.7mm_Pitch1.27mm
- U3: renamed from U4; footprint Package_LGA:LGA-14_3x2.5mm_P0.5mm_LayoutBorder3x4y -> Housings_LGA:Bosch_LGA-14_3x2.5mm_Pitch0.5mm
- U4: renamed from U7; footprint (none) -> Payload_StandardPackages:12-PowerWFQFN
- U5: renamed from U?; footprint (none) -> TO_SOT_Packages_SMD:SOT-23-5_HandSoldering
- Y1: footprint (none) -> Crystals:Crystal_HC49-U_Vertical
Connections:
- net labels added: INT0
- wire segments 143 -> 148
