File: Hardware/Flight/Experiment Board/GateDriver.sch (KiCad schematic (older format))
At the start: 8 parts, among them U6 A4919GETTR-T

Commit message: updated battery, experiment board. Added temp sensor to ARM board
Parts:
- removed R2: 10k, symbol Device:R
Connections:
- net labels removed: +5V
- wire segments 50 -> 48
Changed lines of the file:
@@
 Connection ~ 3800 3850
-$Comp
-L Device:R R?
-U 1 1 5CA3645A
-P 3500 3700
-AR Path="/5CA3645A" Ref="R?"  Part="1"
-AR Path="/5CA34EBF/5CA3645A" Ref="R2"  Part="1"
-AR Path="/5CA51947/5CA3645A" Ref="R3"  Part="1"
-AR Path="/5CC8A1AA/5CCA5D1C/5CA3645A" Ref="R2"  Part="1"
-AR Path="/5CCC856A/5CCA5D1C/5CA3645A" Ref="R2"  Part="1"
-F 0 "R2" H 3570 3746 50  0000 L CNN
-F 1 "10k" H 3570 3655 50  0000 L CNN
-F 2 "" V 3430 3700 50  0001 C CNN
-F 3 "~" H 3500 3700 50  0001 C CNN
-	1    3500 3700
-	1    0    0    -1
-$EndComp
-Wire Wire Line
-	3500 3850 3500 3950
-Wire Wire Line
-	3500 3950 4300 3950
-$Comp
-L power:+5V #PWR?
-U 1 1 5CA36463
-P 3500 3550
-AR Path="/5CA36463" Ref="#PWR?"  Part="1"
-AR Path="/5CA34EBF/5CA36463" Ref="#PWR019"  Part="1"
-AR Path="/5CA51947/5CA36463" Ref="#PWR034"  Part="1"
-AR Path="/5CC8A1AA/5CCA5D1C/5CA36463" Ref="#PWR019"  Part="1"
-AR Path="/5CCC856A/5CCA5D1C/5CA36463" Ref="#PWR019"  Part="1"
-F 0 "#PWR019" H 3500 3400 50  0001 C CNN
-F 1 "+5V" H 3515 3723 50  0000 C CNN
-F 2 "" H 3500 3550 50  0001 C CNN
-F 3 "" H 3500 3550 50  0001 C CNN
-	1    3500 3550
-	1    0    0    -1
-$EndComp
-Wire Wire Line
-	3500 3950 3450 3950
-Connection ~ 3500 3950
 $Comp
 L Device:C C?
@@
 Text HLabel 3450 3950 0    50   Input ~ 0
 FAULT
+Wire Wire Line
+	3450 3950 4300 3950
 $EndSCHEMATC

Commit message: fixed changes in experiment board
Parts:
- C17: renamed from C10; footprint (none) -> Capacitors_SMD:C_0603_HandSoldering
- C18: renamed from C11; footprint (none) -> Capacitors_SMD:C_0603_HandSoldering
- C19: renamed from C12; footprint (none) -> Capacitors_SMD:C_0603_HandSoldering
- C20: renamed from C13; footprint (none) -> Capacitors_SMD:C_0603_HandSoldering
- C21: renamed from C14; footprint (none) -> Capacitors_SMD:C_0603_HandSoldering
- D8: renamed from D1; footprint (none) -> Diodes_SMD:D_SMA_Handsoldering
- U10: renamed from U6; footprint (none) -> Housings_DFN_QFN:QFN-28-1EP_5x5mm_Pitch0.5mm
Changed lines of the file:
@@
 P 5050 3850
 AR Path="/5CA36403" Ref="U?"  Part="1"
-AR Path="/5CA34EBF/5CA36403" Ref="U6"  Part="1"
-AR Path="/5CA51947/5CA36403" Ref="U11"  Part="1"
-AR Path="/5CC8A1AA/5CCA5D1C/5CA36403" Ref="U6"  Part="1"
-AR Path="/5CCC856A/5CCA5D1C/5CA36403" Ref="U6"  Part="1"
-F 0 "U6" H 5000 3750 50  0000 L CNN
+AR Path="/5CA34EBF/5CA36403" Ref="U?"  Part="1"
+AR Path="/5CA51947/5CA36403" Ref="U?"  Part="1"
+AR Path="/5CC8A1AA/5CCA5D1C/5CA36403" Ref="U10"  Part="1"
+AR Path="/5CCC856A/5CCA5D1C/5CA36403" Ref="U15"  Part="1"
+F 0 "U15" H 5000 3750 50  0000 L CNN
 F 1 "A4919GETTR-T" H 4800 3650 50  0000 L CNN
-F 2 "" H 4350 3900 50  0001 C CNN
+F 2 "Housings_DFN_QFN:QFN-28-1EP_5x5mm_Pitch0.5mm" H 4350 3900 50  0001 C CNN
 F 3 "" H 4350 3900 50  0001 C CNN
 	1    5050 3850
@@
 P 4850 2450
 AR Path="/5CA3640A" Ref="C?"  Part="1"
-AR Path="/5CA34EBF/5CA3640A" Ref="C11"  Part="1"
-AR Path="/5CA51947/5CA3640A" Ref="C20"  Part="1"
-AR Path="/5CC8A1AA/5CCA5D1C/5CA3640A" Ref="C11"  Part="1"
-AR Path="/5CCC856A/5CCA5D1C/5CA3640A" Ref="C11"  Part="1"
-F 0 "C11" H 4750 2650 50  0000 C CNN
+AR Path="/5CA34EBF/5CA3640A" Ref="C?"  Part="1"
+AR Path="/5CA51947/5CA3640A" Ref="C?"  Part="1"
+AR Path="/5CC8A1AA/5CCA5D1C/5CA3640A" Ref="C18"  Part="1"
+AR Path="/5CCC856A/5CCA5D1C/5CA3640A" Ref="C29"  Part="1"
+F 0 "C29" H 4750 2650 50  0000 C CNN
 F 1 "470nF" H 4700 2550 50  0000 C CNN
-F 2 "" H 4888 2300 50  0001 C CNN
+F 2 "Capacitors_SMD:C_0603_HandSoldering" H 4888 2300 50  0001 C CNN
 F 3 "~" H 4850 2450 50  0001 C CNN
 	1    4850 2450
@@
 P 4550 2800
 AR Path="/5CA36411" Ref="D?"  Part="1"
-AR Path="/5CA34EBF/5CA36411" Ref="D1"  Part="1"
-AR Path="/5CA51947/5CA36411" Ref="D2"  Part="1"
-AR Path="/5CC8A1AA/5CCA5D1C/5CA36411" Ref="D1"  Part="1"
-AR Path="/5CCC856A/5CCA5D1C/5CA36411" Ref="D1"  Part="1"
-F 0 "D1" H 4550 3065 50  0000 C CNN
+AR Path="/5CA34EBF/5CA36411" Ref="D?"  Part="1"
+AR Path="/5CA51947/5CA36411" Ref="D?"  Part="1"
+AR Path="/5CC8A1AA/5CCA5D1C/5CA36411" Ref="D8"  Part="1"
+AR Path="/5CCC856A/5CCA5D1C/5CA36411" Ref="D13"  Part="1"
+F 0 "D13" H 4550 3065 50  0000 C CNN
 F 1 "DIODE" H 4550 2974 50  0000 C CNN
-F 2 "" H 4550 2800 50  0001 C CNN
+F 2 "Diodes_SMD:D_SMA_Handsoldering" H 4550 2800 50  0001 C CNN
 F 3 "" H 4550 2800 50  0001 C CNN
 	1    4550 2800
@@
 P 4250 2500
 AR Path="/5CA36419" Ref="#PWR?"  Part="1"
-AR Path="/5CA34EBF/5CA36419" Ref="#PWR023"  Part="1"
-AR Path="/5CA51947/5CA36419" Ref="#PWR038"  Part="1"
-AR Path="/5CC8A1AA/5CCA5D1C/5CA36419" Ref="#PWR023"  Part="1"
-AR Path="/5CCC856A/5CCA5D1C/5CA36419" Ref="#PWR023"  Part="1"
-F 0 "#PWR023" H 4250 2350 50  0001 C CNN
+AR Path="/5CA34EBF/5CA36419" Ref="#PWR?"  Part="1"
+AR Path="/5CA51947/5CA36419" Ref="#PWR?"  Part="1"
+AR Path="/5CC8A1AA/5CCA5D1C/5CA36419" Ref="#PWR051"  Part="1"
+AR Path="/5CCC856A/5CCA5D1C/5CA36419" Ref="#PWR067"  Part="1"
+F 0 "#PWR067" H 4250 2350 50  0001 C CNN
 F 1 "+24V" H 4265 2673 50  0000 C CNN
 F 2 "" H 4250 2500 50  0001 C CNN
@@
 P 4150 3050
 AR Path="/5CA36421" Ref="C?"  Part="1"
-AR Path="/5CA34EBF/5CA36421" Ref="C10"  Part="1"
-AR Path="/5CA51947/5CA36421" Ref="C19"  Part="1"
-AR Path="/5CC8A1AA/5CCA5D1C/5CA36421" Ref="C10"  Part="1"
-AR Path="/5CCC856A/5CCA5D1C/5CA36421" Ref="C10"  Part="1"
-F 0 "C10" V 3898 3050 50  0000 C CNN
+AR Path="/5CA34EBF/5CA36421" Ref="C?"  Part="1"
+AR Path="/5CA51947/5CA36421" Ref="C?"  Part="1"
+AR Path="/5CC8A1AA/5CCA5D1C/5CA36421" Ref="C17"  Part="1"
+AR Path="/5CCC856A/5CCA5D1C/5CA36421" Ref="C28"  Part="1"
+F 0 "C28" V 3898 3050 50  0000 C CNN
 F 1 "220nF" V 3989 3050 50  0000 C CNN
-F 2 "" H 4188 2900 50  0001 C CNN
+F 2 "Capacitors_SMD:C_0603_HandSoldering" H 4188 2900 50  0001 C CNN
 F 3 "~" H 4150 3050 50  0001 C CNN
 	1    4150 3050
@@
 P 4000 3150
 AR Path="/5CA3642A" Ref="#PWR?"  Part="1"
-AR Path="/5CA34EBF/5CA3642A" Ref="#PWR022"  Part="1"
-AR Path="/5CA51947/5CA3642A" Ref="#PWR037"  Part="1"
-AR Path="/5CC8A1AA/5CCA5D1C/5CA3642A" Ref="#PWR022"  Part="1"
-AR Path="/5CCC856A/5CCA5D1C/5CA3642A" Ref="#PWR022"  Part="1"
-F 0 "#PWR022" H 4000 2900 50  0001 C CNN
+AR Path="/5CA34EBF/5CA3642A" Ref="#PWR?"  Part="1"
+AR Path="/5CA51947/5CA3642A" Ref="#PWR?"  Part="1"
+AR Path="/5CC8A1AA/5CCA5D1C/5CA3642A" Ref="#PWR050"  Part="1"
+AR Path="/5CCC856A/5CCA5D1C/5CA3642A" Ref="#PWR066"  Part="1"
+F 0 "#PWR066" H 4000 2900 50  0001 C CNN
 F 1 "GND" H 4005 2977 50  0000 C CNN
 F 2 "" H 4000 3150 50  0001 C CNN
@@
 P 5700 2550
 AR Path="/5CA36432" Ref="C?"  Part="1"
-AR Path="/5CA34EBF/5CA36432" Ref="C13"  Part="1"
-AR Path="/5CA51947/5CA36432" Ref="C22"  Part="1"
-AR Path="/5CC8A1AA/5CCA5D1C/5CA36432" Ref="C13"  Part="1"
-AR Path="/5CCC856A/5CCA5D1C/5CA36432" Ref="C13"  Part="1"
-F 0 "C13" V 5952 2550 50  0000 C CNN
+AR Path="/5CA34EBF/5CA36432" Ref="C?"  Part="1"
+AR Path="/5CA51947/5CA36432" Ref="C?"  Part="1"
+AR Path="/5CC8A1AA/5CCA5D1C/5CA36432" Ref="C20"  Part="1"
+AR Path="/5CCC856A/5CCA5D1C/5CA36432" Ref="C31"  Part="1"
+F 0 "C31" V 5952 2550 50  0000 C CNN
 F 1 "388nF" V 5861 2550 50  0000 C CNN
-F 2 "" H 5738 2400 50  0001 C CNN
+F 2 "Capacitors_SMD:C_0603_HandSoldering" H 5738 2400 50  0001 C CNN
 F 3 "~" H 5700 2550 50  0001 C CNN
 	1    5700 2550
@@
 P 6100 2600
 AR Path="/5CA3643B" Ref="#PWR?"  Part="1"
-AR Path="/5CA34EBF/5CA3643B" Ref="#PWR025"  Part="1"
-AR Path="/5CA51947/5CA3643B" Ref="#PWR040"  Part="1"
-AR Path="/5CC8A1AA/5CCA5D1C/5CA3643B" Ref="#PWR025"  Part="1"
-AR Path="/5CCC856A/5CCA5D1C/5CA3643B" Ref="#PWR025"  Part="1"
-F 0 "#PWR025" H 6100 2350 50  0001 C CNN
+AR Path="/5CA34EBF/5CA3643B" Ref="#PWR?"  Part="1"
+AR Path="/5CA51947/5CA3643B" Ref="#PWR?"  Part="1"
+AR Path="/5CC8A1AA/5CCA5D1C/5CA3643B" Ref="#PWR053"  Part="1"
+AR Path="/5CCC856A/5CCA5D1C/5CA3643B" Ref="#PWR069"  Part="1"
+F 0 "#PWR069" H 6100 2350 50  0001 C CNN
 F 1 "GND" H 6105 2427 50  0000 C CNN
 F 2 "" H 6100 2600 50  0001 C CNN
@@
 P 3800 2500
 AR Path="/5CA36443" Ref="#PWR?"  Part="1"
-AR Path="/5CA34EBF/5CA36443" Ref="#PWR020"  Part="1"
-AR Path="/5CA51947/5CA36443" Ref="#PWR035"  Part="1"
-AR Path="/5CC8A1AA/5CCA5D1C/5CA36443" Ref="#PWR020"  Part="1"
-AR Path="/5CCC856A/5CCA5D1C/5CA36443" Ref="#PWR020"  Part="1"
-F 0 "#PWR020" H 3800 2350 50  0001 C CNN
+AR Path="/5CA34EBF/5CA36443" Ref="#PWR?"  Part="1"
+AR Path="/5CA51947/5CA36443" Ref="#PWR?"  Part="1"
+AR Path="/5CC8A1AA/5CCA5D1C/5CA36443" Ref="#PWR048"  Part="1"
+AR Path="/5CCC856A/5CCA5D1C/5CA36443" Ref="#PWR064"  Part="1"
+F 0 "#PWR064" H 3800 2350 50  0001 C CNN
 F 1 "+24V" H 3815 2673 50  0000 C CNN
 F 2 "" H 3800 2500 50  0001 C CNN
@@
 P 3800 4200
 AR Path="/5CA36450" Ref="#PWR?"  Part="1"
-AR Path="/5CA34EBF/5CA36450" Ref="#PWR021"  Part="1"
-AR Path="/5CA51947/5CA36450" Ref="#PWR036"  Part="1"
-AR Path="/5CC8A1AA/5CCA5D1C/5CA36450" Ref="#PWR021"  Part="1"
-AR Path="/5CCC856A/5CCA5D1C/5CA36450" Ref="#PWR021"  Part="1"
-F 0 "#PWR021" H 3800 3950 50  0001 C CNN
+AR Path="/5CA34EBF/5CA36450" Ref="#PWR?"  Part="1"
+AR Path="/5CA51947/5CA36450" Ref="#PWR?"  Part="1"
+AR Path="/5CC8A1AA/5CCA5D1C/5CA36450" Ref="#PWR049"  Part="1"
+AR Path="/5CCC856A/5CCA5D1C/5CA36450" Ref="#PWR065"  Part="1"
+F 0 "#PWR065" H 3800 3950 50  0001 C CNN
 F 1 "GND" H 3805 4027 50  0000 C CNN
 F 2 "" H 3800 4200 50  0001 C CNN
@@
 P 5150 2750
 AR Path="/5CA3646C" Ref="C?"  Part="1"
-AR Path="/5CA34EBF/5CA3646C" Ref="C12"  Part="1"
-AR Path="/5CA51947/5CA3646C" Ref="C21"  Part="1"
-AR Path="/5CC8A1AA/5CCA5D1C/5CA3646C" Ref="C12"  Part="1"
-AR Path="/5CCC856A/5CCA5D1C/5CA3646C" Ref="C12"  Part="1"
-F 0 "C12" H 5300 2800 50  0000 L CNN
+AR Path="/5CA34EBF/5CA3646C" Ref="C?"  Part="1"
+AR Path="/5CA51947/5CA3646C" Ref="C?"  Part="1"
+AR Path="/5CC8A1AA/5CCA5D1C/5CA3646C" Ref="C19"  Part="1"
+AR Path="/5CCC856A/5CCA5D1C/5CA3646C" Ref="C30"  Part="1"
+F 0 "C30" H 5300 2800 50  0000 L CNN
 F 1 "9.7nF" H 5300 2700 50  0000 L CNN
-F 2 "" H 5188 2600 50  0001 C CNN
+F 2 "Capacitors_SMD:C_0603_HandSoldering" H 5188 2600 50  0001 C CNN
 F 3 "~" H 5150 2750 50  0001 C CNN
 	1    5150 2750
@@
 P 5150 4550
 AR Path="/5CA36479" Ref="#PWR?"  Part="1"
-AR Path="/5CA34EBF/5CA36479" Ref="#PWR024"  Part="1"
-AR Path="/5CA51947/5CA36479" Ref="#PWR039"  Part="1"
-AR Path="/5CC8A1AA/5CCA5D1C/5CA36479" Ref="#PWR024"  Part="1"
-AR Path="/5CCC856A/5CCA5D1C/5CA36479" Ref="#PWR024"  Part="1"
-F 0 "#PWR024" H 5150 4300 50  0001 C CNN
+AR Path="/5CA34EBF/5CA36479" Ref="#PWR?"  Part="1"
+AR Path="/5CA51947/5CA36479" Ref="#PWR?"  Part="1"
+AR Path="/5CC8A1AA/5CCA5D1C/5CA36479" Ref="#PWR052"  Part="1"
+AR Path="/5CCC856A/5CCA5D1C/5CA36479" Ref="#PWR068"  Part="1"
+F 0 "#PWR068" H 5150 4300 50  0001 C CNN
 F 1 "GND" H 5155 4377 50  0000 C CNN
 F 2 "" H 5150 4550 50  0001 C CNN
@@
 P 5950 3650
 AR Path="/5CA3647F" Ref="C?"  Part="1"
-AR Path="/5CA34EBF/5CA3647F" Ref="C14"  Part="1"
-AR Path="/5CA51947/5CA3647F" Ref="C23"  Part="1"
-AR Path="/5CC8A1AA/5CCA5D1C/5CA3647F" Ref="C14"  Part="1"
-AR Path="/5CCC856A/5CCA5D1C/5CA3647F" Ref="C14"  Part="1"
-F 0 "C14" V 5900 3900 50  0000 C CNN
+AR Path="/5CA34EBF/5CA3647F" Ref="C?"  Part="1"
+AR Path="/5CA51947/5CA3647F" Ref="C?"  Part="1"
+AR Path="/5CC8A1AA/5CCA5D1C/5CA3647F" Ref="C21"  Part="1"
+AR Path="/5CCC856A/5CCA5D1C/5CA3647F" Ref="C32"  Part="1"
+F 0 "C32" V 5900 3900 50  0000 C CNN
 F 1 "9.7nF" V 6000 3950 50  0000 C CNN
-F 2 "" H 5988 3500 50  0001 C CNN
+F 2 "Capacitors_SMD:C_0603_HandSoldering" H 5988 3500 50  0001 C CNN
 F 3 "~" H 5950 3650 50  0001 C CNN
 	1    5950 3650
