File: Hardware/Flight/Experiment Board/HalfBridge.sch (KiCad schematic (older format))
At the start: 4 parts, among them U2 SIRA22DP-T1-RE3, U3 SIRA22DP-T1-RE3

Commit message: fixed changes in experiment board
Parts:
- removed U2, U3: SIRA22DP-T1-RE3, symbol Payload_Transistors:SIRA22DP-T1-RE3
- added D4, D5: DIODE, Diodes_SMD:D_SMA_Handsoldering, symbol pspice:DIODE
- added U6, U7: TPH1R204PL,L1Q, Payload_StandardPackages:TPH8R80ANH, symbol Payload_Transistors:TPH1R204PL,L1Q
- C13: renamed from C6; footprint (none) -> Capacitors_SMD:C_0603_HandSoldering
- C14: renamed from C7; footprint (none) -> Capacitors_SMD:C_0603_HandSoldering
Connections:
- wire segments 35 -> 44
