File: Hardware/Flight/Pressure Breakout/Pressure Breakout.sch (KiCad schematic (older format))
At the start: 3 parts

Commit message: addressed Alex's ARM review comments
Parts:
- added J1: Conn_01x03, Connectors_Molex:Molex_KK-6410-03_03x2.54mm_Straight, symbol Connector_Generic:Conn_01x03
- C1, C2: renamed from C?; footprint (none) -> Capacitors_SMD:C_0603_HandSoldering
- U1: renamed from U?; footprint (none) -> Payload_StandardPackages:DIP-6_W11.25mm
Connections:
- net labels added: +5V, VOUT
- wire segments 6 -> 12
Changed lines of the file:
@@
 EESchema Schematic File Version 4
+LIBS:Pressure Breakout-cache
 EELAYER 26 0
 EELAYER END
@@
 $EndDescr
 $Comp
-L Payload_Sensors:ABPDANT005PGAA5 U?
+L Payload_Sensors:ABPDANT005PGAA5 U1
 U 1 1 5C9BD3E8
 P 5600 3450
-F 0 "U?" H 5625 3775 50  0000 C CNN
+F 0 "U1" H 5625 3775 50  0000 C CNN
 F 1 "ABPDANT005PGAA5" H 5625 3684 50  0000 C CNN
-F 2 "" H 5600 3450 50  0001 C CNN
+F 2 "Payload_StandardPackages:DIP-6_W11.25mm" H 5600 3450 50  0001 C CNN
 F 3 "" H 5600 3450 50  0001 C CNN
 	1    5600 3450
@@
 $EndComp
 $Comp
-L Device:C C?
+L Device:C C2
 U 1 1 5C9BD46B
 P 6250 3750
-F 0 "C?" H 6365 3796 50  0000 L CNN
+F 0 "C2" H 6365 3796 50  0000 L CNN
 F 1 "0.1uF" H 6365 3705 50  0000 L CNN
-F 2 "" H 6288 3600 50  0001 C CNN
+F 2 "Capacitors_SMD:C_0603_HandSoldering" H 6288 3600 50  0001 C CNN
 F 3 "~" H 6250 3750 50  0001 C CNN
 	1    6250 3750
@@
 	6250 3550 6250 3600
 $Comp
-L power:GND #PWR?
+L power:GND #PWR03
 U 1 1 5C9BD604
 P 6250 3900
-F 0 "#PWR?" H 6250 3650 50  0001 C CNN
+F 0 "#PWR03" H 6250 3650 50  0001 C CNN
 F 1 "GND" H 6255 3727 50  0000 C CNN
 F 2 "" H 6250 3900 50  0001 C CNN
@@
 $EndComp
 $Comp
-L Device:C C?
+L Device:C C1
 U 1 1 5C9BD66E
 P 5000 3750
-F 0 "C?" H 5115 3796 50  0000 L CNN
+F 0 "C1" H 5115 3796 50  0000 L CNN
 F 1 "0.001uF" H 5115 3705 50  0000 L CNN
-F 2 "" H 5038 3600 50  0001 C CNN
+F 2 "Capacitors_SMD:C_0603_HandSoldering" H 5038 3600 50  0001 C CNN
 F 3 "~" H 5000 3750 50  0001 C CNN
 	1    5000 3750
@@
 	5000 3550 5050 3550
 $Comp
-L power:GND #PWR?
+L power:GND #PWR02
 U 1 1 5C9BD731
 P 5000 3900
-F 0 "#PWR?" H 5000 3650 50  0001 C CNN
+F 0 "#PWR02" H 5000 3650 50  0001 C CNN
 F 1 "GND" H 5005 3727 50  0000 C CNN
 F 2 "" H 5000 3900 50  0001 C CNN
@@
 $EndComp
 $Comp
-L power:GND #PWR?
+L power:GND #PWR01
 U 1 1 5C9BD7F5
-P 4800 3450
-F 0 "#PWR?" H 4800 3200 50  0001 C CNN
-F 1 "GND" H 4805 3277 50  0000 C CNN
-F 2 "" H 4800 3450 50  0001 C CNN
-F 3 "" H 4800 3450 50  0001 C CNN
-	1    4800 3450
+P 4500 3450
+F 0 "#PWR01" H 4500 3200 50  0001 C CNN
+F 1 "GND" H 4505 3277 50  0000 C CNN
+F 2 "" H 4500 3450 50  0001 C CNN
+F 3 "" H 4500 3450 50  0001 C CNN
+	1    4500 3450
 	1    0    0    -1
 $EndComp
 Wire Wire Line
-	4800 3450 4800 3350
+	4500 3450 4500 3350
 Wire Wire Line
-	4800 3350 5050 3350
+	4500 3350 5050 3350
 NoConn ~ 5050 3450
 NoConn ~ 6200 3450
 NoConn ~ 6200 3350
+$Comp
+L power:+5V #PWR04
+U 1 1 5CCFF07E
+P 6400 3350
+F 0 "#PWR04" H 6400 3200 50  0001 C CNN
+F 1 "+5V" H 6415 3523 50  0000 C CNN
+F 2 "" H 6400 3350 50  0001 C CNN
+F 3 "" H 6400 3350 50  0001 C CNN
+	1    6400 3350
+	1    0    0    -1
+$EndComp
+Wire Wire Line
+	6400 3350 6400 3550
+Wire Wire Line
+	6400 3550 6250 3550
+Connection ~ 6250 3550
+Text Label 5000 3550 2    50   ~ 0
+VOUT
+$Comp
+L Connector_Generic:Conn_01x03 J1
+U 1 1 5CCFF23E
+P 8200 3450
+F 0 "J1" H 8280 3492 50  0000 L CNN
+F 1 "Conn_01x03" H 8280 3401 50  0000 L CNN
+F 2 "Connectors_Molex:Molex_KK-6410-03_03x2.54mm_Straight" H 8200 3450 50  0001 C CNN
+F 3 "~" H 8200 3450 50  0001 C CNN
+	1    8200 3450
+	1    0    0    -1
+$EndComp
+$Comp
+L power:+5V #PWR05
+U 1 1 5CCFF27C
+P 7950 3300
+F 0 "#PWR05" H 7950 3150 50  0001 C CNN
+F 1 "+5V" H 7965 3473 50  0000 C CNN
+F 2 "" H 7950 3300 50  0001 C CNN
+F 3 "" H 7950 3300 50  0001 C CNN
+	1    7950 3300
+	1    0    0    -1
+$EndComp
+Wire Wire Line
+	7950 3300 7950 3350
+Wire Wire Line
+	7950 3350 8000 3350
+Text Label 8000 3450 2    50   ~ 0
+VOUT
+$Comp
+L power:GND #PWR06
+U 1 1 5CCFF3CA
+P 7950 3600
+F 0 "#PWR06" H 7950 3350 50  0001 C CNN
+F 1 "GND" H 7955 3427 50  0000 C CNN
+F 2 "" H 7950 3600 50  0001 C CNN
+F 3 "" H 7950 3600 50  0001 C CNN
+	1    7950 3600
+	1    0    0    -1
+$EndComp
+Wire Wire Line
+	7950 3600 7950 3550
+Wire Wire Line
+	7950 3550 8000 3550
 $EndSCHEMATC

Commit message: updated pressure breakout
Changed lines of the file:
@@
 L Connector_Generic:Conn_01x03 J1
 U 1 1 5CCFF23E
-P 8200 3450
-F 0 "J1" H 8280 3492 50  0000 L CNN
-F 1 "Conn_01x03" H 8280 3401 50  0000 L CNN
-F 2 "Connectors_Molex:Molex_KK-6410-03_03x2.54mm_Straight" H 8200 3450 50  0001 C CNN
-F 3 "~" H 8200 3450 50  0001 C CNN
-	1    8200 3450
+P 7150 3500
+F 0 "J1" H 7230 3542 50  0000 L CNN
+F 1 "Conn_01x03" H 7230 3451 50  0000 L CNN
+F 2 "Connectors_Molex:Molex_KK-6410-03_03x2.54mm_Straight" H 7150 3500 50  0001 C CNN
+F 3 "~" H 7150 3500 50  0001 C CNN
+	1    7150 3500
 	1    0    0    -1
 $EndComp
@@
 L power:+5V #PWR05
 U 1 1 5CCFF27C
-P 7950 3300
-F 0 "#PWR05" H 7950 3150 50  0001 C CNN
-F 1 "+5V" H 7965 3473 50  0000 C CNN
-F 2 "" H 7950 3300 50  0001 C CNN
-F 3 "" H 7950 3300 50  0001 C CNN
-	1    7950 3300
+P 6900 3350
+F 0 "#PWR05" H 6900 3200 50  0001 C CNN
+F 1 "+5V" H 6915 3523 50  0000 C CNN
+F 2 "" H 6900 3350 50  0001 C CNN
+F 3 "" H 6900 3350 50  0001 C CNN
+	1    6900 3350
 	1    0    0    -1
 $EndComp
 Wire Wire Line
-	7950 3300 7950 3350
+	6900 3350 6900 3400
 Wire Wire Line
-	7950 3350 8000 3350
-Text Label 8000 3450 2    50   ~ 0
+	6900 3400 6950 3400
+Text Label 6950 3500 2    50   ~ 0
 VOUT
 $Comp
 L power:GND #PWR06
 U 1 1 5CCFF3CA
-P 7950 3600
-F 0 "#PWR06" H 7950 3350 50  0001 C CNN
-F 1 "GND" H 7955 3427 50  0000 C CNN
-F 2 "" H 7950 3600 50  0001 C CNN
-F 3 "" H 7950 3600 50  0001 C CNN
-	1    7950 3600
+P 6900 3650
+F 0 "#PWR06" H 6900 3400 50  0001 C CNN
+F 1 "GND" H 6905 3477 50  0000 C CNN
+F 2 "" H 6900 3650 50  0001 C CNN
+F 3 "" H 6900 3650 50  0001 C CNN
+	1    6900 3650
 	1    0    0    -1
 $EndComp
 Wire Wire Line
-	7950 3600 7950 3550
+	6900 3650 6900 3600
 Wire Wire Line
-	7950 3550 8000 3550
+	6900 3600 6950 3600
 $EndSCHEMATC
